File: MicropendousX/Hardware/MicropendousX-LPC183x/MicropendousX-LPC183x-LCD.sch (KiCad schematic (older format))
At the start: 18 parts, among them IC1 LPC185X, IC6 CAT4237, U5 NHD-TS, U6 NHD-3.5-320240MF-ATXL-T-1

Commit message: Update unfinished LPC183x-based design.
Parts:
- removed C100: 4u7, symbol C_MINI
- removed C101, C102: 0u1, symbol C_MINI
- removed C123, C124: 5pF, symbol C_MINI
- removed U5: NHD-TS, symbol NHD-TS
- removed U6: NHD-3.5-320240MF-ATXL-T-1, symbol NHD-3.5-320240MF-ATXL-T-1
- added IC10: STMPE610, symbol STMPE610
- added TP3: IN2, symbol CONN_1
- added TP6: IN3, symbol CONN_1
- added U5: COG-C172MVHC-04, symbol COG-C172MVHC-04
- IC1: value LPC185X -> LPC183X
- renumbered C96 to C18, C97 to C19, C98 to C20, C99 to C21, IC6 to IC9, L2 to L4, R34 to R10, R35 to R11, R33 to R9
Connections:
- net labels added: GPS_ON-nOFF, GPS_WAKEUP, I2C1_SCL-U3_RXD, I2C1_SDA-U3_TXD, WAKEUP0
- net labels removed: GNDPWR, LCD_DB00, LCD_DB01, LCD_DB02, LCD_DB03, LCD_DB04, LCD_DB05, LCD_DB06, LCD_DB07, LCD_DB08, LCD_DB09, LCD_DB10, LCD_DB11, LCD_DB12, LCD_DB13, LCD_DB14, LCD_DB15, LCD_DB16, LCD_DB17, LCD_DB18, LCD_DB19, LCD_DB20, LCD_DB21, LCD_DB22, LCD_DB23, LCD_DOTCLK, LCD_HSYNC, LCD_VSYNC, X+, X-, Y+, Y-
- wire segments 66 -> 77
- no-connect marks 17 -> 30
Other:
- note removed: "Filter capacitors of 5pF allow\nfor faster settling time."
- note removed: "Molex 512965494"
- note removed: "Molex 522070485"
- note removed: "Use CTOUT_14 for PWM"
- moved on the sheet: C18, C19, C20, C21, IC9, L4, R10, R11, R9
