File: MicropendousX/Hardware/MicropendousX-LPC183x/MicropendousX-LPC183x-EMI.sch (KiCad schematic (older format))
At the start: 5 parts, among them IC1 LPC183X, P1 CONN-24, P2 CONN-24

Commit message: Update unfinished LPC183x-based design.
Parts:
- added IC3: NAND, symbol NAND_TSOP48
Connections:
- net labels added: GPS_CTS, GPS_RTS, GPS_RXD, GPS_TXD
- no-connect marks 53 -> 49
Changed lines of the file:
@@
-EESchema Schematic File Version 2  date 8/15/2011 4:26:38 PM
+EESchema Schematic File Version 2  date 8/20/2011 8:34:09 PM
 LIBS:power
 LIBS:device
@@
 $Descr A4 11700 8267
 encoding utf-8
-Sheet 2 7
+Sheet 4 9
 Title "MicropendousX-LPC183x"
-Date "15 aug 2011"
+Date "21 aug 2011"
 Rev "1.0"
 Comp "Opendous Inc."
@@
 Comment4 "www.MicropendousX.org"
 $EndDescr
+Text GLabel 4000 1750 1    40   Output ~ 0
+GPS_CTS
+Text GLabel 4300 1750 1    40   Input ~ 0
+GPS_TXD
+Text GLabel 4600 1750 1    40   Input ~ 0
+GPS_RTS
+Text GLabel 4200 1750 1    40   Output ~ 0
+GPS_RXD
+Text GLabel 9600 1250 1    40   BiDi ~ 0
+~EMC_CS0~
+Text GLabel 9500 1250 1    40   BiDi ~ 0
+~EMC_OE~
+Text GLabel 9400 1250 1    40   BiDi ~ 0
+~EMC_WE~
+Text GLabel 10550 1250 1    40   BiDi ~ 0
+~EMC_RAS~
+Text GLabel 10450 1250 1    40   BiDi ~ 0
+~EMC_CAS~
+Text GLabel 10000 1250 1    40   BiDi ~ 0
+~EMC_BLS0~
+Text GLabel 10250 1850 1    40   BiDi ~ 0
+EMC_D00
+Text GLabel 10350 1850 1    40   BiDi ~ 0
+EMC_D01
+Text GLabel 10550 1850 1    40   BiDi ~ 0
+EMC_D03
+Text GLabel 10450 1850 1    40   BiDi ~ 0
+EMC_D02
+Text GLabel 10750 1850 1    40   BiDi ~ 0
+EMC_D05
+Text GLabel 10650 1850 1    40   BiDi ~ 0
+EMC_D04
+Text GLabel 10950 1850 1    40   BiDi ~ 0
+EMC_D07
+Text GLabel 10850 1850 1    40   BiDi ~ 0
+EMC_D06
+$Comp
+L NAND_TSOP48 IC3
+U 1 1 4E4F96C3
+P 10250 3200
+F 0 "IC3" H 9950 2300 40  0000 C CNN
+F 1 "NAND" H 10000 4150 40  0000 C CNN
+	1    10250 3200
+	1    0    0    -1
+$EndComp
 $Comp
 L CONN-24 P2
@@
 NoConn ~ 4800 1750
 NoConn ~ 4700 1750
-NoConn ~ 4600 1750
 NoConn ~ 4500 1750
 NoConn ~ 4400 1750
-NoConn ~ 4300 1750
-NoConn ~ 4200 1750
 NoConn ~ 4100 1750
-NoConn ~ 4000 1750
 NoConn ~ 3650 6350
 NoConn ~ 8350 1750
@@
 Connection ~ 10200 5750
 $Comp
-L VDDIO_3V3 #PWR01
+L VDDIO_3V3 #PWR031
 U 1 1 4E23BF04
 P 10300 5400
-F 0 "#PWR01" H 10300 5500 30  0001 C CNN
+F 0 "#PWR031" H 10300 5500 30  0001 C CNN
 F 1 "VDDIO_3V3" H 10300 5500 30  0000 C CNN
 	1    10300 5400

Commit message: Updated LPC183x Hardware Design
Parts:
- removed unit 6 of IC1
- removed unit 4 of IC1
- removed IC3: NAND, symbol NAND_TSOP48
- removed P1, P2: CONN-24, symbol CONN-24
- removed R54, R55: 2k2, symbol R_MINI
- added C118: 10u, symbol C_MINI
- added C119: 0u1, symbol C_MINI
- added C120: u01, symbol C_MINI
- added D2, D3: MBR120, symbol D_SCHOTTKY
- added IC5: TPS22960, symbol TPS22960
- added U11: MMC, symbol CONN_MMC_AMPHENOL_101-00565
Connections:
- net labels added: CLKOUT-I2S1_RX_SCK, EMC_D02-MMC_DAT0, EMC_D03-MMC_DAT1, EMC_D04-MMC_DAT2, EMC_D05-MMC_DAT3, EMC_D06-MMC_CD, GND, GPIO0_11, GPIO3_3, GPIO3_4, GPIO5_0-EMC_A13-ENET_MDC, GPIO5_1-EMC_A12, MMC_CLK, MMC_VDD, VDD1V8, ~EMC_CS0~-MMC_POW, ~EMC_WE~-MMC_CMD
- net labels removed: ADC0_0-DAC, ADC0_1, ADC0_2, ADC0_3, ADCTRIG1, CLK0, EMC_A12, EMC_A13-ENET_MDC, EMC_CLK3, EMC_D02, EMC_D03, EMC_D04, EMC_D05, EMC_D06, ENET_MDIO, ENET_REF_CLK-SSP1_SCK, ENET_RXD0, ENET_RXD1-SSP1_MISO, ENET_RX_DV, ENET_RX_ER, ENET_TXD0, ENET_TXD1-SSP1_SSEL, ENET_TX_EN-SSP1_MOSI, GPS_CTS, GPS_RTS, GPS_RXD, GPS_TXD, GP_CLKIN, I2C1_SCL, I2C1_SCL-U3_RXD, I2C1_SDA, I2C1_SDA-U3_TXD, ~EMC_BLS0~, ~EMC_CAS~, ~EMC_CS0~, ~EMC_RAS~, ~EMC_WE~
- wire segments 10 -> 13
- no-connect marks 49 -> 51
Other:
- note added: "Slew Rate set to 660uS"
- note added: "Used in Sheet 2 -\nOpennect Connector"

Commit message: Updated LPC183x Hardware Design
Connections:
- net labels added: GPIO5_2
- net labels removed: EMC_A11
Other:
- note added: "From Sheet 2 -\nOpennect Connector"
Changed lines of the file:
@@
-EESchema Schematic File Version 2  date 9/18/2011 3:49:57 PM
+EESchema Schematic File Version 2  date 9/18/2011 8:03:49 PM
 LIBS:power
 LIBS:device
@@
 Sheet 3 7
 Title "MicropendousX-LPC183x"
-Date "18 sep 2011"
+Date "19 sep 2011"
 Rev "1.0"
 Comp "Opendous Inc."
@@
 Comment4 "www.MicropendousX.org"
 $EndDescr
+Text Notes 5300 6800 0    30   ~ 0
+From Sheet 2 -\nOpennect Connector
 Text Notes 10050 1950 1    40   ~ 0
 Used in Sheet 2 -\nOpennect Connector
@@
 Text GLabel 3500 2050 1    40   BiDi ~ 0
 GPIO5_0-EMC_A13-ENET_MDC
-Text GLabel 3300 1950 1    40   BiDi ~ 0
-EMC_A11
+Text GLabel 3300 2050 1    40   BiDi ~ 0
+GPIO5_2
 Text GLabel 3200 1950 1    40   BiDi ~ 0
 EMC_A10

Commit message: Updated LPC183x Hardware Design
Parts:
- removed D2, D3: MBR120, symbol D_SCHOTTKY
- removed IC5: TPS22960, symbol TPS22960
- added C116: 0u1, symbol C_MINI
- added C117: 470p, symbol C_MINI
- added IC5: FDC6331, symbol LOAD_SWITCH
- added R51: 199k, symbol R_MINI
- added R52: 10k, symbol R_MINI
Connections:
- net labels added: GPIO5_0-EMC_A13, R1-C1, R2, ~EMC_CS0~, ~EMC_RAS~
- net labels removed: GPIO3_4, GPIO5_0-EMC_A13-ENET_MDC, VDD1V8, ~EMC_CS0~-MMC_POW
- wire segments 13 -> 19
Other:
- note added: "Si3865BDV"
- note removed: "Slew Rate set to 660uS"
Changed lines of the file:
@@
-EESchema Schematic File Version 2  date 9/18/2011 8:03:49 PM
+EESchema Schematic File Version 2  date 9/19/2011 7:25:32 AM
 LIBS:power
 LIBS:device
@@
 Comment4 "www.MicropendousX.org"
 $EndDescr
+Wire Wire Line
+	5250 6900 5250 6050
+Connection ~ 4950 6050
+Wire Wire Line
+	5250 6050 4950 6050
+Connection ~ 5050 6300
+Wire Wire Line
+	5050 6750 5050 6300
+Wire Wire Line
+	5050 6750 4850 6750
+Wire Wire Line
+	4500 6550 4500 6500
+Wire Wire Line
+	4500 6750 4500 6800
+Wire Wire Line
+	4000 6450 4050 6450
+Wire Wire Line
+	4050 6450 4050 6300
+Wire Wire Line
+	3850 5950 3850 6000
+Wire Wire Line
+	3850 6200 3850 6250
+Wire Wire Line
+	3850 6000 4050 6000
+Connection ~ 3850 6000
+Wire Wire Line
+	5050 6300 4950 6300
+Wire Wire Line
+	4850 6500 4850 6550
+Wire Wire Line
+	4950 6000 4950 6100
+Wire Wire Line
+	5050 6100 5050 6050
+Connection ~ 5050 6050
+Connection ~ 6800 7050
+Connection ~ 5050 6900
+Wire Wire Line
+	4850 7100 5250 7100
+Connection ~ 5050 7100
+Connection ~ 5250 6900
+Wire Wire Line
+	5050 7150 5050 7100
+Wire Wire Line
+	4850 6900 6100 6900
+Wire Wire Line
+	6800 7000 6800 7350
+Connection ~ 6800 7100
 Text Notes 5300 6800 0    30   ~ 0
 From Sheet 2 -\nOpennect Connector
 Text Notes 10050 1950 1    40   ~ 0
 Used in Sheet 2 -\nOpennect Connector
-Connection ~ 6800 7100
-Wire Wire Line
-	6800 7350 6800 7000
-Wire Wire Line
-	4750 5950 4750 6100
-Wire Wire Line
-	4350 6100 4450 6100
-Wire Wire Line
-	3300 6100 3450 6100
-Wire Wire Line
-	6100 6900 4850 6900
-Wire Wire Line
-	5050 7150 5050 7100
-Connection ~ 5250 6900
-Connection ~ 5050 7100
-Wire Wire Line
-	5250 7100 4850 7100
-Connection ~ 5050 6900
-Wire Wire Line
-	3900 6600 3900 6650
-Wire Wire Line
-	3300 5950 3450 5950
-Wire Wire Line
-	4350 5950 4450 5950
-Wire Wire Line
-	4350 6350 4450 6350
-Wire Wire Line
-	4750 6025 5250 6025
-Wire Wire Line
-	5250 6025 5250 6900
-Connection ~ 4750 6025
-Connection ~ 6800 7050
-Text Notes 4250 6450 0    40   ~ 0
-Slew Rate set to 660uS
-$Comp
-L VDDIO_3V3 #PWR037
-U 1 1 4E753477
-P 4450 6350
-F 0 "#PWR037" H 4450 6450 30  0001 C CNN
-F 1 "VDDIO_3V3" V 4450 6550 30  0000 C CNN
-	1    4450 6350
-	0    1    1    0
-$EndComp
-Text GLabel 3450 6350 0    40   BiDi ~ 0
-GPIO3_4
-Text GLabel 3450 6250 0    40   BiDi ~ 0
+Text GLabel 4000 6450 0    40   BiDi ~ 0
 GPIO3_3
-$Comp
-L VDD1V8 #PWR038
-U 1 1 4E753410
-P 3300 6100
-F 0 "#PWR038" H 3300 6200 30  0001 C CNN
-F 1 "VDD1V8" H 3300 6200 30  0000 C CNN
-	1    3300 6100
-	1    0    0    -1
-$EndComp
-$Comp
-L VDDIO_3V3 #PWR039
-U 1 1 4E7533F9
-P 3300 5950
-F 0 "#PWR039" H 3300 6050 30  0001 C CNN
-F 1 "VDDIO_3V3" H 3300 6050 30  0000 C CNN
-	1    3300 5950
-	1    0    0    -1
-$EndComp
-$Comp
-L D_SCHOTTKY D3
-U 1 1 4E7533C9
-P 4600 6100
-F 0 "D3" H 4700 6000 35  0000 C CNN
-F 1 "MBR120" H 4550 6000 30  0000 C CNN
-	1    4600 6100
-	1    0    0    -1
-$EndComp
-$Comp
-L D_SCHOTTKY D2
-U 1 1 4E7533AE
-P 4600 5950
-F 0 "D2" H 4700 6050 35  0000 C CNN
-F 1 "MBR120" H 4550 6050 30  0000 C CNN
-	1    4600 5950
-	1    0    0    -1
-$EndComp
-$Comp
-L TPS22960 IC5
-U 1 1 4E75339A
-P 3900 6150
-F 0 "IC5" H 3700 5800 60  0000 C CNN
-F 1 "TPS22960" H 3900 6500 60  0000 C CNN
-	1    3900 6150
-	1    0    0    -1
-$EndComp
 Text GLabel 8950 2050 1    40   BiDi ~ 0
 GPIO3_3
@@
 GPIO5_1-EMC_A12
 Text GLabel 3500 2050 1    40   BiDi ~ 0
-GPIO5_0-EMC_A13-ENET_MDC
+GPIO5_0-EMC_A13
 Text GLabel 3300 2050 1    40   BiDi ~ 0
 GPIO5_2
@@
 Text GLabel 9900 2050 1    40   BiDi ~ 0
 CLKOUT-I2S1_RX_SCK
-Text GLabel 9050 2050 1    40   BiDi ~ 0
-GPIO3_4
+Text GLabel 9050 1950 1    40   BiDi ~ 0
+~EMC_RAS~
 Text GLabel 7900 2050 1    40   BiDi ~ 0
 ~EMC_WE~-MMC_CMD
@@
 ~EMC_OE~
 Text GLabel 8100 2050 1    40   BiDi ~ 0
-~EMC_CS0~-MMC_POW
+~EMC_CS0~
 Text GLabel 5250 2050 1    40   BiDi ~ 0
 EMC_D06-MMC_CD
@@
 MMC_VDD
 $Comp
-L GND #PWR040
+L GND #PWR037
 U 1 1 4E23313A
 P 5050 7150
-F 0 "#PWR040" H 5050 7150 30  0001 C CNN
+F 0 "#PWR037" H 5050 7150 30  0001 C CNN
 F 1 "GND" H 5050 7080 30  0001 C CNN
 	1    5050 7150
@@
 $EndComp
 $Comp
-L GND #PWR041
-U 1 1 4E232F75
-P 3900 6650
-F 0 "#PWR041" H 3900 6650 30  0001 C CNN
-F 1 "GND" H 3900 6580 30  0001 C CNN
-	1    3900 6650
-	1    0    0    -1
-$EndComp
-$Comp
 L C_MINI C119
 U 1 1 4E232F74
@@
 $EndComp
 $Comp
-L GND #PWR042
+L GND #PWR038
 U 1 1 4E232CE9
 P 6800 7350
-F 0 "#PWR042" H 6800 7350 30  0001 C CNN
+F 0 "#PWR038" H 6800 7350 30  0001 C CNN
 F 1 "GND" H 6800 7280 30  0001 C CNN
 	1    6800 7350
@@
 	1    0    0    -1
 $EndComp
+Text Label 4950 6300 1    25   ~ 0
+R1-C1
+Text Label 4500 6500 0    30   ~ 0
+R2
+$Comp
+L VDDIO_3V3 #PWR039
+U 1 1 4E23302F
+P 4850 6500
+F 0 "#PWR039" H 4850 6600 30  0001 C CNN
+F 1 "VDDIO_3V3" H 4850 6600 30  0000 C CNN
+	1    4850 6500
+	1    0    0    -1
+$EndComp
+$Comp
+L C_MINI C117
+U 1 1 4E233026
+P 5050 6200
+F 0 "C117" V 5000 6275 30  0000 C CNN
+F 1 "470p" V 5100 6250 25  0000 C CNN
+	1    5050 6200
+	0    1    1    0
+$EndComp
+$Comp
+L GND #PWR040
+U 1 1 4E232F75
+P 4500 6800
+F 0 "#PWR040" H 4500 6800 30  0001 C CNN
+F 1 "GND" H 4500 6730 30  0001 C CNN
+	1    4500 6800
+	1    0    0    -1
+$EndComp
+$Comp
+L GND #PWR041
+U 1 1 4E232F44
+P 3850 6250
+F 0 "#PWR041" H 3850 6250 30  0001 C CNN
+F 1 "GND" H 3850 6180 30  0001 C CNN
+	1    3850 6250
+	1    0    0    -1
+$EndComp
+$Comp
+L C_MINI C116
+U 1 1 4E232F43
+P 3850 6100
+F 0 "C116" V 3800 6175 30  0000 C CNN
+F 1 "0u1" V 3900 6150 25  0000 C CNN
+	1    3850 6100
+	0    1    1    0
+$EndComp
+$Comp
+L VDDIO_3V3 #PWR042
+U 1 1 4E232F42
+P 3850 5950
+F 0 "#PWR042" H 3850 6050 30  0001 C CNN
+F 1 "VDDIO_3V3" H 3850 6050 30  0000 C CNN
+	1    3850 5950
+	1    0    0    -1
+$EndComp
+$Comp
+L R_MINI R52
+U 1 1 4E232ED0
+P 4500 6650
+F 0 "R52" V 4475 6700 25  0000 C CNN
+F 1 "10k" V 4525 6700 20  0000 C CNN
+	1    4500 6650
+	0    1    1    0
+$EndComp
+$Comp
+L R_MINI R51
+U 1 1 4E232E52
+P 4850 6650
+F 0 "R51" V 4825 6700 25  0000 C CNN
+F 1 "199k" V 4875 6700 20  0000 C CNN
+	1    4850 6650
+	0    1    1    0
+$EndComp
+Text Notes 4250 5850 0    60   ~ 0
+Si3865BDV
+$Comp
+L LOAD_SWITCH IC5
+U 1 1 4E232D75
+P 4500 6200
+F 0 "IC5" H 4300 6000 60  0000 C CNN
+F 1 "FDC6331" H 4500 6500 60  0000 C CNN
+	1    4500 6200
+	1    0    0    -1
+$EndComp

Commit message: Updated LPC183x Hardware Design
Other:
- note added: "SC70-6 Load Switches:\nSi1865DL, Si1869DH, FDG6342L"
Changed lines of the file:
@@
-EESchema Schematic File Version 2  date 9/19/2011 7:25:32 AM
+EESchema Schematic File Version 2  date 9/23/2011 8:04:30 AM
 LIBS:power
 LIBS:device
@@
 Sheet 3 7
 Title "MicropendousX-LPC183x"
-Date "19 sep 2011"
+Date "23 sep 2011"
 Rev "1.0"
 Comp "Opendous Inc."
@@
 Comment4 "www.MicropendousX.org"
 $EndDescr
+Text Notes 4100 7550 0    40   ~ 0
+SC70-6 Load Switches:\nSi1865DL, Si1869DH, FDG6342L
 Wire Wire Line
 	5250 6900 5250 6050
@@
 MMC_VDD
 $Comp
-L GND #PWR037
+L GND #PWR040
 U 1 1 4E23313A
 P 5050 7150
-F 0 "#PWR037" H 5050 7150 30  0001 C CNN
+F 0 "#PWR040" H 5050 7150 30  0001 C CNN
 F 1 "GND" H 5050 7080 30  0001 C CNN
 	1    5050 7150
@@
 $EndComp
 $Comp
-L GND #PWR038
+L GND #PWR041
 U 1 1 4E232CE9
 P 6800 7350
-F 0 "#PWR038" H 6800 7350 30  0001 C CNN
+F 0 "#PWR041" H 6800 7350 30  0001 C CNN
 F 1 "GND" H 6800 7280 30  0001 C CNN
 	1    6800 7350
@@
 R2
 $Comp
-L VDDIO_3V3 #PWR039
+L VDDIO_3V3 #PWR042
 U 1 1 4E23302F
 P 4850 6500
-F 0 "#PWR039" H 4850 6600 30  0001 C CNN
+F 0 "#PWR042" H 4850 6600 30  0001 C CNN
 F 1 "VDDIO_3V3" H 4850 6600 30  0000 C CNN
 	1    4850 6500
@@
 $EndComp
 $Comp
-L GND #PWR040
+L GND #PWR043
 U 1 1 4E232F75
 P 4500 6800
-F 0 "#PWR040" H 4500 6800 30  0001 C CNN
+F 0 "#PWR043" H 4500 6800 30  0001 C CNN
 F 1 "GND" H 4500 6730 30  0001 C CNN
 	1    4500 6800
@@
 $EndComp
 $Comp
-L GND #PWR041
+L GND #PWR044
 U 1 1 4E232F44
 P 3850 6250
-F 0 "#PWR041" H 3850 6250 30  0001 C CNN
+F 0 "#PWR044" H 3850 6250 30  0001 C CNN
 F 1 "GND" H 3850 6180 30  0001 C CNN
 	1    3850 6250
@@
 $EndComp
 $Comp
-L VDDIO_3V3 #PWR042
+L VDDIO_3V3 #PWR045
 U 1 1 4E232F42
 P 3850 5950
-F 0 "#PWR042" H 3850 6050 30  0001 C CNN
+F 0 "#PWR045" H 3850 6050 30  0001 C CNN
 F 1 "VDDIO_3V3" H 3850 6050 30  0000 C CNN
 	1    3850 5950

Commit message: Updated LPC183x Hardware Design
Changed lines of the file:
@@
-EESchema Schematic File Version 2  date 9/23/2011 8:04:30 AM
+EESchema Schematic File Version 2  date 9/24/2011 9:18:58 PM
 LIBS:power
 LIBS:device
@@
 Sheet 3 7
 Title "MicropendousX-LPC183x"
-Date "23 sep 2011"
+Date "25 sep 2011"
 Rev "1.0"
 Comp "Opendous Inc."
@@
 Comment4 "www.MicropendousX.org"
 $EndDescr
+Text GLabel 6650 7700 2    40   BiDi ~ 0
+MMC_VDD
+Text Label 6100 6900 2    30   ~ 0
+MMC_VDD
 Text Notes 4100 7550 0    40   ~ 0
 SC70-6 Load Switches:\nSi1865DL, Si1869DH, FDG6342L
@@
 Text GLabel 4650 2050 1    40   BiDi ~ 0
 EMC_D00
-Text Label 6100 6900 2    30   ~ 0
+Text Label 6650 7700 2    30   ~ 0
 MMC_VDD
 $Comp
-L GND #PWR040
+L GND #PWR041
 U 1 1 4E23313A
 P 5050 7150
-F 0 "#PWR040" H 5050 7150 30  0001 C CNN
+F 0 "#PWR041" H 5050 7150 30  0001 C CNN
 F 1 "GND" H 5050 7080 30  0001 C CNN
 	1    5050 7150
@@
 $EndComp
 $Comp
-L GND #PWR041
+L GND #PWR042
 U 1 1 4E232CE9
 P 6800 7350
-F 0 "#PWR041" H 6800 7350 30  0001 C CNN
+F 0 "#PWR042" H 6800 7350 30  0001 C CNN
 F 1 "GND" H 6800 7280 30  0001 C CNN
 	1    6800 7350
@@
 R2
 $Comp
-L VDDIO_3V3 #PWR042
+L VDDIO_3V3 #PWR043
 U 1 1 4E23302F
 P 4850 6500
-F 0 "#PWR042" H 4850 6600 30  0001 C CNN
+F 0 "#PWR043" H 4850 6600 30  0001 C CNN
 F 1 "VDDIO_3V3" H 4850 6600 30  0000 C CNN
 	1    4850 6500
@@
 $EndComp
 $Comp
-L GND #PWR043
+L GND #PWR044
 U 1 1 4E232F75
 P 4500 6800
-F 0 "#PWR043" H 4500 6800 30  0001 C CNN
+F 0 "#PWR044" H 4500 6800 30  0001 C CNN
 F 1 "GND" H 4500 6730 30  0001 C CNN
 	1    4500 6800
@@
 $EndComp
 $Comp
-L GND #PWR044
+L GND #PWR045
 U 1 1 4E232F44
 P 3850 6250
-F 0 "#PWR044" H 3850 6250 30  0001 C CNN
+F 0 "#PWR045" H 3850 6250 30  0001 C CNN
 F 1 "GND" H 3850 6180 30  0001 C CNN
 	1    3850 6250
@@
 $EndComp
 $Comp
-L VDDIO_3V3 #PWR045
+L VDDIO_3V3 #PWR046
 U 1 1 4E232F42
 P 3850 5950
-F 0 "#PWR045" H 3850 6050 30  0001 C CNN
+F 0 "#PWR046" H 3850 6050 30  0001 C CNN
 F 1 "VDDIO_3V3" H 3850 6050 30  0000 C CNN
 	1    3850 5950

Commit message: Updated LPC183x Hardware Design
Connections:
- net labels added: VDD3V3
- net labels removed: VDDIO_3V3
Changed lines of the file:
@@
-EESchema Schematic File Version 2  date 9/24/2011 9:18:58 PM
+EESchema Schematic File Version 2  date 9/25/2011 2:41:21 AM
 LIBS:power
 LIBS:device
@@
 Comment4 "www.MicropendousX.org"
 $EndDescr
+$Comp
+L VDD3V3 #PWR041
+U 1 1 4E7EA660
+P 4850 6500
+F 0 "#PWR041" H 4850 6600 30  0001 C CNN
+F 1 "VDD3V3" H 4850 6600 30  0000 C CNN
+	1    4850 6500
+	1    0    0    -1
+$EndComp
+$Comp
+L VDD3V3 #PWR042
+U 1 1 4E7EA63F
+P 3850 5950
+F 0 "#PWR042" H 3850 6050 30  0001 C CNN
+F 1 "VDD3V3" H 3850 6050 30  0000 C CNN
+	1    3850 5950
+	1    0    0    -1
+$EndComp
 Text GLabel 6650 7700 2    40   BiDi ~ 0
 MMC_VDD
@@
 MMC_VDD
 $Comp
-L GND #PWR041
+L GND #PWR043
 U 1 1 4E23313A
 P 5050 7150
-F 0 "#PWR041" H 5050 7150 30  0001 C CNN
+F 0 "#PWR043" H 5050 7150 30  0001 C CNN
 F 1 "GND" H 5050 7080 30  0001 C CNN
 	1    5050 7150
@@
 $EndComp
 $Comp
-L GND #PWR042
+L GND #PWR044
 U 1 1 4E232CE9
 P 6800 7350
-F 0 "#PWR042" H 6800 7350 30  0001 C CNN
+F 0 "#PWR044" H 6800 7350 30  0001 C CNN
 F 1 "GND" H 6800 7280 30  0001 C CNN
 	1    6800 7350
@@
 R2
 $Comp
-L VDDIO_3V3 #PWR043
-U 1 1 4E23302F
-P 4850 6500
-F 0 "#PWR043" H 4850 6600 30  0001 C CNN
-F 1 "VDDIO_3V3" H 4850 6600 30  0000 C CNN
-	1    4850 6500
-	1    0    0    -1
-$EndComp
-$Comp
 L C_MINI C117
 U 1 1 4E233026
@@
 $EndComp
 $Comp
-L GND #PWR044
+L GND #PWR045
 U 1 1 4E232F75
 P 4500 6800
-F 0 "#PWR044" H 4500 6800 30  0001 C CNN
+F 0 "#PWR045" H 4500 6800 30  0001 C CNN
 F 1 "GND" H 4500 6730 30  0001 C CNN
 	1    4500 6800
@@
 $EndComp
 $Comp
-L GND #PWR045
+L GND #PWR046
 U 1 1 4E232F44
 P 3850 6250
-F 0 "#PWR045" H 3850 6250 30  0001 C CNN
+F 0 "#PWR046" H 3850 6250 30  0001 C CNN
 F 1 "GND" H 3850 6180 30  0001 C CNN
 	1    3850 6250
@@
 $EndComp
 $Comp
-L VDDIO_3V3 #PWR046
-U 1 1 4E232F42
-P 3850 5950
-F 0 "#PWR046" H 3850 6050 30  0001 C CNN
-F 1 "VDDIO_3V3" H 3850 6050 30  0000 C CNN
-	1    3850 5950
-	1    0    0    -1
-$EndComp
-$Comp
