File: MicropendousX/Hardware/MicropendousX-LPC183x/MicropendousX-LPC183x-Power.sch (KiCad schematic (older format))
At the start: 43 parts, among them IC1 LPC183X, IC2 XC6222

Commit message: Update unfinished LPC183x-based design.
Parts:
- removed IC2: XC6222, symbol REGULATOR_SOT89-5_TOREX
- added BT1: Li-Ion, symbol BATTERY_LI-ION
- added D2: CHRG, symbol D_LED
- added IC6: LTC3559, symbol LTC3559
- added L5, L6: 4.7uH, symbol L_MINI
- added R12, R15: 1k, symbol R_MINI
- added R13: 10k, symbol R_MINI
- added R14: 1k74, symbol R_MINI
- added R16, R18: 806k, symbol R_MINI
- added R17: 324k, symbol R_MINI
- added R19: 649k, symbol R_MINI
- C26: value 0u1 -> 2u2
- C30: value 33n -> 22p
- C32: value 0u1 -> 22p
- C54: value 33n -> 10u
- C55: value 0u1 -> 10u
Connections:
- net labels added: +BATT, VDD1V8
- wire segments 123 -> 152
Other:
- note added: "1.8V"
- note added: "2.8V"
- note added: "This rail is 3.3V nominally but\nset to 2.8V to conserve power."
- moved on the sheet: C13, C14, C23, C26, C30, C31, C32, C33, C54, C55, C6, C7

Commit message: Updated LPC183x Hardware Design
Parts:
- removed C23, C33, C52: 33n, symbol C_MINI
- removed C31, C43, C44, C53, C7: 0u1, symbol C_MINI
- removed C38, C40: 4u7, symbol C_MINI
- removed R24, R25: 1, symbol R_MINI
- added C10: u22, symbol C_MINI
- added C11: 4u7, symbol CP_TANTALUM_MINI
- added C9: 1u0, symbol C_MINI
- added IC2: STC3100, symbol STC3100
- added R3: 0R03, symbol R_MINI
- added R4: 1k, symbol R_MINI
- added R6: 200k, symbol R_MINI
- added R9: 10k, symbol R_MINI
- added TP6: IO0, symbol CONN_1
- C51: value n1 -> 1u0
- C6: value 10u -> 0u1
- R17: value 324k -> 259k
- R19: value 649k -> 499k
- renumbered D2 to D1
Connections:
- net labels added: GPIO3_7, I2C1_SCL-U3_RXD, I2C1_SDA-U3_TXD, IO0
- wire segments 152 -> 140
Other:
- note added: "0.1%"
- note added: "0.2<ESR(Ohm)<1"
- note added: "0805"
- note added: "1206"
- note added: "2.1V"
- note added: "From Sheet 2 -\nOpennect Connector"
- note added: "Li-Ion Charger, Guage, and Dual Buck Regulators"
- note added: "Pin is nominally 1.8V but set to 2.1V\nto account for MMC diode drop.\nSee Sheet 1 - EMI."
- note added: "Power Management"
- note added: "R14 = 1.74k limits USB\ncharge current to 500mA"
- note added: "USB VBUS Fuse F1\nlimits inrush current"
- note removed: "1.8V"
- note removed: "2.8V"
- note removed: "This rail is 3.3V nominally but\nset to 2.8V to conserve power."
- moved on the sheet: BT1, C107, C109, C112, C113, C114, C13, C14, C17, C24, C26, C27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

Commit message: Updated LPC183x Hardware Design
Parts:
- added D5: RECTIFIER, symbol D_RECTIFIER
- added Q1: MOSFET, symbol MOSFET_N_OPENDOUS
- added Q2: FDN304, symbol MOSFET_P_OPENDOUS
- added R10: 1k2, symbol R_MINI
- added R11: 1k65, symbol R_MINI
- added R20: 10k, symbol R_MINI
Connections:
- net labels added: 6V0, GPIO5_2, LTC3559_HPWR, LTC3559_PROG, LTC3559_SUSP, LTC3559_VCC, LTC3559_~CHRG~
- wire segments 140 -> 155
Other:
- note added: "DC Power Jack Support"
- note added: "From Sheet\n1 - EMI"
- note added: "Use Rectifier with >500mOhm Vdrop for D1\nas LTC3559 has maximum Vcc of 5.5V"
- note removed: "USB VBUS Fuse F1\nlimits inrush current"
- moved on the sheet: BT1, C10, C13, C14, C26, C30, C32, C54, C55, C9, D1, IC2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

Commit message: Updated LPC183x Hardware Design
Parts:
- removed C11: 4u7, symbol CP_TANTALUM_MINI
- added C11: 4u7, symbol C_MINI
- added R21: 0R5, symbol R_MINI
- C37: value n1 -> 1n0
- L2: value FB -> DNI
- Q1: value MOSFET -> Si2312
- R19: value 499k -> 259k
- renumbered BT1 to BAT1
Connections:
- net labels added: LTC3559_NTC
- net labels removed: VBAT, VDD1V8
- wire segments 155 -> 159
Other:
- note added: "DNI"
- note removed: "0.2<ESR(Ohm)<1"
- note removed: "2.1V"
- note removed: "Pin is nominally 1.8V but set to 2.1V\nto account for MMC diode drop.\nSee Sheet 1 - EMI."
- moved on the sheet: C26

Commit message: Updated LPC183x Hardware Design
Parts:
- removed C6: 0u1, symbol C_MINI
- added C18: 1u0, symbol C_MINI
- added C19: 0u1, symbol C_MINI
- D5: value RECTIFIER -> PMEG3030
Connections:
- wire segments 159 -> 157
Other:
- note added: "RSX501L-20\nPMEG3030EP\nCMS01"
- moved on the sheet: C17, C24

Commit message: Updated LPC183x Hardware Design
Parts:
- D5: value PMEG3030 -> CGRM4004
Connections:
- wire segments 157 -> 156
Other:
- note removed: "RSX501L-20\nPMEG3030EP\nCMS01"

Commit message: Updated LPC183x Hardware Design
Parts:
- C107: value 0u1 -> u01
- TP6: value IO0 -> STC_IO0
Changed lines of the file:
@@
-EESchema Schematic File Version 2  date 9/24/2011 9:18:58 PM
+EESchema Schematic File Version 2  date 9/25/2011 2:41:21 AM
 LIBS:power
 LIBS:device
@@
 P 5450 1400
 F 0 "TP6" H 5500 1400 40  0000 L CNN
-F 1 "IO0" H 5450 1455 30  0001 C CNN
+F 1 "STC_IO0" H 5450 1455 30  0001 C CNN
 	1    5450 1400
 	-1   0    0    1
@@
 P 5450 5750
 F 0 "C107" V 5400 5825 30  0000 C CNN
-F 1 "0u1" V 5500 5800 25  0000 C CNN
+F 1 "u01" V 5500 5800 25  0000 C CNN
 	1    5450 5750
 	0    1    1    0

Commit message: Updated LPC183x Hardware Design
Parts:
- added C21: 33n, symbol C_MINI
Other:
- moved on the sheet: C17, C18, C19, C24, C50
Changed lines of the file:
@@
-EESchema Schematic File Version 2  date 9/25/2011 2:41:21 AM
+EESchema Schematic File Version 2  date 9/25/2011 4:24:57 AM
 LIBS:power
 LIBS:device
@@
 Comment4 "www.MicropendousX.org"
 $EndDescr
-Text GLabel 6450 7600 2    40   Input ~ 0
-LTC3559_VCC
-Text Label 6450 7600 2    30   ~ 0
-LTC3559_VCC
-Text Label 3150 2050 2    30   ~ 0
-LTC3559_VCC
+Connection ~ 5100 4250
+Wire Wire Line
+	5300 4250 4300 4250
 Connection ~ 2750 1700
 Wire Wire Line
 	2950 1700 2350 1700
-Connection ~ 4650 4250
-Wire Wire Line
-	5250 4250 4450 4250
-Connection ~ 5050 4050
+Connection ~ 4500 4250
+Connection ~ 4900 4050
 Wire Wire Line
 	3150 950  3150 1900
@@
 	3150 2350 2250 2350
 Wire Wire Line
-	4850 4050 4850 4000
+	4700 4050 4700 4000
 Connection ~ 4450 5650
 Wire Wire Line
@@
 Connection ~ 5250 5850
 Connection ~ 4650 5850
-Connection ~ 4850 4250
+Connection ~ 4700 4250
 Connection ~ 5050 5850
 Connection ~ 4850 5650
@@
 	6050 6700 6050 6650
 Wire Wire Line
-	4850 4300 4850 4250
+	4700 4300 4700 4250
 Connection ~ 2450 1900
 Wire Wire Line
@@
 	5450 5850 4250 5850
 Connection ~ 4450 5850
-Connection ~ 4850 4050
+Connection ~ 4700 4050
 Wire Wire Line
 	5700 1550 5650 1550
@@
 	3100 1300 3150 1300
 Connection ~ 3150 1300
-Connection ~ 5050 4250
-Wire Wire Line
-	5250 4050 4450 4050
-Connection ~ 4650 4050
+Connection ~ 4900 4250
+Connection ~ 4500 4050
+Wire Wire Line
+	5300 4050 4300 4050
+Connection ~ 5100 4050
+$Comp
+L C_MINI C21
+U 1 1 4E7EE540
+P 5300 4150
+F 0 "C21" V 5250 4200 30  0000 C CNN
+F 1 "33n" V 5350 4200 25  0000 C CNN
+	1    5300 4150
+	0    1    1    0
+$EndComp
+Text GLabel 6450 7600 2    40   Input ~ 0
+LTC3559_VCC
+Text Label 6450 7600 2    30   ~ 0
+LTC3559_VCC
+Text Label 3150 2050 2    30   ~ 0
+LTC3559_VCC
 $Comp
 L C_MINI C19
 U 1 1 4E7C660E
-P 5050 4150
-F 0 "C19" V 5000 4200 30  0000 C CNN
-F 1 "0u1" V 5100 4200 25  0000 C CNN
-	1    5050 4150
+P 4900 4150
+F 0 "C19" V 4850 4200 30  0000 C CNN
+F 1 "0u1" V 4950 4200 25  0000 C CNN
+	1    4900 4150
 	0    1    1    0
 $EndComp
@@
 L C_MINI C18
 U 1 1 4E7C6609
-P 4650 4150
-F 0 "C18" V 4600 4200 30  0000 C CNN
-F 1 "1u0" V 4700 4200 25  0000 C CNN
-	1    4650 4150
+P 4500 4150
+F 0 "C18" V 4450 4200 30  0000 C CNN
+F 1 "1u0" V 4550 4200 25  0000 C CNN
+	1    4500 4150
 	0    1    1    0
 $EndComp
@@
 L VDD3V3 #PWR0104
 U 1 1 4E495263
-P 4850 4000
-F 0 "#PWR0104" H 4850 4100 30  0001 C CNN
-F 1 "VDD3V3" H 4850 4100 30  0000 C CNN
-	1    4850 4000
+P 4700 4000
+F 0 "#PWR0104" H 4700 4100 30  0001 C CNN
+F 1 "VDD3V3" H 4700 4100 30  0000 C CNN
+	1    4700 4000
 	1    0    0    -1
 $EndComp
@@
 L C_MINI C50
 U 1 1 4DE9D212
-P 5250 4150
-F 0 "C50" V 5200 4200 30  0000 C CNN
-F 1 "33n" V 5300 4200 25  0000 C CNN
-	1    5250 4150
+P 5100 4150
+F 0 "C50" V 5050 4200 30  0000 C CNN
+F 1 "33n" V 5150 4200 25  0000 C CNN
+	1    5100 4150
 	0    1    1    0
 $EndComp
@@
 L GND #PWR0133
 U 1 1 4DE9D210
-P 4850 4300
-F 0 "#PWR0133" H 4850 4300 30  0001 C CNN
-F 1 "GND" H 4850 4230 30  0001 C CNN
-	1    4850 4300
+P 4700 4300
+F 0 "#PWR0133" H 4700 4300 30  0001 C CNN
+F 1 "GND" H 4700 4230 30  0001 C CNN
+	1    4700 4300
 	1    0    0    -1
 $EndComp
@@
 L C_MINI C17
 U 1 1 4DE9D20F
-P 4850 4150
-F 0 "C17" V 4800 4200 30  0000 C CNN
-F 1 "4u7" V 4900 4200 25  0000 C CNN
-	1    4850 4150
+P 4700 4150
+F 0 "C17" V 4650 4200 30  0000 C CNN
+F 1 "4u7" V 4750 4200 25  0000 C CNN
+	1    4700 4150
 	0    1    1    0
 $EndComp
@@
 L C_MINI C24
 U 1 1 4DE1FF8D
-P 4450 4150
-F 0 "C24" V 4400 4200 30  0000 C CNN
-F 1 "10u" V 4500 4200 25  0000 C CNN
-	1    4450 4150
-	0    1    1    0
-$EndComp
+P 4300 4150
+F 0 "C24" V 4250 4200 30  0000 C CNN
+F 1 "10u" V 4350 4200 25  0000 C CNN
+	1    4300 4150
+	0    1    1    0
+$EndComp
