File: MicropendousX/Hardware/MicropendousX-LPC183x/MicropendousX-LPC183x-Power.sch (KiCad schematic (older format))
At the start: 61 parts, among them IC1 LPC183X, IC2 STC3100, IC6 LTC3559, Q1 Si2312, Q2 FDN304

Commit message: Updated LPC183x Hardware Design
Parts:
- D5: value CGRM4004 -> PMEG3020EH
Connections:
- wire segments 156 -> 158
Other:
- note added: "From Sheet 1 - EMI"
- note added: "Use Rectifier with >500mOhm Vdrop for D1\nas LTC3559 has maximum Vcc of 5.5V.\nPMEG3020EH, SMD26PL, MBRX160"
- note removed: "From Sheet\n1 - EMI"
- note removed: "Use Rectifier with >500mOhm Vdrop for D1\nas LTC3559 has maximum Vcc of 5.5V"
- moved on the sheet: BAT1, C10, C11, C13, C14, C26, C30, C32, C54, C55, C9, D1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

Commit message: Updated LPC183x Hardware Design
Parts:
- added C22: u01, symbol C_MINI
Changed lines of the file:
@@
-EESchema Schematic File Version 2  date 9/25/2011 6:49:29 PM
+EESchema Schematic File Version 2  date 9/25/2011 11:28:51 PM
 LIBS:power
 LIBS:device
@@
 Sheet 6 7
 Title "MicropendousX-LPC183x"
-Date "25 sep 2011"
+Date "26 sep 2011"
 Rev "1.0"
 Comp "Opendous Inc."
@@
 Comment4 "www.MicropendousX.org"
 $EndDescr
-$Comp
-L VDDIO_3V3 #PWR078
-U 1 1 4E7F4AB8
-P 2600 3150
-F 0 "#PWR078" H 2600 3250 30  0001 C CNN
-F 1 "VDDIO_3V3" H 2600 3250 30  0000 C CNN
-	1    2600 3150
-	1    0    0    -1
-$EndComp
+Connection ~ 5450 5850
+Wire Wire Line
+	5650 5850 4250 5850
 Wire Wire Line
 	2600 3250 2750 3250
@@
 	4700 4050 4700 4000
 Connection ~ 4450 5650
-Wire Wire Line
-	4250 5650 5450 5650
 Connection ~ 4050 2050
 Wire Wire Line
@@
 Wire Wire Line
 	2750 3000 2750 2800
-Wire Wire Line
-	4250 5850 5450 5850
 Connection ~ 4450 5850
 Connection ~ 4700 4050
@@
 Wire Wire Line
 	3150 2600 1600 2600
+Wire Wire Line
+	5650 5650 4250 5650
+Connection ~ 5450 5650
+$Comp
+L C_MINI C22
+U 1 1 4E7FE693
+P 5650 5750
+F 0 "C22" V 5600 5825 30  0000 C CNN
+F 1 "u01" V 5700 5800 25  0000 C CNN
+	1    5650 5750
+	0    1    1    0
+$EndComp
+$Comp
+L VDDIO_3V3 #PWR078
+U 1 1 4E7F4AB8
+P 2600 3150
+F 0 "#PWR078" H 2600 3250 30  0001 C CNN
+F 1 "VDDIO_3V3" H 2600 3250 30  0000 C CNN
+	1    2600 3150
+	1    0    0    -1
+$EndComp
 $Comp
 L C_MINI C21
