File: MicropendousX/Hardware/MicropendousX-LPC183x/MicropendousX-LPC183x-System.sch (KiCad schematic (older format))
At the start: 36 parts, among them IC1 LPC183X, IC7 25Q, SW1 RESET, SW2 NMI, U4 JTAG, X1 12MHz, X2 32.768kHz

Commit message: Update unfinished LPC183x-based design.
Parts:
- removed TP3: WAKEUP0, symbol CONN_1
- added C116, C119: 0u1, symbol C_MINI
- added C117: 470p, symbol C_MINI
- added C118: 10u, symbol C_MINI
- added C120: u01, symbol C_MINI
- added unit 3 of IC1
- added IC8: FDC6331L, symbol LOAD_SWITCH
- added R51: 200k, symbol R_MINI
- added R52: 10k, symbol R_MINI
- added R53: DNI, symbol R_MINI
- added U11: MMC, symbol CONN_MMC_AMPHENOL_101-00565
Connections:
- net labels added: MMC_CLK, MMC_CMD, MMC_DAT0, MMC_DAT1, MMC_DAT2, MMC_DAT3, MMC_DAT4, MMC_DAT5, MMC_DAT6, MMC_DAT7, MMC_POW, MMC_RST, MMC_VDD, MMC_VOLT1, MMC_WP, R1-C1, R2, ~MMC_CD~
- wire segments 75 -> 96
Other:
- note added: "Si3865BDV"

Commit message: Updated LPC183x Hardware Design
Parts:
- removed C116, C119: 0u1, symbol C_MINI
- removed C117: 470p, symbol C_MINI
- removed C118: 10u, symbol C_MINI
- removed C120: u01, symbol C_MINI
- removed unit 3 of IC1
- removed IC8: FDC6331L, symbol LOAD_SWITCH
- removed R38: 100, symbol R_MINI
- removed R51: 200k, symbol R_MINI
- removed R52: 10k, symbol R_MINI
- removed R53: DNI, symbol R_MINI
- removed SW2: NMI, symbol SWITCH_PUSHBUTTON
- removed U11: MMC, symbol CONN_MMC_AMPHENOL_101-00565
- added TP3: NMI, symbol CONN_1
- renumbered JP9 to JP0
Connections:
- net labels added: EMC_A00, SPIFI_SCK-CGU_OUT1, SPIFI_SIO2-I2S1_RX_WS, SPIFI_SIO3-I2S1_RX_SDA
- net labels removed: EMC_A09, MMC_CLK, MMC_CMD, MMC_DAT0, MMC_DAT1, MMC_DAT2, MMC_DAT3, MMC_DAT4, MMC_DAT5, MMC_DAT6, MMC_DAT7, MMC_POW, MMC_RST, MMC_VDD, MMC_VOLT1, MMC_WP, R1-C1, R2, SPIFI_SCK, SPIFI_SIO2, SPIFI_SIO3, ~MMC_CD~
- wire segments 96 -> 73
- no-connect marks 3 -> 4
Other:
- note added: "P2_9(A0)"
- note added: "Taken from 2011-08-22 LPC18x0 Datasheet - Table 5"
- note removed: "P2_7(A9)"
- note removed: "Si3865BDV"
- note removed: "Taken from 2011-07-13 LPC18x0 Datasheet - Table 5"
- moved on the sheet: C108, IC7

Commit message: Updated LPC183x Hardware Design
Parts:
- added TP7: WAKEUP0, symbol CONN_1
Connections:
- wire segments 73 -> 74
Changed lines of the file:
@@
-EESchema Schematic File Version 2  date 9/18/2011 3:49:57 PM
+EESchema Schematic File Version 2  date 9/18/2011 8:03:49 PM
 LIBS:power
 LIBS:device
@@
 Sheet 5 7
 Title "MicropendousX-LPC183x"
-Date "18 sep 2011"
+Date "19 sep 2011"
 Rev "1.0"
 Comp "Opendous Inc."
@@
 Comment4 "www.MicropendousX.org"
 $EndDescr
+Connection ~ 4000 3200
+Wire Wire Line
+	4000 3300 4000 3200
+Connection ~ 4950 1700
+Wire Wire Line
+	4950 1750 4950 1050
+Wire Wire Line
+	3650 2550 4000 2550
+Wire Wire Line
+	8000 3800 7900 3800
+Wire Wire Line
+	8300 3600 8300 3550
+Wire Wire Line
+	5100 1700 4950 1700
+Connection ~ 6350 900
+Wire Wire Line
+	6350 900  5550 900
+Wire Wire Line
+	6650 1000 6650 1150
+Wire Wire Line
+	6000 4200 6000 4150
+Wire Wire Line
+	5450 5050 5350 5050
+Wire Wire Line
+	5350 5050 5350 5150
+Wire Wire Line
+	4200 3050 4300 3050
+Wire Wire Line
+	4300 3050 4300 3000
+Wire Wire Line
+	4000 3050 3650 3050
+Connection ~ 4000 2350
+Wire Wire Line
+	3650 2350 4000 2350
+Wire Wire Line
+	4300 2300 4300 2350
+Wire Wire Line
+	4300 2350 4200 2350
+Connection ~ 5100 2900
+Wire Wire Line
+	5100 2900 5100 2600
+Wire Wire Line
+	5100 2600 5150 2600
+Connection ~ 5200 900
+Wire Wire Line
+	3650 900  5350 900
+Connection ~ 4100 1600
+Wire Wire Line
+	3650 1600 4300 1600
+Connection ~ 4100 1800
+Wire Wire Line
+	3650 1800 4300 1800
+Connection ~ 4550 1450
+Wire Wire Line
+	4650 1500 4650 1450
+Wire Wire Line
+	4250 1500 4250 1400
+Connection ~ 4950 2500
+Wire Wire Line
+	5150 2500 4950 2500
+Wire Wire Line
+	4950 2950 4950 2800
+Wire Wire Line
+	4950 2450 4950 2600
+Wire Wire Line
+	5150 2900 4950 2900
+Connection ~ 4950 2900
+Wire Wire Line
+	4500 1300 4550 1300
+Wire Wire Line
+	4550 1300 4550 1600
+Wire Wire Line
+	4550 1600 4500 1600
+Wire Wire Line
+	4650 1450 4250 1450
+Connection ~ 4250 1450
+Wire Wire Line
+	4550 1950 4650 1950
+Wire Wire Line
+	4500 2100 4550 2100
+Wire Wire Line
+	4550 2100 4550 1800
+Wire Wire Line
+	4550 1800 4500 1800
+Wire Wire Line
+	4650 1950 4650 2000
+Connection ~ 4550 1950
+Wire Wire Line
+	3650 2100 4300 2100
+Connection ~ 4100 2100
+Wire Wire Line
+	3650 1300 4300 1300
+Connection ~ 4100 1300
+Connection ~ 5650 900
+Wire Wire Line
+	5200 1100 5200 1150
+Wire Wire Line
+	5650 650  5650 700
+Wire Wire Line
+	5150 2700 5100 2700
+Connection ~ 5100 2700
+Wire Wire Line
+	4000 2350 4000 2450
+Wire Wire Line
+	4000 3500 3650 3500
+Wire Wire Line
+	6550 4750 6650 4750
+Wire Wire Line
+	6650 4750 6650 4650
+Wire Wire Line
+	6000 4400 6000 4450
+Wire Wire Line
+	6350 1000 6350 800
+Wire Wire Line
+	7900 4000 7900 4050
+Wire Wire Line
+	8200 3800 8300 3800
+Wire Wire Line
+	8000 3650 8100 3650
+Wire Wire Line
+	8100 3650 8100 3750
+Wire Wire Line
+	8900 3750 8900 3650
+Wire Wire Line
+	8900 3650 8800 3650
+Wire Wire Line
+	9000 3800 9100 3800
+Wire Wire Line
+	8700 4000 8700 4050
+Wire Wire Line
+	9100 3600 9100 3550
+Wire Wire Line
+	8800 3800 8700 3800
+Wire Wire Line
+	10400 3800 10300 3800
+Wire Wire Line
+	10700 3600 10700 3550
+Wire Wire Line
+	10300 4000 10300 4050
+Wire Wire Line
+	10600 3800 10700 3800
+Wire Wire Line
+	10400 3650 10500 3650
+Wire Wire Line
+	10500 3650 10500 3750
+Wire Wire Line
+	9700 3750 9700 3650
+Wire Wire Line
+	9700 3650 9600 3650
+Wire Wire Line
+	9800 3800 9900 3800
+Wire Wire Line
+	9500 4000 9500 4050
+Wire Wire Line
+	9900 3600 9900 3550
+Wire Wire Line
+	9600 3800 9500 3800
+Wire Wire Line
+	4950 1050 3650 1050
+Wire Wire Line
+	4950 2000 4950 1950
+Wire Wire Line
+	3850 3050 3850 3200
+Wire Wire Line
+	3850 3200 4050 3200
+Connection ~ 3850 3050
+$Comp
+L CONN_1 TP7
+U 1 1 4E7650C6
+P 4150 3300
+F 0 "TP7" H 4230 3300 40  0000 L CNN
+F 1 "WAKEUP0" H 4150 3355 30  0001 C CNN
+	1    4150 3300
+	1    0    0    -1
+$EndComp
 Text Notes 8700 5250 0    60   ~ 0
 LOW
@@
 $EndComp
 NoConn ~ 3650 3350
-Connection ~ 3850 3050
-Wire Wire Line
-	4050 3200 3850 3200
-Wire Wire Line
-	3850 3200 3850 3050
-Wire Wire Line
-	4950 2000 4950 1950
-Wire Wire Line
-	3650 1050 4950 1050
-Wire Wire Line
-	9600 3800 9500 3800
-Wire Wire Line
-	9900 3600 9900 3550
-Wire Wire Line
-	9500 4000 9500 4050
-Wire Wire Line
-	9800 3800 9900 3800
-Wire Wire Line
-	9600 3650 9700 3650
-Wire Wire Line
-	9700 3650 9700 3750
-Wire Wire Line
-	10500 3750 10500 3650
-Wire Wire Line
-	10500 3650 10400 3650
-Wire Wire Line
-	10600 3800 10700 3800
-Wire Wire Line
-	10300 4000 10300 4050
-Wire Wire Line
-	10700 3600 10700 3550
-Wire Wire Line
-	10400 3800 10300 3800
-Wire Wire Line
-	8800 3800 8700 3800
-Wire Wire Line
-	9100 3600 9100 3550
-Wire Wire Line
-	8700 4000 8700 4050
-Wire Wire Line
-	9000 3800 9100 3800
-Wire Wire Line
-	8800 3650 8900 3650
-Wire Wire Line
-	8900 3650 8900 3750
-Wire Wire Line
-	8100 3750 8100 3650
-Wire Wire Line
-	8100 3650 8000 3650
-Wire Wire Line
-	8200 3800 8300 3800
-Wire Wire Line
-	7900 4000 7900 4050
-Wire Wire Line
-	6350 1000 6350 800
-Wire Wire Line
-	6000 4400 6000 4450
-Wire Wire Line
-	6650 4650 6650 4750
-Wire Wire Line
-	6650 4750 6550 4750
-Wire Wire Line
-	4000 3500 3650 3500
-Wire Wire Line
-	4000 2450 4000 2350
-Connection ~ 5100 2700
-Wire Wire Line
-	5150 2700 5100 2700
-Wire Wire Line
-	5650 650  5650 700
-Wire Wire Line
-	5200 1100 5200 1150
-Connection ~ 5650 900
-Connection ~ 4100 1300
-Wire Wire Line
-	3650 1300 4300 1300
-Connection ~ 4100 2100
-Wire Wire Line
-	3650 2100 4300 2100
-Connection ~ 4550 1950
-Wire Wire Line
-	4650 2000 4650 1950
-Wire Wire Line
-	4500 1800 4550 1800
-Wire Wire Line
-	4550 1800 4550 2100
-Wire Wire Line
-	4550 2100 4500 2100
-Wire Wire Line
-	4650 1950 4550 1950
-Connection ~ 4250 1450
-Wire Wire Line
-	4250 1450 4650 1450
-Wire Wire Line
-	4500 1600 4550 1600
-Wire Wire Line
-	4550 1600 4550 1300
-Wire Wire Line
-	4550 1300 4500 1300
-Connection ~ 4950 2900
-Wire Wire Line
-	5150 2900 4950 2900
-Wire Wire Line
-	4950 2450 4950 2600
-Wire Wire Line
-	4950 2950 4950 2800
-Wire Wire Line
-	5150 2500 4950 2500
-Connection ~ 4950 2500
-Wire Wire Line
-	4250 1500 4250 1400
-Wire Wire Line
-	4650 1450 4650 1500
-Connection ~ 4550 1450
-Wire Wire Line
-	3650 1800 4300 1800
-Connection ~ 4100 1800
-Wire Wire Line
-	3650 1600 4300 1600
-Connection ~ 4100 1600
-Wire Wire Line
-	3650 900  5350 900
-Connection ~ 5200 900
-Wire Wire Line
-	5150 2600 5100 2600
-Wire Wire Line
-	5100 2600 5100 2900
-Connection ~ 5100 2900
-Wire Wire Line
-	4200 2350 4300 2350
-Wire Wire Line
-	4300 2350 4300 2300
-Wire Wire Line
-	4000 2350 3650 2350
-Connection ~ 4000 2350
-Wire Wire Line
-	4000 3050 3650 3050
-Wire Wire Line
-	4300 3000 4300 3050
-Wire Wire Line
-	4300 3050 4200 3050
-Wire Wire Line
-	5350 5150 5350 5050
-Wire Wire Line
-	5350 5050 5450 5050
-Wire Wire Line
-	6000 4200 6000 4150
-Wire Wire Line
-	6650 1000 6650 1150
-Wire Wire Line
-	6350 900  5550 900
-Connection ~ 6350 900
-Wire Wire Line
-	5100 1700 4950 1700
-Wire Wire Line
-	8300 3600 8300 3550
-Wire Wire Line
-	8000 3800 7900 3800
-Wire Wire Line
-	3650 2550 4000 2550
-Wire Wire Line
-	4950 1050 4950 1750
-Connection ~ 4950 1700
 Text GLabel 4050 3200 2    40   Input ~ 0
 WAKEUP0

Commit message: Updated LPC183x Hardware Design
Connections:
- wire segments 74 -> 75
Other:
- moved on the sheet: TP1
Changed lines of the file:
@@
-EESchema Schematic File Version 2  date 9/18/2011 8:03:49 PM
+EESchema Schematic File Version 2  date 9/19/2011 7:25:32 AM
 LIBS:power
 LIBS:device
@@
 Comment4 "www.MicropendousX.org"
 $EndDescr
+Connection ~ 3950 2550
+Wire Wire Line
+	3950 2550 3950 2650
+Connection ~ 3850 3050
+Wire Wire Line
+	4050 3200 3850 3200
+Wire Wire Line
+	3850 3200 3850 3050
+Wire Wire Line
+	4950 2000 4950 1950
+Wire Wire Line
+	3650 1050 4950 1050
+Wire Wire Line
+	9600 3800 9500 3800
+Wire Wire Line
+	9900 3600 9900 3550
+Wire Wire Line
+	9500 4000 9500 4050
+Wire Wire Line
+	9800 3800 9900 3800
+Wire Wire Line
+	9600 3650 9700 3650
+Wire Wire Line
+	9700 3650 9700 3750
+Wire Wire Line
+	10500 3750 10500 3650
+Wire Wire Line
+	10500 3650 10400 3650
+Wire Wire Line
+	10600 3800 10700 3800
+Wire Wire Line
+	10300 4000 10300 4050
+Wire Wire Line
+	10700 3600 10700 3550
+Wire Wire Line
+	10400 3800 10300 3800
+Wire Wire Line
+	8800 3800 8700 3800
+Wire Wire Line
+	9100 3600 9100 3550
+Wire Wire Line
+	8700 4000 8700 4050
+Wire Wire Line
+	9000 3800 9100 3800
+Wire Wire Line
+	8800 3650 8900 3650
+Wire Wire Line
+	8900 3650 8900 3750
+Wire Wire Line
+	8100 3750 8100 3650
+Wire Wire Line
+	8100 3650 8000 3650
+Wire Wire Line
+	8200 3800 8300 3800
+Wire Wire Line
+	7900 4000 7900 4050
+Wire Wire Line
+	6350 800  6350 1000
+Wire Wire Line
+	6000 4400 6000 4450
+Wire Wire Line
+	6650 4650 6650 4750
+Wire Wire Line
+	6650 4750 6550 4750
+Wire Wire Line
+	4000 3500 3650 3500
+Wire Wire Line
+	4000 2450 4000 2350
+Connection ~ 5100 2700
+Wire Wire Line
+	5150 2700 5100 2700
+Wire Wire Line
+	5650 650  5650 700
+Wire Wire Line
+	5200 1100 5200 1150
+Connection ~ 5650 900
+Connection ~ 4100 1300
+Wire Wire Line
+	4300 1300 3650 1300
+Connection ~ 4100 2100
+Wire Wire Line
+	4300 2100 3650 2100
+Connection ~ 4550 1950
+Wire Wire Line
+	4650 2000 4650 1950
+Wire Wire Line
+	4500 1800 4550 1800
+Wire Wire Line
+	4550 1800 4550 2100
+Wire Wire Line
+	4550 2100 4500 2100
+Wire Wire Line
+	4650 1950 4550 1950
+Connection ~ 4250 1450
+Wire Wire Line
+	4250 1450 4650 1450
+Wire Wire Line
+	4500 1600 4550 1600
+Wire Wire Line
+	4550 1600 4550 1300
+Wire Wire Line
+	4550 1300 4500 1300
+Connection ~ 4950 2900
+Wire Wire Line
+	5150 2900 4950 2900
+Wire Wire Line
+	4950 2600 4950 2450
+Wire Wire Line
+	4950 2800 4950 2950
+Wire Wire Line
+	5150 2500 4950 2500
+Connection ~ 4950 2500
+Wire Wire Line
+	4250 1400 4250 1500
+Wire Wire Line
+	4650 1450 4650 1500
+Connection ~ 4550 1450
+Wire Wire Line
+	4300 1800 3650 1800
+Connection ~ 4100 1800
+Wire Wire Line
+	4300 1600 3650 1600
+Connection ~ 4100 1600
+Wire Wire Line
+	5350 900  3650 900
+Connection ~ 5200 900
+Wire Wire Line
+	5150 2600 5100 2600
+Wire Wire Line
+	5100 2600 5100 2900
+Connection ~ 5100 2900
+Wire Wire Line
+	4200 2350 4300 2350
+Wire Wire Line
+	4300 2350 4300 2300
+Wire Wire Line
+	4000 2350 3650 2350
+Connection ~ 4000 2350
+Wire Wire Line
+	3650 3050 4000 3050
+Wire Wire Line
+	4300 3000 4300 3050
+Wire Wire Line
+	4300 3050 4200 3050
+Wire Wire Line
+	5350 5150 5350 5050
+Wire Wire Line
+	5350 5050 5450 5050
+Wire Wire Line
+	6000 4200 6000 4150
+Wire Wire Line
+	6650 1000 6650 1150
+Wire Wire Line
+	5550 900  6350 900
+Connection ~ 6350 900
+Wire Wire Line
+	5100 1700 4950 1700
+Wire Wire Line
+	8300 3600 8300 3550
+Wire Wire Line
+	8000 3800 7900 3800
+Wire Wire Line
+	4950 1050 4950 1750
+Connection ~ 4950 1700
+Wire Wire Line
+	4000 3300 4000 3200
 Connection ~ 4000 3200
 Wire Wire Line
-	4000 3300 4000 3200
-Connection ~ 4950 1700
-Wire Wire Line
-	4950 1750 4950 1050
-Wire Wire Line
-	3650 2550 4000 2550
-Wire Wire Line
-	8000 3800 7900 3800
-Wire Wire Line
-	8300 3600 8300 3550
-Wire Wire Line
-	5100 1700 4950 1700
-Connection ~ 6350 900
-Wire Wire Line
-	6350 900  5550 900
-Wire Wire Line
-	6650 1000 6650 1150
-Wire Wire Line
-	6000 4200 6000 4150
-Wire Wire Line
-	5450 5050 5350 5050
-Wire Wire Line
-	5350 5050 5350 5150
-Wire Wire Line
-	4200 3050 4300 3050
-Wire Wire Line
-	4300 3050 4300 3000
-Wire Wire Line
-	4000 3050 3650 3050
-Connection ~ 4000 2350
-Wire Wire Line
-	3650 2350 4000 2350
-Wire Wire Line
-	4300 2300 4300 2350
-Wire Wire Line
-	4300 2350 4200 2350
-Connection ~ 5100 2900
-Wire Wire Line
-	5100 2900 5100 2600
-Wire Wire Line
-	5100 2600 5150 2600
-Connection ~ 5200 900
-Wire Wire Line
-	3650 900  5350 900
-Connection ~ 4100 1600
-Wire Wire Line
-	3650 1600 4300 1600
-Connection ~ 4100 1800
-Wire Wire Line
-	3650 1800 4300 1800
-Connection ~ 4550 1450
-Wire Wire Line
-	4650 1500 4650 1450
-Wire Wire Line
-	4250 1500 4250 1400
-Connection ~ 4950 2500
-Wire Wire Line
-	5150 2500 4950 2500
-Wire Wire Line
-	4950 2950 4950 2800
-Wire Wire Line
-	4950 2450 4950 2600
-Wire Wire Line
-	5150 2900 4950 2900
-Connection ~ 4950 2900
-Wire Wire Line
-	4500 1300 4550 1300
-Wire Wire Line
-	4550 1300 4550 1600
-Wire Wire Line
-	4550 1600 4500 1600
-Wire Wire Line
-	4650 1450 4250 1450
-Connection ~ 4250 1450
-Wire Wire Line
-	4550 1950 4650 1950
-Wire Wire Line
-	4500 2100 4550 2100
-Wire Wire Line
-	4550 2100 4550 1800
-Wire Wire Line
-	4550 1800 4500 1800
-Wire Wire Line
-	4650 1950 4650 2000
-Connection ~ 4550 1950
-Wire Wire Line
-	3650 2100 4300 2100
-Connection ~ 4100 2100
-Wire Wire Line
-	3650 1300 4300 1300
-Connection ~ 4100 1300
-Connection ~ 5650 900
-Wire Wire Line
-	5200 1100 5200 1150
-Wire Wire Line
-	5650 650  5650 700
-Wire Wire Line
-	5150 2700 5100 2700
-Connection ~ 5100 2700
-Wire Wire Line
-	4000 2350 4000 2450
-Wire Wire Line
-	4000 3500 3650 3500
-Wire Wire Line
-	6550 4750 6650 4750
-Wire Wire Line
-	6650 4750 6650 4650
-Wire Wire Line
-	6000 4400 6000 4450
-Wire Wire Line
-	6350 1000 6350 800
-Wire Wire Line
-	7900 4000 7900 4050
-Wire Wire Line
-	8200 3800 8300 3800
-Wire Wire Line
-	8000 3650 8100 3650
-Wire Wire Line
-	8100 3650 8100 3750
-Wire Wire Line
-	8900 3750 8900 3650
-Wire Wire Line
-	8900 3650 8800 3650
-Wire Wire Line
-	9000 3800 9100 3800
-Wire Wire Line
-	8700 4000 8700 4050
-Wire Wire Line
-	9100 3600 9100 3550
-Wire Wire Line
-	8800 3800 8700 3800
-Wire Wire Line
-	10400 3800 10300 3800
-Wire Wire Line
-	10700 3600 10700 3550
-Wire Wire Line
-	10300 4000 10300 4050
-Wire Wire Line
-	10600 3800 10700 3800
-Wire Wire Line
-	10400 3650 10500 3650
-Wire Wire Line
-	10500 3650 10500 3750
-Wire Wire Line
-	9700 3750 9700 3650
-Wire Wire Line
-	9700 3650 9600 3650
-Wire Wire Line
-	9800 3800 9900 3800
-Wire Wire Line
-	9500 4000 9500 4050
-Wire Wire Line
-	9900 3600 9900 3550
-Wire Wire Line
-	9600 3800 9500 3800
-Wire Wire Line
-	4950 1050 3650 1050
-Wire Wire Line
-	4950 2000 4950 1950
-Wire Wire Line
-	3850 3050 3850 3200
-Wire Wire Line
-	3850 3200 4050 3200
-Connection ~ 3850 3050
+	4000 2550 3650 2550
+Text GLabel 4000 2550 2    40   BiDi ~ 0
+nTRST
 $Comp
 L CONN_1 TP7
@@
 Text Label 3650 2350 0    30   ~ 0
 DBGEN
-Text Label 3650 2550 0    30   ~ 0
-nTRST
 $Comp
 L CONN_1 TP1
 U 1 1 4E48FDEB
-P 4150 2550
-F 0 "TP1" H 4230 2550 40  0000 L CNN
-F 1 "nTRST" H 4150 2605 30  0001 C CNN
-	1    4150 2550
-	1    0    0    -1
-$EndComp
+P 4100 2650
+F 0 "TP1" H 4180 2650 40  0000 L CNN
+F 1 "nTRST" H 4100 2705 30  0001 C CNN
+	1    4100 2650
+	1    0    0    -1
+$EndComp

Commit message: Updated LPC183x Hardware Design
Parts:
- added R22: 199k, symbol R_MINI
Connections:
- wire segments 75 -> 78
