File: MicropendousX/Hardware/MicropendousX-LPC183x/MicropendousX-LPC183x-System.sch (KiCad schematic (older format))
At the start: 36 parts, among them IC1 LPC183X, IC7 25Q, SW1 RESET, U4 JTAG, X1 12MHz, X2 32.768kHz

Commit message: Updated MicropendousX-LPC183x portable design with minor post-prototyping corrections.
Connections:
- wire segments 80 -> 100
Other:
- note added: "EMC 16-Bit"
- note added: "EMC 32-Bit"
- note added: "EMC 8-Bit"
- note added: "SPI (SSP)"
- note added: "SPIFI"
- note added: "USART0"
- note added: "USART3"
- note added: "USB0"
- note added: "USB1"
- note removed: "UART"
- moved on the sheet: R40, R41, R42, R43, R44, R45, R46, R47
