File: MicropendousX/Hardware/MicropendousX-LPC183x/MicropendousX-LPC183x-USB.sch (KiCad schematic (older format))
At the start: 17 parts, among them IC1 LPC183X, U1 USB-A, U2 USB-A

Commit message: Update unfinished LPC183x-based design.
Other:
- moved on the sheet: CR1, CR2, CR3, CR4, CR5, F1, L10, L11, L8, L9, R1, R2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

Commit message: Updated LPC183x Hardware Design
Parts:
- removed CR3, CR4: ESD, symbol ESD
- removed L8, L9: FBY, symbol L_MINI
- removed R3, R4: 0, symbol R_MINI
- removed U2: USB-A, symbol USBCONN
- added unit 2 of IC1
- added unit 3 of IC1
- U1: value USB-A -> USB-microAB
Connections:
- net labels removed: USB-A_D+, USB-A_D-, USB1_DM, USB1_DP
- wire segments 60 -> 39
- no-connect marks 2 -> 53
Other:
- note removed: "To Device"
- moved on the sheet: CR1, CR2, CR5, F1, L10, L11, R1, R2

Commit message: Updated LPC183x Hardware Design
Other:
- note added: "Notes:\n- USB VBUS Fuse F1 limits inrush current\n- FBX ferrite bead is high DCR 0805\n- FBY ferrite beads are high current 0805\n- all other FB are 1A 0603, moderate DCR"
- note removed: "Notes:\n- FBX ferrite bead is high DCR 0805\n- FBY ferrite beads are high current 0805\n- all other FB are 1A 0603, moderate DCR"
Changed lines of the file:
@@
-EESchema Schematic File Version 2  date 9/18/2011 3:49:57 PM
+EESchema Schematic File Version 2  date 9/18/2011 8:03:49 PM
 LIBS:power
 LIBS:device
@@
 Sheet 4 7
 Title "MicropendousX-LPC183x"
-Date "18 sep 2011"
+Date "19 sep 2011"
 Rev "1.0"
 Comp "Opendous Inc."
@@
 $EndComp
 Text Notes 8082 2100 0    60   ~ 0
-Notes:\n- FBX ferrite bead is high DCR 0805\n- FBY ferrite beads are high current 0805\n- all other FB are 1A 0603, moderate DCR
+Notes:\n- USB VBUS Fuse F1 limits inrush current\n- FBX ferrite bead is high DCR 0805\n- FBY ferrite beads are high current 0805\n- all other FB are 1A 0603, moderate DCR
 Text Notes 7433 1950 0    20   ~ 0
 High DCR
