File: MicropendousX/Hardware/MicropendousX-LPC183x/MicropendousX-LPC183x-Vias.sch (KiCad schematic (older format))
At the start: 297 parts

Commit message: Updated LPC183x Hardware Design
Connections:
- net labels removed: 3V3_ETH_ANALOG, LEDL_A, LEDR_A, MAX8677_PEN1, MAX8677_PEN2, MAX8677_THM, MAX8677_USUS, MAX8677_VL, MAX8677_nCEN, MAX8677_nCHG, MAX8677_nDOK, MAX8677_nDONE, MAX8677_nFLT, MAX8677_nUOK
- wire segments 23 -> 25
Changed lines of the file:
@@
-EESchema Schematic File Version 2  date 8/20/2011 8:34:09 PM
+EESchema Schematic File Version 2  date 9/18/2011 3:49:57 PM
 LIBS:power
 LIBS:device
@@
 LIBS:contrib
 LIBS:valves
+LIBS:opendous
+LIBS:Opennect_Schematic_Symbols_Library
 LIBS:MicropendousX-LPC183x-cache
 EELAYER 25  0
@@
 $Descr A4 11700 8267
 encoding utf-8
-Sheet 9 9
+Sheet 7 7
 Title "MicropendousX-LPC183x"
-Date "21 aug 2011"
+Date "18 sep 2011"
 Rev "1.0"
 Comp "Opendous Inc."
@@
 Comment4 "www.MicropendousX.org"
 $EndDescr
-Text GLabel 11000 3250 0    40   Input ~ 0
-USB0_ID
-Text GLabel 11000 3350 0    40   Input ~ 0
-USB0_ID
-Text GLabel 11000 3450 0    40   BiDi ~ 0
-SPIFI_SIO2
-Text GLabel 11000 3550 0    40   BiDi ~ 0
-SPIFI_SIO2
-Text GLabel 11000 3950 0    40   UnSpc ~ 0
-USB0_DM
-Text GLabel 11000 3850 0    40   UnSpc ~ 0
-USB0_DP
-Text GLabel 11000 3650 0    40   UnSpc ~ 0
-USB0_DP
-Text GLabel 11000 3750 0    40   UnSpc ~ 0
-USB0_DM
+Connection ~ 11000 5250
+Wire Wire Line
+	11000 5350 11000 4150
+Connection ~ 11000 5050
+Connection ~ 11000 4850
+Connection ~ 11000 4650
+Connection ~ 11000 4450
+Connection ~ 11000 4250
+Wire Wire Line
+	11000 4650 10850 4650
+Wire Wire Line
+	10850 4650 10850 4800
 Connection ~ 6900 3400
 Connection ~ 6900 3500
@@
 Connection ~ 6900 4500
 Wire Wire Line
-	6900 3300 6900 4900
+	6900 4900 6900 3300
 Connection ~ 6900 4600
 Connection ~ 6900 4700
@@
 Connection ~ 6900 6300
 Wire Wire Line
-	6900 5000 6900 6400
+	6900 6400 6900 5000
 Wire Wire Line
 	10900 4050 11000 4050
@@
 Connection ~ 9000 2550
 Wire Wire Line
-	9000 6450 9000 550
+	9000 550  9000 6450
 Connection ~ 9000 2350
 Connection ~ 9000 2250
@@
 Connection ~ 11000 6050
 Wire Wire Line
-	11000 5950 11000 6150
+	11000 6150 11000 5950
 Wire Wire Line
 	10850 6050 11000 6050
@@
 	2300 5100 2450 5100
 Wire Wire Line
-	2450 6200 2450 4300
+	2450 4300 2450 6200
 Connection ~ 2450 6100
 Connection ~ 2450 6000
@@
 Connection ~ 2450 6400
 Wire Wire Line
-	2450 4200 2450 3300
-Wire Wire Line
-	11000 6250 11000 6450
+	2450 3300 2450 4200
+Wire Wire Line
+	11000 6450 11000 6250
 Connection ~ 11000 6350
 Connection ~ 9000 4550
 Connection ~ 9000 4450
 Wire Wire Line
-	11000 4150 10900 4150
-Wire Wire Line
-	2450 3200 2450 500
+	2450 500  2450 3200
 Connection ~ 2450 2500
 Connection ~ 2450 2400
 Wire Wire Line
-	6750 5700 6900 5700
-Wire Wire Line
-	6650 4100 6900 4100
-$Comp
-L VDDIO_3V3 #PWR0141
+	6900 5700 6750 5700
+Wire Wire Line
+	6900 4100 6650 4100
+Connection ~ 11000 4350
+Connection ~ 11000 4550
+Connection ~ 11000 4750
+Connection ~ 11000 4950
+Connection ~ 11000 5150
+$Comp
+L GND #PWR0131
+U 1 1 4E74194B
+P 10850 4800
+F 0 "#PWR0131" H 10850 4800 30  0001 C CNN
+F 1 "GND" H 10850 4730 30  0001 C CNN
+	1    10850 4800
+	1    0    0    -1
+$EndComp
+Text GLabel 11000 3250 0    40   Input ~ 0
+USB0_ID
+Text GLabel 11000 3350 0    40   Input ~ 0
+USB0_ID
+Text GLabel 11000 3450 0    40   BiDi ~ 0
+SPIFI_SIO2
+Text GLabel 11000 3550 0    40   BiDi ~ 0
+SPIFI_SIO2
+Text GLabel 11000 3950 0    40   UnSpc ~ 0
+USB0_DM
+Text GLabel 11000 3850 0    40   UnSpc ~ 0
+USB0_DP
+Text GLabel 11000 3650 0    40   UnSpc ~ 0
+USB0_DP
+Text GLabel 11000 3750 0    40   UnSpc ~ 0
+USB0_DM
+$Comp
+L VDDIO_3V3 #PWR0132
 U 1 1 4E49585F
 P 6650 4100
-F 0 "#PWR0141" H 6650 4200 30  0001 C CNN
+F 0 "#PWR0132" H 6650 4200 30  0001 C CNN
 F 1 "VDDIO_3V3" H 6650 4200 30  0000 C CNN
 	1    6650 4100
@@
 $EndComp
 $Comp
-L VDD3V3 #PWR0142
+L VDD3V3 #PWR0133
 U 1 1 4E49554D
 P 6750 5700
-F 0 "#PWR0142" H 6750 5800 30  0001 C CNN
+F 0 "#PWR0133" H 6750 5800 30  0001 C CNN
 F 1 "VDD3V3" H 6750 5800 30  0000 C CNN
 	1    6750 5700
@@
 $EndComp
 $Comp
-L DC_VIN #PWR0143
+L DC_VIN #PWR0134
 U 1 1 4E266D31
 P 10900 4050
-F 0 "#PWR0143" H 10900 4150 30  0001 C CNN
+F 0 "#PWR0134" H 10900 4150 30  0001 C CNN
 F 1 "DC_VIN" V 10900 4200 30  0000 C CNN
 	1    10900 4050
@@
 $EndComp
 $Comp
-L 3V3_ETH_ANALOG #PWR0144
-U 1 1 4E2662BA
-P 10900 4150
-F 0 "#PWR0144" H 10900 4250 30  0001 C CNN
-F 1 "3V3_ETH_ANALOG" V 10900 4450 30  0000 C CNN
-	1    10900 4150
-	0    -1   -1   0
-$EndComp
-Text GLabel 11000 4250 0    40   Input ~ 0
-LEDL_A
-Text GLabel 11000 4350 0    40   Input ~ 0
-LEDR_A
-Text GLabel 11000 4550 0    40   Input ~ 0
-MAX8677_VL
-Text GLabel 11000 4450 0    40   Input ~ 0
-MAX8677_VL
-$Comp
-L GNDPWR #PWR0145
+L GNDPWR #PWR0135
 U 1 1 4E24500E
 P 8850 5500
-F 0 "#PWR0145" H 8850 5550 40  0001 C CNN
+F 0 "#PWR0135" H 8850 5550 40  0001 C CNN
 F 1 "GNDPWR" H 8850 5420 40  0000 C CNN
 	1    8850 5500
 	1    0    0    -1
 $EndComp
-Text GLabel 11000 4650 0    40   Input ~ 0
-MAX8677_THM
-Text GLabel 11000 4950 0    40   Input ~ 0
-MAX8677_nDONE
-Text GLabel 11000 4850 0    40   Input ~ 0
-MAX8677_nCHG
-Text GLabel 11000 5150 0    40   Input ~ 0
-MAX8677_nFLT
-Text GLabel 11000 5350 0    40   Input ~ 0
-MAX8677_nDOK
-Text GLabel 11000 5750 0    40   Input ~ 0
-MAX8677_nCEN
-Text GLabel 11000 5550 0    40   Input ~ 0
-MAX8677_nUOK
-Text GLabel 11000 5650 0    40   Input ~ 0
-MAX8677_nUOK
-Text GLabel 11000 5850 0    40   Input ~ 0
-MAX8677_nCEN
-Text GLabel 11000 5450 0    40   Input ~ 0
-MAX8677_nDOK
-Text GLabel 11000 5250 0    40   Input ~ 0
-MAX8677_nFLT
-Text GLabel 11000 4750 0    40   Input ~ 0
-MAX8677_nCHG
-Text GLabel 11000 5050 0    40   Input ~ 0
-MAX8677_nDONE
-$Comp
-L VSYS #PWR0146
+$Comp
+L VSYS #PWR0136
 U 1 1 4E24421B
 P 10850 6050
-F 0 "#PWR0146" H 10850 6150 30  0001 C CNN
+F 0 "#PWR0136" H 10850 6150 30  0001 C CNN
 F 1 "VSYS" H 10850 6150 30  0000 C CNN
 	1    10850 6050
@@
 $EndComp
 $Comp
-L 5V0 #PWR0147
+L 5V0 #PWR0137
 U 1 1 4E244116
 P 10850 6350
-F 0 "#PWR0147" H 10850 6450 30  0001 C CNN
+F 0 "#PWR0137" H 10850 6450 30  0001 C CNN
 F 1 "5V0" H 10850 6450 30  0000 C CNN
 	1    10850 6350
@@
 $EndComp
 $Comp
-L VDDIO_3V3 #PWR0148
+L VDDIO_3V3 #PWR0138
 U 1 1 4E2437D2
 P 2200 3900
-F 0 "#PWR0148" H 2200 4000 30  0001 C CNN
+F 0 "#PWR0138" H 2200 4000 30  0001 C CNN
 F 1 "VDDIO_3V3" H 2200 4000 30  0000 C CNN
 	1    2200 3900
@@
 $EndComp
 $Comp
-L GND #PWR0149
+L GND #PWR0139
 U 1 1 4E24344B
 P 2300 5250
-F 0 "#PWR0149" H 2300 5250 30  0001 C CNN
+F 0 "#PWR0139" H 2300 5250 30  0001 C CNN
 F 1 "GND" H 2300 5180 30  0001 C CNN
 	1    2300 5250
@@
 $EndComp
 $Comp
-L VBUS #PWR0150
+L VBUS #PWR0140
 U 1 1 4E2423A0
 P 2200 6500
-F 0 "#PWR0150" H 2200 6600 30  0001 C CNN
+F 0 "#PWR0140" H 2200 6600 30  0001 C CNN
 F 1 "VBUS" H 2200 6600 30  0000 C CNN
 	1    2200 6500
 	1    0    0    -1
 $EndComp
-Text GLabel 2450 6700 0    40   Input ~ 0
-MAX8677_USUS
-Text GLabel 2450 6600 0    40   Input ~ 0
-MAX8677_USUS
-Text GLabel 2450 6800 0    40   Input ~ 0
-MAX8677_PEN2
-Text GLabel 2450 6900 0    40   Input ~ 0
-MAX8677_PEN2
-Text GLabel 2450 7100 0    40   Input ~ 0
-MAX8677_PEN1
-Text GLabel 2450 7000 0    40   Input ~ 0
-MAX8677_PEN1
 Text GLabel 2450 7200 0    40   Input ~ 0
 GND_microAB
@@
 GND_microAB
 $Comp
-L GND #PWR0151
+L GND #PWR0141
 U 1 1 4E241B4C
 P 2300 1450
-F 0 "#PWR0151" H 2300 1450 30  0001 C CNN
+F 0 "#PWR0141" H 2300 1450 30  0001 C CNN
 F 1 "GND" H 2300 1380 30  0001 C CNN
 	1    2300 1450

Commit message: Updated LPC183x Hardware Design
Connections:
- net labels added: 6V0, CLKOUT-I2S1_RX_SCK, GPIO0_12-ENET_MDIO, SPIFI_SCK-CGU_OUT1, SPIFI_SIO2-I2S1_RX_WS, SSP1_SCK-ENET_REF_CLK, SSP1_SSEL-ENET_TXD1, U2_RXD-GPIO0_3-ENET_RX_DV, U2_TXD-GPIO0_2-ENET_RXD0
- net labels removed: DC_VIN, SPIFI_SIO2
Changed lines of the file:
@@
-EESchema Schematic File Version 2  date 9/18/2011 3:49:57 PM
+EESchema Schematic File Version 2  date 9/18/2011 8:03:49 PM
 LIBS:power
 LIBS:device
@@
 Sheet 7 7
 Title "MicropendousX-LPC183x"
-Date "18 sep 2011"
+Date "19 sep 2011"
 Rev "1.0"
 Comp "Opendous Inc."
@@
 Comment4 "www.MicropendousX.org"
 $EndDescr
+Text GLabel 11000 2550 0    40   Input ~ 0
+CLKOUT-I2S1_RX_SCK
+Text GLabel 11000 2650 0    40   Input ~ 0
+SPIFI_SCK-CGU_OUT1
+Text GLabel 11000 2750 0    40   Input ~ 0
+SSP1_SCK-ENET_REF_CLK
+Text GLabel 11000 3150 0    40   BiDi ~ 0
+U2_RXD-GPIO0_3-ENET_RX_DV
+Text GLabel 11000 3050 0    40   BiDi ~ 0
+U2_TXD-GPIO0_2-ENET_RXD0
+Text GLabel 11000 2950 0    40   Input ~ 0
+GPIO0_12-ENET_MDIO
+Text GLabel 11000 2850 0    40   Input ~ 0
+SSP1_SSEL-ENET_TXD1
+$Comp
+L 6V0 #PWR0136
+U 1 1 4E766648
+P 10900 4050
+F 0 "#PWR0136" H 10900 4190 20  0001 C CNN
+F 1 "6V0" V 10900 4200 30  0000 C CNN
+	1    10900 4050
+	0    -1   -1   0
+$EndComp
 Connection ~ 11000 5250
 Wire Wire Line
@@
 Connection ~ 11000 5150
 $Comp
-L GND #PWR0131
+L GND #PWR0137
 U 1 1 4E74194B
 P 10850 4800
-F 0 "#PWR0131" H 10850 4800 30  0001 C CNN
+F 0 "#PWR0137" H 10850 4800 30  0001 C CNN
 F 1 "GND" H 10850 4730 30  0001 C CNN
 	1    10850 4800
@@
 USB0_ID
 Text GLabel 11000 3450 0    40   BiDi ~ 0
-SPIFI_SIO2
+SPIFI_SIO2-I2S1_RX_WS
 Text GLabel 11000 3550 0    40   BiDi ~ 0
-SPIFI_SIO2
+SPIFI_SIO2-I2S1_RX_WS
 Text GLabel 11000 3950 0    40   UnSpc ~ 0
 USB0_DM
@@
 USB0_DM
 $Comp
-L VDDIO_3V3 #PWR0132
+L VDDIO_3V3 #PWR0138
 U 1 1 4E49585F
 P 6650 4100
-F 0 "#PWR0132" H 6650 4200 30  0001 C CNN
+F 0 "#PWR0138" H 6650 4200 30  0001 C CNN
 F 1 "VDDIO_3V3" H 6650 4200 30  0000 C CNN
 	1    6650 4100
@@
 $EndComp
 $Comp
-L VDD3V3 #PWR0133
+L VDD3V3 #PWR0139
 U 1 1 4E49554D
 P 6750 5700
-F 0 "#PWR0133" H 6750 5800 30  0001 C CNN
+F 0 "#PWR0139" H 6750 5800 30  0001 C CNN
 F 1 "VDD3V3" H 6750 5800 30  0000 C CNN
 	1    6750 5700
@@
 $EndComp
 $Comp
-L DC_VIN #PWR0134
-U 1 1 4E266D31
-P 10900 4050
-F 0 "#PWR0134" H 10900 4150 30  0001 C CNN
-F 1 "DC_VIN" V 10900 4200 30  0000 C CNN
-	1    10900 4050
-	0    -1   -1   0
-$EndComp
-$Comp
-L GNDPWR #PWR0135
+L GNDPWR #PWR0140
 U 1 1 4E24500E
 P 8850 5500
-F 0 "#PWR0135" H 8850 5550 40  0001 C CNN
+F 0 "#PWR0140" H 8850 5550 40  0001 C CNN
 F 1 "GNDPWR" H 8850 5420 40  0000 C CNN
 	1    8850 5500
@@
 $EndComp
 $Comp
-L VSYS #PWR0136
+L VSYS #PWR0141
 U 1 1 4E24421B
 P 10850 6050
-F 0 "#PWR0136" H 10850 6150 30  0001 C CNN
+F 0 "#PWR0141" H 10850 6150 30  0001 C CNN
 F 1 "VSYS" H 10850 6150 30  0000 C CNN
 	1    10850 6050
@@
 $EndComp
 $Comp
-L 5V0 #PWR0137
+L 5V0 #PWR0142
 U 1 1 4E244116
 P 10850 6350
-F 0 "#PWR0137" H 10850 6450 30  0001 C CNN
+F 0 "#PWR0142" H 10850 6450 30  0001 C CNN
 F 1 "5V0" H 10850 6450 30  0000 C CNN
 	1    10850 6350
@@
 $EndComp
 $Comp
-L VDDIO_3V3 #PWR0138
+L VDDIO_3V3 #PWR0143
 U 1 1 4E2437D2
 P 2200 3900
-F 0 "#PWR0138" H 2200 4000 30  0001 C CNN
+F 0 "#PWR0143" H 2200 4000 30  0001 C CNN
 F 1 "VDDIO_3V3" H 2200 4000 30  0000 C CNN
 	1    2200 3900
@@
 $EndComp
 $Comp
-L GND #PWR0139
+L GND #PWR0144
 U 1 1 4E24344B
 P 2300 5250
-F 0 "#PWR0139" H 2300 5250 30  0001 C CNN
+F 0 "#PWR0144" H 2300 5250 30  0001 C CNN
 F 1 "GND" H 2300 5180 30  0001 C CNN
 	1    2300 5250
@@
 $EndComp
 $Comp
-L VBUS #PWR0140
+L VBUS #PWR0145
 U 1 1 4E2423A0
 P 2200 6500
-F 0 "#PWR0140" H 2200 6600 30  0001 C CNN
+F 0 "#PWR0145" H 2200 6600 30  0001 C CNN
 F 1 "VBUS" H 2200 6600 30  0000 C CNN
 	1    2200 6500
@@
 GND_microAB
 $Comp
-L GND #PWR0141
+L GND #PWR0146
 U 1 1 4E241B4C
 P 2300 1450
-F 0 "#PWR0141" H 2300 1450 30  0001 C CNN
+F 0 "#PWR0146" H 2300 1450 30  0001 C CNN
 F 1 "GND" H 2300 1380 30  0001 C CNN
 	1    2300 1450

Commit message: Updated LPC183x Hardware Design
Connections:
- net GND: now also V167.1 (Via), V168.1 (Via), V169.1 (Via), V170.1 (Via), V171.1 (Via), V172.1 (Via), V173.1 (Via), V174.1 (Via), V175.1 (Via), V176.1 (Via), V62.1 (Via), V63.1 (Via), V64.1 (Via), V65.1 (Via), V66.1 (Via), V67.1 (Via)
- net VBUS: now also V305.1 (Via)
- net +BATT: now reaches V178.1 (Via)
- net +BATT: now also V177.1 (Via), V179.1 (Via), V180.1 (Via), V181.1 (Via), V182.1 (Via), V183.1 (Via)
- net LTC3559_NTC: now reaches V306.1 (Via)
- net LTC3559_~CHRG~: now reaches V307.1 (Via)
- net LTC3559_~CHRG~: now also V308.1 (Via)
- net GPIO5_2: now reaches V312.1 (Via)
- net GPIO5_2: now also V311.1 (Via)
- net I2C1_SCL-U3_RXD: now reaches V309.1 (Via)
- net I2C1_SCL-U3_RXD: now also V315.1 (Via)
- net I2C1_SDA-U3_TXD: now reaches V310.1 (Via)
- net I2C1_SDA-U3_TXD: now also V316.1 (Via)
- net nTRST: now reaches V302.1 (Via)
- net TDO: now reaches V303.1 (Via)
- net TMS: now reaches V304.1 (Via)
- net GPIO3_7: now reaches V313.1 (Via)
- net GPIO3_7: now also V314.1 (Via)
- net GPIO0_12-ENET_MDIO renamed GPIO0_12
- net SSP1_SCK-ENET_REF_CLK renamed SSP1_SCK
- net SSP1_SSEL-ENET_TXD1 renamed SSP1_SSEL
- net U2_RXD-GPIO0_3-ENET_RX_DV renamed U2_RXD-GPIO0_3
- net U2_TXD-GPIO0_2-ENET_RXD0 renamed U2_TXD-GPIO0_2
Changed lines of the file:
@@
-EESchema Schematic File Version 2  date 9/18/2011 8:03:49 PM
+EESchema Schematic File Version 2  date 9/19/2011 7:25:32 AM
 LIBS:power
 LIBS:device
@@
 Comment4 "www.MicropendousX.org"
 $EndDescr
-Text GLabel 11000 2550 0    40   Input ~ 0
-CLKOUT-I2S1_RX_SCK
-Text GLabel 11000 2650 0    40   Input ~ 0
-SPIFI_SCK-CGU_OUT1
-Text GLabel 11000 2750 0    40   Input ~ 0
-SSP1_SCK-ENET_REF_CLK
-Text GLabel 11000 3150 0    40   BiDi ~ 0
-U2_RXD-GPIO0_3-ENET_RX_DV
-Text GLabel 11000 3050 0    40   BiDi ~ 0
-U2_TXD-GPIO0_2-ENET_RXD0
-Text GLabel 11000 2950 0    40   Input ~ 0
-GPIO0_12-ENET_MDIO
-Text GLabel 11000 2850 0    40   Input ~ 0
-SSP1_SSEL-ENET_TXD1
-$Comp
-L 6V0 #PWR0136
-U 1 1 4E766648
-P 10900 4050
-F 0 "#PWR0136" H 10900 4190 20  0001 C CNN
-F 1 "6V0" V 10900 4200 30  0000 C CNN
-	1    10900 4050
-	0    -1   -1   0
-$EndComp
+Text GLabel 11000 1050 0    40   Input ~ 0
+nTRST
+Text GLabel 11000 1150 0    40   Input ~ 0
+TDO
+Text GLabel 11000 1250 0    40   Input ~ 0
+TMS
+Wire Wire Line
+	10950 1350 11000 1350
+Connection ~ 6900 900
+Wire Wire Line
+	2300 5250 2300 5100
+Wire Wire Line
+	2300 5100 2450 5100
+Wire Wire Line
+	2450 6700 2300 6700
+Wire Wire Line
+	2300 6700 2300 6850
+Connection ~ 4650 6900
+Wire Wire Line
+	4650 6800 4650 7700
+Connection ~ 4650 7100
+Connection ~ 4650 7300
+Connection ~ 4650 7500
+Connection ~ 2450 6900
+Connection ~ 2450 6700
+Wire Wire Line
+	6700 700  6900 700
+Connection ~ 6900 600
 Connection ~ 11000 5250
 Wire Wire Line
@@
 	2450 3900 2200 3900
 Wire Wire Line
-	2300 5250 2300 5100
-Wire Wire Line
-	2300 5100 2450 5100
+	4500 7450 4500 7300
+Wire Wire Line
+	4500 7300 4650 7300
 Wire Wire Line
 	2450 4300 2450 6200
@@
 Connection ~ 11000 4950
 Connection ~ 11000 5150
-$Comp
-L GND #PWR0137
+Connection ~ 6900 700
+Connection ~ 2450 6800
+Wire Wire Line
+	2450 7100 2450 6600
+Connection ~ 2450 7000
+Connection ~ 4650 7600
+Connection ~ 4650 7400
+Connection ~ 4650 7200
+Connection ~ 4650 7000
+Connection ~ 6900 800
+Wire Wire Line
+	6900 1100 6900 500
+Connection ~ 6900 1000
+$Comp
+L VBUS #PWR0137
+U 1 1 4E771EB8
+P 10950 1350
+F 0 "#PWR0137" H 10950 1450 30  0001 C CNN
+F 1 "VBUS" V 10950 1500 30  0000 C CNN
+	1    10950 1350
+	0    -1   -1   0
+$EndComp
+Text GLabel 11000 1450 0    40   Input ~ 0
+LTC3559_NTC
+Text GLabel 11000 1550 0    40   Input ~ 0
+LTC3559_~CHRG~
+Text GLabel 11000 1650 0    40   Input ~ 0
+LTC3559_~CHRG~
+Text GLabel 11000 1750 0    40   Input ~ 0
+I2C1_SCL-U3_RXD
+Text GLabel 11000 1850 0    40   Input ~ 0
+I2C1_SDA-U3_TXD
+Text GLabel 11000 2050 0    40   Input ~ 0
+GPIO5_2
+Text GLabel 11000 1950 0    40   Input ~ 0
+GPIO5_2
+Text GLabel 11000 2150 0    40   Input ~ 0
+GPIO3_7
+Text GLabel 11000 2250 0    40   Input ~ 0
+GPIO3_7
+Text GLabel 11000 2450 0    40   Input ~ 0
+I2C1_SDA-U3_TXD
+Text GLabel 11000 2350 0    40   Input ~ 0
+I2C1_SCL-U3_RXD
+$Comp
+L GND #PWR0138
+U 1 1 4E76CD8A
+P 2300 5250
+F 0 "#PWR0138" H 2300 5250 30  0001 C CNN
+F 1 "GND" H 2300 5180 30  0001 C CNN
+	1    2300 5250
+	1    0    0    -1
+$EndComp
+$Comp
+L GND #PWR0139
+U 1 1 4E76CCD0
+P 2300 6850
+F 0 "#PWR0139" H 2300 6850 30  0001 C CNN
+F 1 "GND" H 2300 6780 30  0001 C CNN
+	1    2300 6850
+	1    0    0    -1
+$EndComp
+$Comp
+L +BATT #PWR0140
+U 1 1 4E76C805
+P 6700 700
+F 0 "#PWR0140" H 6700 650 20  0001 C CNN
+F 1 "+BATT" H 6700 800 30  0000 C CNN
+	1    6700 700
+	1    0    0    -1
+$EndComp
+Text GLabel 11000 2550 0    40   Input ~ 0
+CLKOUT-I2S1_RX_SCK
+Text GLabel 11000 2650 0    40   Input ~ 0
+SPIFI_SCK-CGU_OUT1
+Text GLabel 11000 2750 0    40   Input ~ 0
+SSP1_SCK
+Text GLabel 11000 3150 0    40   BiDi ~ 0
+U2_RXD-GPIO0_3
+Text GLabel 11000 3050 0    40   BiDi ~ 0
+U2_TXD-GPIO0_2
+Text GLabel 11000 2950 0    40   Input ~ 0
+GPIO0_12
+Text GLabel 11000 2850 0    40   Input ~ 0
+SSP1_SSEL
+$Comp
+L 6V0 #PWR0141
+U 1 1 4E766648
+P 10900 4050
+F 0 "#PWR0141" H 10900 4190 20  0001 C CNN
+F 1 "6V0" V 10900 4200 30  0000 C CNN
+	1    10900 4050
+	0    -1   -1   0
+$EndComp
+$Comp
+L GND #PWR0142
 U 1 1 4E74194B
 P 10850 4800
-F 0 "#PWR0137" H 10850 4800 30  0001 C CNN
+F 0 "#PWR0142" H 10850 4800 30  0001 C CNN
 F 1 "GND" H 10850 4730 30  0001 C CNN
 	1    10850 4800
@@
 USB0_DM
 $Comp
-L VDDIO_3V3 #PWR0138
+L VDDIO_3V3 #PWR0143
 U 1 1 4E49585F
 P 6650 4100
-F 0 "#PWR0138" H 6650 4200 30  0001 C CNN
+F 0 "#PWR0143" H 6650 4200 30  0001 C CNN
 F 1 "VDDIO_3V3" H 6650 4200 30  0000 C CNN
 	1    6650 4100
@@
 $EndComp
 $Comp
-L VDD3V3 #PWR0139
+L VDD3V3 #PWR0144
 U 1 1 4E49554D
 P 6750 5700
-F 0 "#PWR0139" H 6750 5800 30  0001 C CNN
+F 0 "#PWR0144" H 6750 5800 30  0001 C CNN
 F 1 "VDD3V3" H 6750 5800 30  0000 C CNN
 	1    6750 5700
@@
 $EndComp
 $Comp
-L GNDPWR #PWR0140
+L GNDPWR #PWR0145
 U 1 1 4E24500E
 P 8850 5500
-F 0 "#PWR0140" H 8850 5550 40  0001 C CNN
+F 0 "#PWR0145" H 8850 5550 40  0001 C CNN
 F 1 "GNDPWR" H 8850 5420 40  0000 C CNN
 	1    8850 5500
@@
 $EndComp
 $Comp
-L VSYS #PWR0141
+L VSYS #PWR0146
 U 1 1 4E24421B
 P 10850 6050
-F 0 "#PWR0141" H 10850 6150 30  0001 C CNN
+F 0 "#PWR0146" H 10850 6150 30  0001 C CNN
 F 1 "VSYS" H 10850 6150 30  0000 C CNN
 	1    10850 6050
@@
 $EndComp
 $Comp
-L 5V0 #PWR0142
+L 5V0 #PWR0147
 U 1 1 4E244116
 P 10850 6350
-F 0 "#PWR0142" H 10850 6450 30  0001 C CNN
+F 0 "#PWR0147" H 10850 6450 30  0001 C CNN
 F 1 "5V0" H 10850 6450 30  0000 C CNN
 	1    10850 6350
@@
 $EndComp
 $Comp
-L VDDIO_3V3 #PWR0143
+L VDDIO_3V3 #PWR0148
 U 1 1 4E2437D2
 P 2200 3900
-F 0 "#PWR0143" H 2200 4000 30  0001 C CNN
+F 0 "#PWR0148" H 2200 4000 30  0001 C CNN
 F 1 "VDDIO_3V3" H 2200 4000 30  0000 C CNN
 	1    2200 3900
@@
 $EndComp
 $Comp
-L GND #PWR0144
+L GND #PWR0149
 U 1 1 4E24344B
-P 2300 5250
-F 0 "#PWR0144" H 2300 5250 30  0001 C CNN
-F 1 "GND" H 2300 5180 30  0001 C CNN
-	1    2300 5250
-	1    0    0    -1
-$EndComp
-$Comp
-L VBUS #PWR0145
+P 4500 7450
+F 0 "#PWR0149" H 4500 7450 30  0001 C CNN
+F 1 "GND" H 4500 7380 30  0001 C CNN
+	1    4500 7450
+	1    0    0    -1
+$EndComp
+$Comp
+L VBUS #PWR0150
 U 1 1 4E2423A0
 P 2200 6500
-F 0 "#PWR0145" H 2200 6600 30  0001 C CNN
+F 0 "#PWR0150" H 2200 6600 30  0001 C CNN
 F 1 "VBUS" H 2200 6600 30  0000 C CNN
 	1    2200 6500
@@
 GND_microAB
 $Comp
-L GND #PWR0146
+L GND #PWR0151
 U 1 1 4E241B4C
 P 2300 1450
-F 0 "#PWR0146" H 2300 1450 30  0001 C CNN
+F 0 "#PWR0151" H 2300 1450 30  0001 C CNN
 F 1 "GND" H 2300 1380 30  0001 C CNN
 	1    2300 1450
