File: MicropendousX/Hardware/MicropendousX-LPC183x/MicropendousX-LPC183x-Vias.sch (KiCad schematic (older format))
At the start: 297 parts

Commit message: Updated LPC183x Hardware Design
Connections:
- net GPIO3_7: now also V301.1 (Via)
- net GPIO5_2: now also V300.1 (Via)
- net ADC1_1: now reaches V299.1 (Via)
- net ADC1_1: now also V298.1 (Via)
Changed lines of the file:
@@
-EESchema Schematic File Version 2  date 9/19/2011 7:25:32 AM
+EESchema Schematic File Version 2  date 9/23/2011 8:04:30 AM
 LIBS:power
 LIBS:device
@@
 Sheet 7 7
 Title "MicropendousX-LPC183x"
-Date "19 sep 2011"
+Date "23 sep 2011"
 Rev "1.0"
 Comp "Opendous Inc."
@@
 Comment4 "www.MicropendousX.org"
 $EndDescr
+Text GLabel 11000 650  0    40   Input ~ 0
+ADC1_1
+Text GLabel 11000 750  0    40   Input ~ 0
+ADC1_1
+Text GLabel 11000 950  0    40   Input ~ 0
+GPIO3_7
+Text GLabel 11000 850  0    40   Input ~ 0
+GPIO5_2
 Text GLabel 11000 1050 0    40   Input ~ 0
 nTRST
@@
 Connection ~ 6900 1000
 $Comp
-L VBUS #PWR0137
+L VBUS #PWR0139
 U 1 1 4E771EB8
 P 10950 1350
-F 0 "#PWR0137" H 10950 1450 30  0001 C CNN
+F 0 "#PWR0139" H 10950 1450 30  0001 C CNN
 F 1 "VBUS" V 10950 1500 30  0000 C CNN
 	1    10950 1350
@@
 I2C1_SCL-U3_RXD
 $Comp
-L GND #PWR0138
+L GND #PWR0140
 U 1 1 4E76CD8A
 P 2300 5250
-F 0 "#PWR0138" H 2300 5250 30  0001 C CNN
+F 0 "#PWR0140" H 2300 5250 30  0001 C CNN
 F 1 "GND" H 2300 5180 30  0001 C CNN
 	1    2300 5250
@@
 $EndComp
 $Comp
-L GND #PWR0139
+L GND #PWR0141
 U 1 1 4E76CCD0
 P 2300 6850
-F 0 "#PWR0139" H 2300 6850 30  0001 C CNN
+F 0 "#PWR0141" H 2300 6850 30  0001 C CNN
 F 1 "GND" H 2300 6780 30  0001 C CNN
 	1    2300 6850
@@
 $EndComp
 $Comp
-L +BATT #PWR0140
+L +BATT #PWR0142
 U 1 1 4E76C805
 P 6700 700
-F 0 "#PWR0140" H 6700 650 20  0001 C CNN
+F 0 "#PWR0142" H 6700 650 20  0001 C CNN
 F 1 "+BATT" H 6700 800 30  0000 C CNN
 	1    6700 700
@@
 SSP1_SSEL
 $Comp
-L 6V0 #PWR0141
+L 6V0 #PWR0143
 U 1 1 4E766648
 P 10900 4050
-F 0 "#PWR0141" H 10900 4190 20  0001 C CNN
+F 0 "#PWR0143" H 10900 4190 20  0001 C CNN
 F 1 "6V0" V 10900 4200 30  0000 C CNN
 	1    10900 4050
@@
 $EndComp
 $Comp
-L GND #PWR0142
+L GND #PWR0144
 U 1 1 4E74194B
 P 10850 4800
-F 0 "#PWR0142" H 10850 4800 30  0001 C CNN
+F 0 "#PWR0144" H 10850 4800 30  0001 C CNN
 F 1 "GND" H 10850 4730 30  0001 C CNN
 	1    10850 4800
@@
 USB0_DM
 $Comp
-L VDDIO_3V3 #PWR0143
+L VDDIO_3V3 #PWR0145
 U 1 1 4E49585F
 P 6650 4100
-F 0 "#PWR0143" H 6650 4200 30  0001 C CNN
+F 0 "#PWR0145" H 6650 4200 30  0001 C CNN
 F 1 "VDDIO_3V3" H 6650 4200 30  0000 C CNN
 	1    6650 4100
@@
 $EndComp
 $Comp
-L VDD3V3 #PWR0144
+L VDD3V3 #PWR0146
 U 1 1 4E49554D
 P 6750 5700
-F 0 "#PWR0144" H 6750 5800 30  0001 C CNN
+F 0 "#PWR0146" H 6750 5800 30  0001 C CNN
 F 1 "VDD3V3" H 6750 5800 30  0000 C CNN
 	1    6750 5700
@@
 $EndComp
 $Comp
-L GNDPWR #PWR0145
+L GNDPWR #PWR0147
 U 1 1 4E24500E
 P 8850 5500
-F 0 "#PWR0145" H 8850 5550 40  0001 C CNN
+F 0 "#PWR0147" H 8850 5550 40  0001 C CNN
 F 1 "GNDPWR" H 8850 5420 40  0000 C CNN
 	1    8850 5500
@@
 $EndComp
 $Comp
-L VSYS #PWR0146
+L VSYS #PWR0148
 U 1 1 4E24421B
 P 10850 6050
-F 0 "#PWR0146" H 10850 6150 30  0001 C CNN
+F 0 "#PWR0148" H 10850 6150 30  0001 C CNN
 F 1 "VSYS" H 10850 6150 30  0000 C CNN
 	1    10850 6050
@@
 $EndComp
 $Comp
-L 5V0 #PWR0147
+L 5V0 #PWR0149
 U 1 1 4E244116
 P 10850 6350
-F 0 "#PWR0147" H 10850 6450 30  0001 C CNN
+F 0 "#PWR0149" H 10850 6450 30  0001 C CNN
 F 1 "5V0" H 10850 6450 30  0000 C CNN
 	1    10850 6350
@@
 $EndComp
 $Comp
-L VDDIO_3V3 #PWR0148
+L VDDIO_3V3 #PWR0150
 U 1 1 4E2437D2
 P 2200 3900
-F 0 "#PWR0148" H 2200 4000 30  0001 C CNN
+F 0 "#PWR0150" H 2200 4000 30  0001 C CNN
 F 1 "VDDIO_3V3" H 2200 4000 30  0000 C CNN
 	1    2200 3900
@@
 $EndComp
 $Comp
-L GND #PWR0149
+L GND #PWR0151
 U 1 1 4E24344B
 P 4500 7450
-F 0 "#PWR0149" H 4500 7450 30  0001 C CNN
+F 0 "#PWR0151" H 4500 7450 30  0001 C CNN
 F 1 "GND" H 4500 7380 30  0001 C CNN
 	1    4500 7450
@@
 $EndComp
 $Comp
-L VBUS #PWR0150
+L VBUS #PWR0152
 U 1 1 4E2423A0
 P 2200 6500
-F 0 "#PWR0150" H 2200 6600 30  0001 C CNN
+F 0 "#PWR0152" H 2200 6600 30  0001 C CNN
 F 1 "VBUS" H 2200 6600 30  0000 C CNN
 	1    2200 6500
@@
 GND_microAB
 $Comp
-L GND #PWR0151
+L GND #PWR0153
 U 1 1 4E241B4C
 P 2300 1450
-F 0 "#PWR0151" H 2300 1450 30  0001 C CNN
+F 0 "#PWR0153" H 2300 1450 30  0001 C CNN
 F 1 "GND" H 2300 1380 30  0001 C CNN
 	1    2300 1450

Commit message: Updated LPC183x Hardware Design
Connections:
- net GND: now also V157.1 (Via), V158.1 (Via), V159.1 (Via), V160.1 (Via), V161.1 (Via), V162.1 (Via), V163.1 (Via), V164.1 (Via), V165.1 (Via), V166.1 (Via)
- net GPIO5_0-EMC_A13: now reaches V198.1 (Via)
- net GPIO5_0-EMC_A13: now also V199.1 (Via)
- net MMC_VDD: now reaches V202.1 (Via)
- net MMC_VDD: now also V200.1 (Via), V201.1 (Via)
- net LTC3559_VCC: now reaches V203.1 (Via)
- net LTC3559_VCC: now also V204.1 (Via)
Changed lines of the file:
@@
-EESchema Schematic File Version 2  date 9/23/2011 8:04:30 AM
+EESchema Schematic File Version 2  date 9/24/2011 9:18:58 PM
 LIBS:power
 LIBS:device
@@
 Sheet 7 7
 Title "MicropendousX-LPC183x"
-Date "23 sep 2011"
+Date "25 sep 2011"
 Rev "1.0"
 Comp "Opendous Inc."
@@
 Comment4 "www.MicropendousX.org"
 $EndDescr
+Text GLabel 6900 2600 0    40   Input ~ 0
+GPIO5_0-EMC_A13
+Text GLabel 6900 2700 0    40   Input ~ 0
+GPIO5_0-EMC_A13
+Text GLabel 6900 2800 0    40   Input ~ 0
+MMC_VDD
+Text GLabel 6900 2900 0    40   Input ~ 0
+MMC_VDD
+Text GLabel 6900 3000 0    40   Input ~ 0
+MMC_VDD
+Text GLabel 6900 3100 0    40   Input ~ 0
+LTC3559_VCC
+Text GLabel 6900 3200 0    40   Input ~ 0
+LTC3559_VCC
+$Comp
+L GND #PWR0139
+U 1 1 4E7E51E9
+P 4500 6450
+F 0 "#PWR0139" H 4500 6450 30  0001 C CNN
+F 1 "GND" H 4500 6380 30  0001 C CNN
+	1    4500 6450
+	1    0    0    -1
+$EndComp
+Connection ~ 4650 6000
+Connection ~ 4650 6200
+Connection ~ 4650 6400
+Connection ~ 4650 6600
+Wire Wire Line
+	4650 6300 4500 6300
+Wire Wire Line
+	4500 6300 4500 6450
+Connection ~ 4650 6500
+Connection ~ 4650 6300
+Connection ~ 4650 6100
+Wire Wire Line
+	4650 5800 4650 6700
+Connection ~ 4650 5900
 Text GLabel 11000 650  0    40   Input ~ 0
 ADC1_1
@@
 Connection ~ 6900 1000
 $Comp
-L VBUS #PWR0139
+L VBUS #PWR0140
 U 1 1 4E771EB8
 P 10950 1350
-F 0 "#PWR0139" H 10950 1450 30  0001 C CNN
+F 0 "#PWR0140" H 10950 1450 30  0001 C CNN
 F 1 "VBUS" V 10950 1500 30  0000 C CNN
 	1    10950 1350
@@
 I2C1_SCL-U3_RXD
 $Comp
-L GND #PWR0140
+L GND #PWR0141
 U 1 1 4E76CD8A
 P 2300 5250
-F 0 "#PWR0140" H 2300 5250 30  0001 C CNN
+F 0 "#PWR0141" H 2300 5250 30  0001 C CNN
 F 1 "GND" H 2300 5180 30  0001 C CNN
 	1    2300 5250
@@
 $EndComp
 $Comp
-L GND #PWR0141
+L GND #PWR0142
 U 1 1 4E76CCD0
 P 2300 6850
-F 0 "#PWR0141" H 2300 6850 30  0001 C CNN
+F 0 "#PWR0142" H 2300 6850 30  0001 C CNN
 F 1 "GND" H 2300 6780 30  0001 C CNN
 	1    2300 6850
@@
 $EndComp
 $Comp
-L +BATT #PWR0142
+L +BATT #PWR0143
 U 1 1 4E76C805
 P 6700 700
-F 0 "#PWR0142" H 6700 650 20  0001 C CNN
+F 0 "#PWR0143" H 6700 650 20  0001 C CNN
 F 1 "+BATT" H 6700 800 30  0000 C CNN
 	1    6700 700
@@
 SSP1_SSEL
 $Comp
-L 6V0 #PWR0143
+L 6V0 #PWR0144
 U 1 1 4E766648
 P 10900 4050
-F 0 "#PWR0143" H 10900 4190 20  0001 C CNN
+F 0 "#PWR0144" H 10900 4190 20  0001 C CNN
 F 1 "6V0" V 10900 4200 30  0000 C CNN
 	1    10900 4050
@@
 $EndComp
 $Comp
-L GND #PWR0144
+L GND #PWR0145
 U 1 1 4E74194B
 P 10850 4800
-F 0 "#PWR0144" H 10850 4800 30  0001 C CNN
+F 0 "#PWR0145" H 10850 4800 30  0001 C CNN
 F 1 "GND" H 10850 4730 30  0001 C CNN
 	1    10850 4800
@@
 USB0_DM
 $Comp
-L VDDIO_3V3 #PWR0145
+L VDDIO_3V3 #PWR0146
 U 1 1 4E49585F
 P 6650 4100
-F 0 "#PWR0145" H 6650 4200 30  0001 C CNN
+F 0 "#PWR0146" H 6650 4200 30  0001 C CNN
 F 1 "VDDIO_3V3" H 6650 4200 30  0000 C CNN
 	1    6650 4100
@@
 $EndComp
 $Comp
-L VDD3V3 #PWR0146
+L VDD3V3 #PWR0147
 U 1 1 4E49554D
 P 6750 5700
-F 0 "#PWR0146" H 6750 5800 30  0001 C CNN
+F 0 "#PWR0147" H 6750 5800 30  0001 C CNN
 F 1 "VDD3V3" H 6750 5800 30  0000 C CNN
 	1    6750 5700
@@
 $EndComp
 $Comp
-L GNDPWR #PWR0147
+L GNDPWR #PWR0148
 U 1 1 4E24500E
 P 8850 5500
-F 0 "#PWR0147" H 8850 5550 40  0001 C CNN
+F 0 "#PWR0148" H 8850 5550 40  0001 C CNN
 F 1 "GNDPWR" H 8850 5420 40  0000 C CNN
 	1    8850 5500
@@
 $EndComp
 $Comp
-L VSYS #PWR0148
+L VSYS #PWR0149
 U 1 1 4E24421B
 P 10850 6050
-F 0 "#PWR0148" H 10850 6150 30  0001 C CNN
+F 0 "#PWR0149" H 10850 6150 30  0001 C CNN
 F 1 "VSYS" H 10850 6150 30  0000 C CNN
 	1    10850 6050
@@
 $EndComp
 $Comp
-L 5V0 #PWR0149
+L 5V0 #PWR0150
 U 1 1 4E244116
 P 10850 6350
-F 0 "#PWR0149" H 10850 6450 30  0001 C CNN
+F 0 "#PWR0150" H 10850 6450 30  0001 C CNN
 F 1 "5V0" H 10850 6450 30  0000 C CNN
 	1    10850 6350
@@
 $EndComp
 $Comp
-L VDDIO_3V3 #PWR0150
+L VDDIO_3V3 #PWR0151
 U 1 1 4E2437D2
 P 2200 3900
-F 0 "#PWR0150" H 2200 4000 30  0001 C CNN
+F 0 "#PWR0151" H 2200 4000 30  0001 C CNN
 F 1 "VDDIO_3V3" H 2200 4000 30  0000 C CNN
 	1    2200 3900
@@
 $EndComp
 $Comp
-L GND #PWR0151
+L GND #PWR0152
 U 1 1 4E24344B
 P 4500 7450
-F 0 "#PWR0151" H 4500 7450 30  0001 C CNN
+F 0 "#PWR0152" H 4500 7450 30  0001 C CNN
 F 1 "GND" H 4500 7380 30  0001 C CNN
 	1    4500 7450
@@
 $EndComp
 $Comp
-L VBUS #PWR0152
+L VBUS #PWR0153
 U 1 1 4E2423A0
 P 2200 6500
-F 0 "#PWR0152" H 2200 6600 30  0001 C CNN
+F 0 "#PWR0153" H 2200 6600 30  0001 C CNN
 F 1 "VBUS" H 2200 6600 30  0000 C CNN
 	1    2200 6500
@@
 GND_microAB
 $Comp
-L GND #PWR0153
+L GND #PWR0154
 U 1 1 4E241B4C
 P 2300 1450
-F 0 "#PWR0153" H 2300 1450 30  0001 C CNN
+F 0 "#PWR0154" H 2300 1450 30  0001 C CNN
 F 1 "GND" H 2300 1380 30  0001 C CNN
 	1    2300 1450

Commit message: Updated LPC183x Hardware Design
Parts:
- added V70, V71, V72, V73, V74, V75, V76, V77, V78, V79, V80, V81, V82, V83, V84, V85, V86, V87, V88, V89: VIA, symbol VIA
Connections:
- net VSYS is gone; now on net GND: V353.1 (Via), V354.1 (Via), V355.1 (Via)
- net 5V0: no longer V356.1 (Via), V358.1 (Via)
- net GND: now also V348.1 (Via), V349.1 (Via), V350.1 (Via), V351.1 (Via), V356.1 (Via), V358.1 (Via)
- net GNDPWR: now also V129.1 (Via), V130.1 (Via), V131.1 (Via), V132.1 (Via), V133.1 (Via), V134.1 (Via), V135.1 (Via), V136.1 (Via), V137.1 (Via), V138.1 (Via), V139.1 (Via), V140.1 (Via), V141.1 (Via), V142.1 (Via), V143.1 (Via), V144.1 (Via)
- net GPIO5_2: now also V151.1 (Via), V152.1 (Via)
- net VDD33: now also V205.1 (Via)
- net VDDIO_3V3: no longer V205.1 (Via)
- net MMC_CLK: now reaches V146.1 (Via)
- net MMC_CLK: now also V145.1 (Via)
- net SSP1_MISO: now reaches V148.1 (Via)
- net SSP1_MISO: now also V147.1 (Via)
- net SSP1_MOSI: now reaches V149.1 (Via)
- net SSP1_MOSI: now also V150.1 (Via)
- net TX0: now reaches V196.1 (Via)
- net EMC_A07: now reaches V195.1 (Via)
- net EMC_A07: now also V194.1 (Via)
- net TX1: now reaches V197.1 (Via)
- net nRESET: now reaches V188.1 (Via)
- net ~RESET~: now reaches V187.1 (Via)
- net ~RESET~: now also V186.1 (Via), V189.1 (Via)
- net EMC_A05: now reaches V190.1 (Via)
- net EMC_A05: now also V191.1 (Via)
- net EMC_A06: now reaches V193.1 (Via)
- net EMC_A06: now also V192.1 (Via)
- net ADC0_0-DAC: now reaches V184.1 (Via)
- net ADC0_0-DAC: now also V185.1 (Via)
- net 3V3: now reaches V352.1 (Via)
- new net EMC_D02-MMC_DAT0: V80.1 (Via), V81.1 (Via)
- new net EMC_D03-MMC_DAT1: V78.1 (Via), V79.1 (Via)
- new net EMC_D04-MMC_DAT2: V76.1 (Via), V77.1 (Via)
- new net EMC_D05-MMC_DAT3: V74.1 (Via), V75.1 (Via)
- new net EMC_D06-MMC_CD: V72.1 (Via), V73.1 (Via)
- new net GPIO0_11: V70.1 (Via), V71.1 (Via)
- new net ~EMC_WE~-MMC_CMD: V82.1 (Via), V83.1 (Via)
Other:
- moved on the sheet: V129, V130, V131, V132, V133, V134, V135, V136, V137, V138, V139, V140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

Commit message: Updated LPC183x Hardware Design
Parts:
- added V100, V101, V102, V103, V104, V105, V106, V107, V108, V109, V110, V111, V112, V113, V114, V115, V116, V117, V118, V119, V90, V91, V92, V93, V94, V95, V96, V97, V98, V99: VIA, symbol VIA
Connections:
- net EMC_A05: now also V102.1 (Via)
- net EMC_A06: now also V103.1 (Via)
- net EMC_A07: now also V104.1 (Via)
- net GND: now also V153.1 (Via), V154.1 (Via), V155.1 (Via), V156.1 (Via)
- net GPIO0_12: now also V93.1 (Via)
- net TX0: now also V96.1 (Via)
- net TX1: now also V97.1 (Via)
- net U2_RXD-GPIO0_3: now also V94.1 (Via)
- net U2_TXD-GPIO0_2: now also V95.1 (Via)
- net ~EMC_WE~-MMC_CMD: now also V297.1 (Via), V98.1 (Via)
- net EMC_D07: now reaches V89.1 (Via)
- net EMC_D07: now also V88.1 (Via)
- net EMC_D00: now reaches V87.1 (Via)
- net ~EMC_OE~: now reaches V86.1 (Via)
- net EMC_D01: now reaches V84.1 (Via)
- net ~EMC_CS0~: now reaches V85.1 (Via)
- net ~EMC_CS0~: now also V105.1 (Via)
- new net EMC_A02: V99.1 (Via)
- new net EMC_A03: V100.1 (Via)
- new net EMC_A04: V101.1 (Via)
- new net GPIO0_13: V92.1 (Via)
- new net I2C0_SCL: V90.1 (Via)
- new net I2C0_SDA: V91.1 (Via)
