File: MicropendousX/Hardware/MicropendousX-LPC183x/MicropendousX-LPC183x-Vias.sch (KiCad schematic (older format))
At the start: 347 parts

Commit message: Updated LPC183x Hardware Design
Parts:
- added V120, V121, V122, V123, V124, V125, V126, V127, V128, V342, V343, V359, V360, V361, V362, V363, V364, V365, V366, V367, V368, V369, V370, V371, V372, V373, V374, V375, V376, V377: VIA, symbol VIA
Connections:
- net 6V0 is gone; now on net GND: V332.1 (Via)
- net CLKOUT-I2S1_RX_SCK: now also V113.1 (Via)
- net EMC_A02: now also V108.1 (Via), V109.1 (Via)
- net EMC_A03: now also V194.1 (Via)
- net EMC_A04: now also V104.1 (Via)
- net EMC_A07: no longer V104.1 (Via), V194.1 (Via)
- net EMC_D00: now also V119.1 (Via), V120.1 (Via)
- net EMC_D01: now also V115.1 (Via)
- net EMC_D03-MMC_DAT1: now also V127.1 (Via)
- net EMC_D04-MMC_DAT2: now also V128.1 (Via)
- net EMC_D05-MMC_DAT3: now also V342.1 (Via)
- net EMC_D06-MMC_CD: now also V126.1 (Via)
- net GND: now also V371.1 (Via), V372.1 (Via), V373.1 (Via), V374.1 (Via), V375.1 (Via), V376.1 (Via), V377.1 (Via)
- net GPIO3_7: now also V300.1 (Via), V311.1 (Via); no longer V314.1 (Via)
- net GPIO5_2: now also V314.1 (Via); no longer V300.1 (Via), V311.1 (Via)
- net SPIFI_SIO2-I2S1_RX_WS: now also V116.1 (Via)
- net ~EMC_CS0~: now also V114.1 (Via)
- net ~EMC_OE~: now also V107.1 (Via)
- net GPIO3_5: now reaches V112.1 (Via)
- net GPIO3_5: now also V121.1 (Via), V122.1 (Via)
- net I2S0_TX_SCK: now reaches V111.1 (Via)
- net I2S0_TX_SCK: now also V110.1 (Via)
- net SPIFI_SIO3-I2S1_RX_SDA: now reaches V118.1 (Via)
- net SPIFI_SIO3-I2S1_RX_SDA: now also V117.1 (Via)
- net EMC_A00: now reaches V106.1 (Via)
- net EMC_A00: now also V125.1 (Via)
- new net EMC_A08: V123.1 (Via), V124.1 (Via)
Other:
- moved on the sheet: V100, V101, V102, V103, V104, V105, V106, V107, V108, V109, V110, V111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

Commit message: Updated LPC183x Hardware Design
Connections:
- net CLKOUT-I2S1_RX_SCK: now also V360.1 (Via)
- net EMC_D00: now also V343.1 (Via)
- net GND: now also V368.1 (Via), V369.1 (Via), V370.1 (Via)
- net SPIFI_SCK-CGU_OUT1: now also V359.1 (Via)

Commit message: Updated LPC183x Hardware Design
Parts:
- removed V192, V213, V231: VIA, symbol VIA
- added V378, V379, V381, V382, V384, V385, V386, V387: VIA, symbol VIA
Connections:
- net GND_microAB is gone; now on net GND: V68.1 (Via), V69.1 (Via)
- net EMC_A02: no longer V99.1 (Via)
- net EMC_A05: no longer V102.1 (Via)
- net EMC_A06: no longer V103.1 (Via)
- net EMC_D00: no longer V119.1 (Via)
- net EMC_D02-MMC_DAT0: now also V361.1 (Via), V362.1 (Via)
- net EMC_D07: now also V365.1 (Via)
- net GND: now also V102.1 (Via), V103.1 (Via), V119.1 (Via), V301.1 (Via), V366.1 (Via), V367.1 (Via), V95.1 (Via), V96.1 (Via), V97.1 (Via), V99.1 (Via)
- net GPIO0_12: now also V386.1 (Via)
- net GPIO3_7: no longer V301.1 (Via)
- net I2C0_SCL: now also V363.1 (Via)
- net I2C0_SDA: now also V364.1 (Via)
- net SSP1_MISO: now also V379.1 (Via)
- net SSP1_MOSI: now also V384.1 (Via)
- net SSP1_SCK: now also V378.1 (Via), V382.1 (Via)
- net SSP1_SSEL: now also V381.1 (Via), V385.1 (Via)
- net TX0: no longer V96.1 (Via)
- net TX1: no longer V97.1 (Via)
- net U2_RXD-GPIO0_3: now also V387.1 (Via)
- net U2_TXD-GPIO0_2: no longer V95.1 (Via)
Other:
- moved on the sheet: V100, V101, V102, V103, V104, V105, V106, V107, V108, V109, V110, V111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
