File: MicropendousX/Hardware/MicropendousX-LPC183x/MicropendousX-LPC183x-Opennect_Connector.sch (KiCad schematic (older format))
At the start: 25 parts, among them IC1 LPC183X, IC3 74CBTLV3257, IC4 3157, IC8 5V_REG, IC9 XC622x, J1 DC_POWER_JACK, U2 Opennect-Analog-ADC_3V3-x2, U9 Opennect-Controller-SingleEnd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

Commit message: Updated LPC183x Hardware Design
Connections:
- net labels added: 6V0
- net labels removed: DC_VIN
Other:
- note added: "SN74LVC1G3157 is a bidirectional analog switch"
- note added: "SPIFIx pins from\nSheet 5 - System"
- note removed: "From Sheet 5 - System"
- note removed: "SN74LVC1G3157 is an analog switch with 0.5ns Tpd"
Changed lines of the file:
@@
-EESchema Schematic File Version 2  date 9/18/2011 3:49:57 PM
+EESchema Schematic File Version 2  date 9/18/2011 8:03:49 PM
 LIBS:power
 LIBS:device
@@
 Sheet 2 7
 Title "MicropendousX-LPC183x"
-Date "18 sep 2011"
+Date "19 sep 2011"
 Rev "1.0"
 Comp "Opendous Inc."
@@
 Comment4 "www.MicropendousX.org"
 $EndDescr
+$Comp
+L 6V0 #PWR01
+U 1 1 4E76663C
+P 8900 6150
+F 0 "#PWR01" H 8900 6290 20  0001 C CNN
+F 1 "6V0" H 8900 6260 30  0000 C CNN
+	1    8900 6150
+	1    0    0    -1
+$EndComp
+$Comp
+L 6V0 #PWR02
+U 1 1 4E76661F
+P 10050 2450
+F 0 "#PWR02" H 10050 2590 20  0001 C CNN
+F 1 "6V0" V 10050 2600 30  0000 C CNN
+	1    10050 2450
+	0    1    1    0
+$EndComp
+$Comp
+L 6V0 #PWR03
+U 1 1 4E766619
+P 8500 1500
+F 0 "#PWR03" H 8500 1640 20  0001 C CNN
+F 1 "6V0" H 8500 1610 30  0000 C CNN
+	1    8500 1500
+	1    0    0    -1
+$EndComp
 Text Notes 9125 1350 0    40   ~ 0
 1117
@@
 SN74LVC1G
 Text Notes 5650 6150 0    40   ~ 0
-SN74LVC1G3157 is an analog switch with 0.5ns Tpd
+SN74LVC1G3157 is a bidirectional analog switch
 Text Notes 7900 650  0    60   ~ 0
 Full compatibility with the Opennect Specification\nrequires running the system from DC Power.\nD4 enables system 3V3 rail to partially power Opennect\nConnector to allow use of Opennect Modules that only\nrequire 3V3 rail when running off Li-Ion or USB.
@@
 $EndComp
 $Comp
-L 3V3 #PWR01
+L 3V3 #PWR04
 U 1 1 4E763CB1
 P 10750 1200
-F 0 "#PWR01" H 10750 1300 40  0001 C CNN
+F 0 "#PWR04" H 10750 1300 40  0001 C CNN
 F 1 "3V3" H 10750 1325 30  0000 C CNN
 	1    10750 1200
@@
 $EndComp
 $Comp
-L VDDIO_3V3 #PWR02
+L VDDIO_3V3 #PWR05
 U 1 1 4E763CAC
 P 10150 1200
-F 0 "#PWR02" H 10150 1300 30  0001 C CNN
+F 0 "#PWR05" H 10150 1300 30  0001 C CNN
 F 1 "VDDIO_3V3" H 10150 1300 30  0000 C CNN
 	1    10150 1200
@@
 $EndComp
 $Comp
-L GND #PWR03
+L GND #PWR06
 U 1 1 4E763C6F
 P 10450 1900
-F 0 "#PWR03" H 10450 1900 30  0001 C CNN
+F 0 "#PWR06" H 10450 1900 30  0001 C CNN
 F 1 "GND" H 10450 1830 30  0001 C CNN
 	1    10450 1900
@@
 $EndComp
 $Comp
-L GND #PWR04
+L GND #PWR07
 U 1 1 4E763C6C
 P 10950 1900
-F 0 "#PWR04" H 10950 1900 30  0001 C CNN
+F 0 "#PWR07" H 10950 1900 30  0001 C CNN
 F 1 "GND" H 10950 1830 30  0001 C CNN
 	1    10950 1900
@@
 $EndComp
 $Comp
-L 3V3 #PWR05
+L 3V3 #PWR08
 U 1 1 4E763C42
 P 10950 1500
-F 0 "#PWR05" H 10950 1600 40  0001 C CNN
+F 0 "#PWR08" H 10950 1600 40  0001 C CNN
 F 1 "3V3" H 10950 1625 30  0000 C CNN
 	1    10950 1500
@@
 $EndComp
 $Comp
-L 3V3 #PWR06
+L 3V3 #PWR09
 U 1 1 4E763C2A
 P 9300 6150
-F 0 "#PWR06" H 9300 6250 40  0001 C CNN
+F 0 "#PWR09" H 9300 6250 40  0001 C CNN
 F 1 "3V3" H 9300 6275 30  0000 C CNN
 	1    9300 6150
@@
 MMC_CLK used\nin Sheet 1 - EMI
 $Comp
-L VDDIO_3V3 #PWR07
+L VDDIO_3V3 #PWR010
 U 1 1 4E76399F
 P 5800 3450
-F 0 "#PWR07" H 5800 3550 30  0001 C CNN
+F 0 "#PWR010" H 5800 3550 30  0001 C CNN
 F 1 "VDDIO_3V3" H 5800 3550 30  0000 C CNN
 	1    5800 3450
@@
 NoConn ~ 3700 3800
 $Comp
-L GND #PWR08
+L GND #PWR011
 U 1 1 4E763086
 P 9200 1900
-F 0 "#PWR08" H 9200 1900 30  0001 C CNN
+F 0 "#PWR011" H 9200 1900 30  0001 C CNN
 F 1 "GND" H 9200 1830 30  0001 C CNN
 	1    9200 1900
@@
 $EndComp
 $Comp
-L GND #PWR09
+L GND #PWR012
 U 1 1 4E763074
 P 9750 1900
-F 0 "#PWR09" H 9750 1900 30  0001 C CNN
+F 0 "#PWR012" H 9750 1900 30  0001 C CNN
 F 1 "GND" H 9750 1830 30  0001 C CNN
 	1    9750 1900
@@
 $EndComp
 $Comp
-L 5V0 #PWR010
+L 5V0 #PWR013
 U 1 1 4E762F51
 P 9750 1500
-F 0 "#PWR010" H 9750 1600 30  0001 C CNN
+F 0 "#PWR013" H 9750 1600 30  0001 C CNN
 F 1 "5V0" H 9750 1600 30  0000 C CNN
 	1    9750 1500
-	1    0    0    -1
-$EndComp
-$Comp
-L DC_VIN #PWR011
-U 1 1 4E762F50
-P 8500 1500
-F 0 "#PWR011" H 8500 1600 30  0001 C CNN
-F 1 "DC_VIN" H 8500 1600 30  0000 C CNN
-	1    8500 1500
 	1    0    0    -1
 $EndComp
@@
 74CBTLV3257_nOE
 $Comp
-L GND #PWR012
+L GND #PWR014
 U 1 1 4E7625CD
 P 7500 4050
-F 0 "#PWR012" H 7500 4050 30  0001 C CNN
+F 0 "#PWR014" H 7500 4050 30  0001 C CNN
 F 1 "GND" H 7500 3980 30  0001 C CNN
 	1    7500 4050
@@
 Text Notes 4025 4400 0    40   ~ 0
 Used in Sheet 6 -\nPower Supply
-Text Notes 5450 5950 0    40   ~ 0
-From Sheet 5 - System
-$Comp
-L GND #PWR013
+Text Notes 4800 4450 0    40   ~ 0
+SPIFIx pins from\nSheet 5 - System
+$Comp
+L GND #PWR015
 U 1 1 4E7415E5
 P 9700 6450
-F 0 "#PWR013" H 9700 6450 30  0001 C CNN
+F 0 "#PWR015" H 9700 6450 30  0001 C CNN
 F 1 "GND" H 9700 6380 30  0001 C CNN
 	1    9700 6450
@@
 $EndComp
 $Comp
-L VDDIO_3V3 #PWR014
+L VDDIO_3V3 #PWR016
 U 1 1 4E74153C
 P 6100 5050
-F 0 "#PWR014" H 6100 5150 30  0001 C CNN
+F 0 "#PWR016" H 6100 5150 30  0001 C CNN
 F 1 "VDDIO_3V3" H 6100 5150 30  0000 C CNN
 	1    6100 5050
@@
 $EndComp
 $Comp
-L GND #PWR015
+L GND #PWR017
 U 1 1 4E74153B
 P 6100 5350
-F 0 "#PWR015" H 6100 5350 30  0001 C CNN
+F 0 "#PWR017" H 6100 5350 30  0001 C CNN
 F 1 "GND" H 6100 5280 30  0001 C CNN
 	1    6100 5350
@@
 $EndComp
 $Comp
-L GND #PWR016
+L GND #PWR018
 U 1 1 4E741516
 P 7000 5350
-F 0 "#PWR016" H 7000 5350 30  0001 C CNN
+F 0 "#PWR018" H 7000 5350 30  0001 C CNN
 F 1 "GND" H 7000 5280 30  0001 C CNN
 	1    7000 5350
@@
 $EndComp
 $Comp
-L VDDIO_3V3 #PWR017
+L VDDIO_3V3 #PWR019
 U 1 1 4E74150E
 P 7000 5050
-F 0 "#PWR017" H 7000 5150 30  0001 C CNN
+F 0 "#PWR019" H 7000 5150 30  0001 C CNN
 F 1 "VDDIO_3V3" H 7000 5150 30  0000 C CNN
 	1    7000 5050
@@
 GPIO0_13-ENET_TXD0
 $Comp
-L GND #PWR018
+L GND #PWR020
 U 1 1 4E7402AE
 P 6550 5000
-F 0 "#PWR018" H 6550 5000 30  0001 C CNN
+F 0 "#PWR020" H 6550 5000 30  0001 C CNN
 F 1 "GND" H 6550 4930 30  0001 C CNN
 	1    6550 5000
@@
 $EndComp
 $Comp
-L GND #PWR019
+L GND #PWR021
 U 1 1 4E7402AA
 P 6650 6000
-F 0 "#PWR019" H 6650 6000 30  0001 C CNN
+F 0 "#PWR021" H 6650 6000 30  0001 C CNN
 F 1 "GND" H 6650 5930 30  0001 C CNN
 	1    6650 6000
@@
 CLKOUT-I2S1_RX_SCK
 $Comp
-L VDDIO_3V3 #PWR020
+L VDDIO_3V3 #PWR022
 U 1 1 4E73E025
 P 6650 5450
-F 0 "#PWR020" H 6650 5550 30  0001 C CNN
+F 0 "#PWR022" H 6650 5550 30  0001 C CNN
 F 1 "VDDIO_3V3" H 6650 5550 30  0000 C CNN
 	1    6650 5450
@@
 TX_WS
 $Comp
-L VDDIO_3V3 #PWR021
+L VDDIO_3V3 #PWR023
 U 1 1 4E73D4C6
 P 6550 3450
-F 0 "#PWR021" H 6550 3550 30  0001 C CNN
+F 0 "#PWR023" H 6550 3550 30  0001 C CNN
 F 1 "VDDIO_3V3" H 6550 3550 30  0000 C CNN
 	1    6550 3450
@@
 TX0
 $Comp
-L VSSA #PWR022
+L VSSA #PWR024
 U 1 1 4E73A195
 P 6500 7500
-F 0 "#PWR022" H 6500 7500 30  0001 C CNN
+F 0 "#PWR024" H 6500 7500 30  0001 C CNN
 F 1 "VSSA" H 6500 7425 30  0000 C CNN
 	1    6500 7500
@@
 $EndComp
 $Comp
-L VDDA #PWR023
+L VDDA #PWR025
 U 1 1 4E73A190
 P 6050 6850
-F 0 "#PWR023" H 6050 6950 30  0001 C CNN
+F 0 "#PWR025" H 6050 6950 30  0001 C CNN
 F 1 "VDDA" V 6050 7000 30  0000 C CNN
 	1    6050 6850
@@
 $EndComp
 $Comp
-L GNDPWR #PWR024
+L GNDPWR #PWR026
 U 1 1 4E73A13B
 P 6000 7500
-F 0 "#PWR024" H 6000 7550 40  0001 C CNN
+F 0 "#PWR026" H 6000 7550 40  0001 C CNN
 F 1 "GNDPWR" H 5995 7445 20  0000 C CNN
 	1    6000 7500
@@
 $EndComp
 $Comp
-L GND #PWR025
+L GND #PWR027
 U 1 1 4E4904B8
 P 8500 1800
-F 0 "#PWR025" H 8500 1800 30  0001 C CNN
+F 0 "#PWR027" H 8500 1800 30  0001 C CNN
 F 1 "GND" H 8500 1730 30  0001 C CNN
 	1    8500 1800
@@
 NoConn ~ 3700 3500
 $Comp
-L VDDIO_3V3 #PWR026
+L VDDIO_3V3 #PWR028
 U 1 1 4E23BF70
 P 4300 900
-F 0 "#PWR026" H 4300 1000 30  0001 C CNN
+F 0 "#PWR028" H 4300 1000 30  0001 C CNN
 F 1 "VDDIO_3V3" H 4300 1000 30  0000 C CNN
 	1    4300 900
@@
 $EndComp
 $Comp
-L GND #PWR027
+L GND #PWR029
 U 1 1 4E22B69E
 P 9100 6450
-F 0 "#PWR027" H 9100 6450 30  0001 C CNN
+F 0 "#PWR029" H 9100 6450 30  0001 C CNN
 F 1 "GND" H 9100 6380 30  0001 C CNN
 	1    9100 6450
@@
 $EndComp
 $Comp
-L DC_VIN #PWR028
-U 1 1 4E22B675
-P 8900 6150
-F 0 "#PWR028" H 8900 6250 30  0001 C CNN
-F 1 "DC_VIN" H 8900 6250 30  0000 C CNN
-	1    8900 6150
-	1    0    0    -1
-$EndComp
-$Comp
-L 5V0 #PWR029
+L 5V0 #PWR030
 U 1 1 4E22B673
 P 9100 6150
-F 0 "#PWR029" H 9100 6250 30  0001 C CNN
+F 0 "#PWR030" H 9100 6250 30  0001 C CNN
 F 1 "5V0" H 9100 6250 30  0000 C CNN
 	1    9100 6150
@@
 $EndComp
 $Comp
-L VDDIO_3V3 #PWR030
+L VDDIO_3V3 #PWR031
 U 1 1 4E22B670
 P 9700 6150
-F 0 "#PWR030" H 9700 6250 30  0001 C CNN
+F 0 "#PWR031" H 9700 6250 30  0001 C CNN
 F 1 "VDDIO_3V3" H 9700 6250 30  0000 C CNN
 	1    9700 6150
@@
 $EndComp
 $Comp
-L GND #PWR031
+L GND #PWR032
 U 1 1 4E22B627
 P 9350 5800
-F 0 "#PWR031" H 9350 5800 30  0001 C CNN
+F 0 "#PWR032" H 9350 5800 30  0001 C CNN
 F 1 "GND" H 9350 5730 30  0001 C CNN
 	1    9350 5800
@@
 GPIO3_5
 $Comp
-L VDDIO_3V3 #PWR032
+L VDDIO_3V3 #PWR033
 U 1 1 4E22B516
 P 8650 4000
-F 0 "#PWR032" H 8650 4100 30  0001 C CNN
+F 0 "#PWR033" H 8650 4100 30  0001 C CNN
 F 1 "VDDIO_3V3" V 8650 4200 30  0000 C CNN
 	1    8650 4000
@@
 $EndComp
 $Comp
-L VDD3V3 #PWR033
+L VDD3V3 #PWR034
 U 1 1 4E22B4E3
 P 8650 2400
-F 0 "#PWR033" H 8650 2500 30  0001 C CNN
+F 0 "#PWR034" H 8650 2500 30  0001 C CNN
 F 1 "VDD3V3" V 8650 2575 30  0000 C CNN
 	1    8650 2400
@@
 $EndComp
 $Comp
-L 5V0 #PWR034
+L 5V0 #PWR035
 U 1 1 4E22B4D4
 P 8650 2500
-F 0 "#PWR034" H 8650 2600 30  0001 C CNN
+F 0 "#PWR035" H 8650 2600 30  0001 C CNN
 F 1 "5V0" V 8650 2625 30  0000 C CNN
 	1    8650 2500
 	0    -1   -1   0
 $EndComp
-$Comp
-L DC_VIN #PWR035
-U 1 1 4E22B4C5
-P 10050 2450
-F 0 "#PWR035" H 10050 2550 30  0001 C CNN
-F 1 "DC_VIN" V 10050 2625 30  0000 C CNN
-	1    10050 2450
-	0    1    1    0
-$EndComp
 Text GLabel 8800 2800 0    40   BiDi ~ 0

Commit message: Updated LPC183x Hardware Design
Parts:
- IC8: value 5V_REG -> 1117-5
Connections:
- net labels added: GPIO0_12, GPIO0_13, GPIO5_0-EMC_A13, SSP1_MISO, SSP1_MOSI, SSP1_SCK, SSP1_SSEL, U2_RXD-GPIO0_3, U2_TXD-GPIO0_2, ~EMC_CS0~
- net labels removed: GPIO0_12-ENET_MDIO, GPIO0_13-ENET_TXD0, GPIO5_0-EMC_A13-ENET_MDC, SSP1_MISO-ENET_RXD1, SSP1_MOSI-ENET_TX_EN, SSP1_SCK-ENET_REF_CLK, SSP1_SSEL-ENET_TXD1, U2_RXD-GPIO0_3-ENET_RX_DV, U2_TXD-GPIO0_2-ENET_RXD0, VDD3V3, ~EMC_CS0~-MMC_POW
Other:
- note added: "ENET_MDC"
- note added: "ENET_MDIO"
- note added: "ENET_REF_CLK"
- note added: "ENET_RXD0"
- note added: "ENET_RXD1"
- note added: "ENET_RX_DV"
- note added: "ENET_TXD0"
- note added: "ENET_TXD1"
- note added: "ENET_TX_EN"
- note removed: "1117"

Commit message: Updated LPC183x Hardware Design
Parts:
- removed IC8: 1117-5, symbol REG_1084_RO252-3L_DPAK
- added C20: 4u7, symbol C_MINI
- added C6: 0u1, symbol C_MINI
- added IC8: AP7361ADJ, symbol AP7361_DFN
- added L4: FB, symbol L_MINI
- added R23: 247k, symbol R_MINI
- added R24: 47k, symbol R_MINI
- C12, C15: value 10u -> 4u7
Connections:
- net labels added: ADC_GND
- net labels removed: VSSA
- wire segments 102 -> 110
Other:
- note added: "10<ESR(mOhm)<300"
- moved on the sheet: C12, C16, J1

Commit message: Updated LPC183x Hardware Design
Parts:
- removed IC9: XC622x, symbol REGULATOR_SOT89-5_TOREX
- added IC9: AP7361, symbol AP7361_DFN
- added R25: 147k, symbol R_MINI
- added R26: 47k, symbol R_MINI
- C16: value 0u1 -> 4u7
- IC8: value AP7361ADJ -> AP7361
- J1: value DC_POWER_JACK -> DC_IN
Connections:
- net labels added: VDD3V3
- wire segments 110 -> 114
- no-connect marks 30 -> 36
Other:
- note added: "Full compatibility with the Opennect Specification\nrequires running the system from DC Power.\nD4 enables system 3V3 rail to partially power Opennect\nConnector when running off Li-Ion or USB to allow use\nof Opennect Modules that only require 3V3 rail."
- note removed: "Full compatibility with the Opennect Specification\nrequires running the system from DC Power.\nD4 enables system 3V3 rail to partially power Opennect\nConnector to allow use of Opennect Modules that only\nrequire 3V3 rail when running off Li-Ion or USB."
- moved on the sheet: C103, C104, C105, C106, C12, C15, C20, C7, IC8, J1, R23, R24

Commit message: Updated LPC183x Hardware Design
Changed lines of the file:
@@
-EESchema Schematic File Version 2  date 9/24/2011 9:18:58 PM
+EESchema Schematic File Version 2  date 9/25/2011 2:41:21 AM
 LIBS:power
 LIBS:device
@@
 Text Notes 10650 3625 0    40   ~ 0
 RX_SCK
+Text GLabel 6150 4550 0    40   BiDi ~ 0
+SPIFI_SIO3-I2S1_RX_SDA
 Text GLabel 6150 4350 0    40   BiDi ~ 0
-SPIFI_SIO3-I2S1_RX_SDA
-Text GLabel 6150 4550 0    40   BiDi ~ 0
 SPIFI_SIO2-I2S1_RX_WS
 NoConn ~ 3700 3600
@@
 $EndComp
 NoConn ~ 3700 6350
+Text Notes 7150 4425 0    40   ~ 0
+RX_WS
 Text Notes 7150 4625 0    40   ~ 0
-RX_WS
-Text Notes 7150 4425 0    40   ~ 0
 RX_SDA
+Text Notes 7150 4225 0    40   ~ 0
+TX_SDA
 Text Notes 7150 4025 0    40   ~ 0
-TX_SDA
-Text Notes 7150 4225 0    40   ~ 0
 TX_WS
 $Comp
@@
 	1    0    0    -1
 $EndComp
+Text GLabel 6950 4400 2    40   BiDi ~ 0
+RX1
 Text GLabel 6950 4600 2    40   BiDi ~ 0
-RX1
-Text GLabel 6950 4400 2    40   BiDi ~ 0
 RX0
 Text GLabel 9900 3900 2    40   Output ~ 0
@@
 Text GLabel 9900 4000 2    40   Output ~ 0
 RX1
+Text GLabel 6950 4200 2    40   BiDi ~ 0
+TX0
 Text GLabel 6950 4000 2    40   BiDi ~ 0
-TX0
-Text GLabel 6950 4200 2    40   BiDi ~ 0
 TX1
 Text GLabel 8800 3800 0    40   Input ~ 0
@@
 Text GLabel 4500 1350 2    40   BiDi ~ 0
 I2C0_SDA
+Text GLabel 6150 4150 0    40   Input ~ 0
+I2S0_TX_SDA
 Text GLabel 6150 3950 0    40   Input ~ 0
-I2S0_TX_SDA
-Text GLabel 6150 4150 0    40   Input ~ 0
 I2S0_TX_WS
 Text GLabel 3700 3300 2    40   Output ~ 0
@@
 Text GLabel 8800 4500 0    40   BiDi ~ 0
 EMC_A03
+Text GLabel 6150 4050 0    40   BiDi ~ 0
+EMC_A01
 Text GLabel 6150 4250 0    40   BiDi ~ 0
-EMC_A01
-Text GLabel 6150 4050 0    40   BiDi ~ 0
 EMC_A00
 Text GLabel 8800 4200 0    40   BiDi ~ 0
@@
 Text GLabel 9900 4300 2    40   BiDi ~ 0
 EMC_D03-MMC_DAT1
+Text GLabel 6150 4450 0    40   BiDi ~ 0
+EMC_D01
 Text GLabel 6150 4650 0    40   BiDi ~ 0
-EMC_D01
-Text GLabel 6150 4450 0    40   BiDi ~ 0
 EMC_D00
 $EndSCHEMATC

Commit message: Updated LPC183x Hardware Design
Other:
- note added: "Full compatibility with the Opennect Specification\nrequires running the system from DC Power.\nD4 enables system 3V3 rail to partially power Opennect\nConnector when running off Li-Ion or USB to allow use\nof Opennect Modules that only require 3.3V rail."
- note added: "Notes:\n - When GPIO3_5 is set to High (default), pins are routed\n for compatibility with Opennect-Controller-I2S. When\n it is set to Low pins are routed for compatibility with\n Opennect-Controller-SingleEnded-x4 Specification.\n - I2S0 used for TX and I2S1 used for RX"
- note removed: "Full compatibility with the Opennect Specification\nrequires running the system from DC Power.\nD4 enables system 3V3 rail to partially power Opennect\nConnector when running off Li-Ion or USB to allow use\nof Opennect Modules that only require 3V3 rail."
- note removed: "Notes:\n - When GPIO3_5 is set to High (default), pins are routed\n for compatibility with Opennect-Controller-I2S. When\n it is set to Low pins are routed for compatibility with\n Opennect-Controller-SingleEnded-x4 Specification."
Changed lines of the file:
@@
-EESchema Schematic File Version 2  date 9/25/2011 4:24:57 AM
+EESchema Schematic File Version 2  date 9/25/2011 6:49:29 PM
 LIBS:power
 LIBS:device
@@
 Comment4 "www.MicropendousX.org"
 $EndDescr
+Text Notes 7400 650  0    60   ~ 0
+Full compatibility with the Opennect Specification\nrequires running the system from DC Power.\nD4 enables system 3V3 rail to partially power Opennect\nConnector when running off Li-Ion or USB to allow use\nof Opennect Modules that only require 3.3V rail.
 Connection ~ 10600 1400
 Wire Wire Line
@@
 Text Notes 5650 6150 0    40   ~ 0
 SN74LVC1G3157 is a bidirectional analog switch
-Text Notes 7400 650  0    60   ~ 0
-Full compatibility with the Opennect Specification\nrequires running the system from DC Power.\nD4 enables system 3V3 rail to partially power Opennect\nConnector when running off Li-Ion or USB to allow use\nof Opennect Modules that only require 3V3 rail.
 $Comp
 L D_SCHOTTKY D4
@@
 	1    0    0    -1
 $EndComp
-Text Notes 4800 2900 0    60   ~ 0
-Notes:\n - When GPIO3_5 is set to High (default), pins are routed\n   for compatibility with Opennect-Controller-I2S.  When\n   it is set to Low pins are routed for compatibility with\n   Opennect-Controller-SingleEnded-x4 Specification.
+Text Notes 4800 2750 0    60   ~ 0
+Notes:\n - When GPIO3_5 is set to High (default), pins are routed\n   for compatibility with Opennect-Controller-I2S.  When\n   it is set to Low pins are routed for compatibility with\n   Opennect-Controller-SingleEnded-x4 Specification.\n - I2S0 used for TX and I2S1 used for RX
 Text GLabel 6150 5650 0    40   BiDi ~ 0
 GPIO3_5
