File: MicropendousX/Hardware/MicropendousX-LPC183x/MicropendousX-LPC183x-Opennect_Connector.sch (KiCad schematic (older format))
At the start: 32 parts, among them IC1 LPC183X, IC3 74CBTLV3257, IC4 3157, IC8 AP7361, IC9 AP7361, J1 DC_IN, U2 Opennect-Analog-ADC_3V3-x2, U9 Opennect-Controller-SingleEnd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

Commit message: Updated MicropendousX-LPC183x portable design with minor post-prototyping corrections.
Parts:
- C106: value 1u0 -> 0u1
- C43: value 0u1 -> 4u7
- R23: value 247k -> 249k
- R25: value 147k -> 249k
Other:
- note added: "SPIFI_SCK pin from\nSheet 5 - System"
Changed lines of the file:
@@
-EESchema Schematic File Version 2  date 9/26/2011 2:10:54 AM
+EESchema Schematic File Version 2  date 11/3/2011 5:56:20 AM
 LIBS:power
 LIBS:device
@@
 Sheet 2 7
 Title "MicropendousX-LPC183x"
-Date "26 sep 2011"
+Date "3 nov 2011"
 Rev "1.0"
 Comp "Opendous Inc."
@@
 Comment4 "www.MicropendousX.org"
 $EndDescr
+Text Notes 4800 5850 0    40   ~ 0
+SPIFI_SCK pin from\nSheet 5 - System
 Text Notes 7400 650  0    60   ~ 0
 Full compatibility with the Opennect Specification\nrequires running the system from DC Power.\nD4 enables system 3V3 rail to partially power Opennect\nConnector when running off Li-Ion or USB to allow use\nof Opennect Modules that only require 3.3V rail.
@@
 P 10400 1500
 F 0 "R25" V 10375 1550 25  0000 C CNN
-F 1 "147k" V 10425 1550 20  0000 C CNN
+F 1 "249k" V 10425 1550 20  0000 C CNN
 	1    10400 1500
 	0    1    1    0
@@
 P 8450 1500
 F 0 "R23" V 8425 1550 25  0000 C CNN
-F 1 "247k" V 8475 1550 20  0000 C CNN
+F 1 "249k" V 8475 1550 20  0000 C CNN
 	1    8450 1500
 	0    1    1    0
@@
 P 6100 5200
 F 0 "C43" V 6050 5250 30  0000 C CNN
-F 1 "0u1" V 6150 5250 25  0000 C CNN
+F 1 "4u7" V 6150 5250 25  0000 C CNN
 	1    6100 5200
 	0    1    1    0
@@
 P 8900 6250
 F 0 "C106" V 8850 6325 30  0000 C CNN
-F 1 "1u0" V 8950 6300 25  0000 C CNN
+F 1 "0u1" V 8950 6300 25  0000 C CNN
 	1    8900 6250
 	0    1    1    0
