File: MicropendousX/Hardware/MicropendousX-GPS/MicropendousX-LPC182x-GPS-EMI.sch (KiCad schematic (older format))
At the start: 11 parts, among them IC1 LPC182x, IC5 FDG6342L, U11 microSD

Commit message: Updated MicropendousX-LPC182x-GPS design.  PCB routing almost complete.
Parts:
- C118: value 10u -> 4u7
- IC5: value FDG6342L -> FDG
Connections:
- net labels added: P2_11-GPIO1_11, P2_2-GPIO5_2, P2_7-ISP
- net labels removed: P1_3-GPIO0_10
Other:
- note added: "6342L"
- note added: "R1-C1, R2 circuitry enables slow\nstartup to limit inrush current\nR1 >> 10*R2\nR1=47k, R2=2k2 ==> Ton=4us\nToff=R1*Co=47000*0.00000481=0.23s"
- note removed: "R1-C1, R2 circuitry enables slow\nstartup to limit inrush current\nR1 >> 10*R2\nR1=47k, R2=2k2 ==> Ton=4us\nToff=R1*Co=47000*0.00001011=0.48s"
- moved on the sheet: TP3
Changed lines of the file:
@@
-EESchema Schematic File Version 2  date 5/31/2012 10:34:44 PM
+EESchema Schematic File Version 2  date 6/8/2012 3:21:19 PM
 LIBS:power
 LIBS:device
@@
 LIBS:contrib
 LIBS:valves
-LIBS:opendous
-LIBS:Opennect_Schematic_Symbols_Library
 LIBS:MicropendousX-LPC182x-GPS-cache
 EELAYER 25  0
@@
 $Descr A4 11700 8267
 encoding utf-8
-Sheet 5 9
+Sheet 6 10
 Title "MicropendousX-LPC182x-GPS"
-Date "1 jun 2012"
+Date "8 jun 2012"
 Rev "1.0"
 Comp "Opendous Inc."
@@
 Comment4 "www.MicropendousX.org"
 $EndDescr
-Text GLabel 3850 3600 2    40   Input ~ 0
-P1_3-GPIO0_10
-Text Notes 4400 3625 0    40   ~ 0
+Text Label 3850 2100 0    20   ~ 0
+P2_7-ISP
+Wire Wire Line
+	3850 2100 4050 2100
+Wire Wire Line
+	9800 3500 9200 3500
+Connection ~ 7750 2650
+Wire Wire Line
+	7750 2650 7750 2700
+Wire Wire Line
+	7550 2900 7750 2900
+Wire Wire Line
+	8600 2600 8600 3450
+Connection ~ 9000 3450
+Wire Wire Line
+	9200 3500 9200 3450
+Wire Wire Line
+	9200 3450 8600 3450
+Wire Wire Line
+	10500 3800 10500 3700
+Wire Wire Line
+	10500 3700 10400 3700
+Connection ~ 8600 3450
+Connection ~ 7550 2650
+Wire Wire Line
+	7100 3150 7100 3100
+Wire Wire Line
+	7100 3350 7100 3400
+Wire Wire Line
+	6600 3050 6650 3050
+Wire Wire Line
+	6650 3050 6650 2900
+Wire Wire Line
+	6450 2550 6450 2600
+Wire Wire Line
+	6450 2800 6450 2850
+Wire Wire Line
+	6450 2600 6650 2600
+Connection ~ 6450 2600
+Wire Wire Line
+	7550 2700 7550 2600
+Connection ~ 8800 3450
+Connection ~ 8800 3650
+Wire Wire Line
+	8800 3650 8800 3700
+Wire Wire Line
+	8600 3650 9200 3650
+Wire Wire Line
+	9200 3650 9200 3600
+Connection ~ 9000 3650
+Wire Wire Line
+	8050 3000 8050 2950
+Wire Wire Line
+	8050 3200 7750 3200
+Wire Wire Line
+	7750 3200 7750 2900
+Connection ~ 7750 2900
+Connection ~ 8600 2650
+Wire Wire Line
+	7550 2650 8600 2650
+Wire Wire Line
+	9200 3600 9800 3600
+Text Notes 7065 2539 0    60   ~ 0
+6342L
+Text GLabel 3850 2300 2    40   Input ~ 0
+P2_2-GPIO5_2
+Text Notes 4350 2325 0    40   ~ 0
+Used in Position Sensors Sheet
+Text GLabel 3850 1400 2    40   Input ~ 0
+P2_11-GPIO1_11
+Text Notes 4450 1425 0    40   ~ 0
 Used in Power Supply Sheet
 Text Notes 4350 4025 0    40   ~ 0
@@
 Text Notes 4350 3725 0    40   ~ 0
 Used in Position Sensors Sheet
-Wire Wire Line
-	9800 3600 9200 3600
-Wire Wire Line
-	7550 2650 8600 2650
-Connection ~ 8600 2650
-Connection ~ 7750 2900
-Wire Wire Line
-	7750 3200 7750 2900
-Wire Wire Line
-	7750 3200 8050 3200
-Wire Wire Line
-	8050 3000 8050 2950
-Connection ~ 9000 3650
-Wire Wire Line
-	9200 3600 9200 3650
-Wire Wire Line
-	9200 3650 8600 3650
-Wire Wire Line
-	8800 3650 8800 3700
-Connection ~ 8800 3650
-Connection ~ 8800 3450
-Wire Wire Line
-	7550 2700 7550 2600
-Connection ~ 6450 2600
-Wire Wire Line
-	6650 2600 6450 2600
-Wire Wire Line
-	6450 2800 6450 2850
-Wire Wire Line
-	6450 2600 6450 2550
-Wire Wire Line
-	6650 2900 6650 3050
-Wire Wire Line
-	6650 3050 6600 3050
-Wire Wire Line
-	7100 3350 7100 3400
-Wire Wire Line
-	7100 3150 7100 3100
-Connection ~ 7550 2650
-Connection ~ 8600 3450
-Wire Wire Line
-	10400 3700 10500 3700
-Wire Wire Line
-	10500 3700 10500 3800
-Wire Wire Line
-	9200 3450 8600 3450
-Wire Wire Line
-	9200 3450 9200 3500
-Connection ~ 9000 3450
-Wire Wire Line
-	3850 2100 3950 2100
-Wire Wire Line
-	8600 3450 8600 2600
-Wire Wire Line
-	7750 2900 7550 2900
-Wire Wire Line
-	7750 2650 7750 2700
-Connection ~ 7750 2650
-Wire Wire Line
-	9200 3500 9800 3500
 Text GLabel 9800 3400 0    40   Output ~ 0
 CLK2-MMC_CLK
@@
 Co = 10.11uF
 $Comp
-L VDD_MMC #PWR?
+L VDD_MMC #PWR0116
 U 1 1 4FC6B70B
 P 8600 2600
-F 0 "#PWR?" H 8600 2700 30  0001 C CNN
+F 0 "#PWR0116" H 8600 2700 30  0001 C CNN
 F 1 "VDD_MMC" H 8600 2700 30  0000 C CNN
 	1    8600 2600
@@
 $EndComp
 $Comp
-L VDDIO_3V3 #PWR?
+L VDDIO_3V3 #PWR0117
 U 1 1 4FC6B4E7
 P 8050 2950
-F 0 "#PWR?" H 8050 3050 30  0001 C CNN
+F 0 "#PWR0117" H 8050 3050 30  0001 C CNN
 F 1 "VDDIO_3V3" H 8050 3050 30  0000 C CNN
 	1    8050 2950
@@
 $EndComp
 $Comp
-L VDDIO_3V3 #PWR23
+L VDDIO_3V3 #PWR0118
 U 1 1 4FC698FB
 P 6450 2550
-F 0 "#PWR23" H 6450 2650 30  0001 C CNN
+F 0 "#PWR0118" H 6450 2650 30  0001 C CNN
 F 1 "VDDIO_3V3" H 6450 2650 30  0000 C CNN
 	1    6450 2550
@@
 $EndComp
 Text Notes 7250 3300 0    40   ~ 0
-R1-C1, R2 circuitry enables slow\nstartup to limit inrush current\nR1 >> 10*R2\nR1=47k, R2=2k2 ==> Ton=4us\nToff=R1*Co=47000*0.00001011=0.48s
+R1-C1, R2 circuitry enables slow\nstartup to limit inrush current\nR1 >> 10*R2\nR1=47k, R2=2k2 ==> Ton=4us\nToff=R1*Co=47000*0.00000481=0.23s
 Text Notes 4350 2525 0    40   ~ 0
 Used in Position Sensors Sheet
@@
 Text GLabel 3850 2000 2    40   BiDi ~ 0
 P2_8
-Text Notes 4325 2125 0    40   ~ 0
+Text Notes 4425 2125 0    40   ~ 0
 P2_7 has weak internal pull-up to disable ISP
 Text GLabel 3850 2500 2    40   Output ~ 0
@@
 L CONN_1 TP3
 U 1 1 4FBDF820
-P 4100 2100
-F 0 "TP3" H 4150 2100 40  0000 L CNN
-F 1 "ISP" H 4100 2155 30  0001 C CNN
-	1    4100 2100
+P 4200 2100
+F 0 "TP3" H 4250 2100 40  0000 L CNN
+F 1 "ISP" H 4200 2155 30  0001 C CNN
+	1    4200 2100
 	1    0    0    -1
 $EndComp
@@
 Hirose DM3D-SF
 $Comp
-L GND #PWR28
+L GND #PWR0119
 U 1 1 4FBDE98A
 P 10500 3800
-F 0 "#PWR28" H 10500 3800 30  0001 C CNN
+F 0 "#PWR0119" H 10500 3800 30  0001 C CNN
 F 1 "GND" H 10500 3730 30  0001 C CNN
 	1    10500 3800
@@
 Notes:\n-
 $Comp
-L GND #PWR27
+L GND #PWR0120
 U 1 1 4E23313A
 P 8800 3700
-F 0 "#PWR27" H 8800 3700 30  0001 C CNN
+F 0 "#PWR0120" H 8800 3700 30  0001 C CNN
 F 1 "GND" H 8800 3630 30  0001 C CNN
 	1    8800 3700
@@
 P 8600 3550
 F 0 "C118" V 8550 3625 30  0000 C CNN
-F 1 "10u" V 8650 3600 25  0000 C CNN
+F 1 "4u7" V 8650 3600 25  0000 C CNN
 	1    8600 3550
 	0    1    1    0
@@
 $EndComp
 $Comp
-L GND #PWR25
+L GND #PWR0121
 U 1 1 4E232F75
 P 7100 3400
-F 0 "#PWR25" H 7100 3400 30  0001 C CNN
+F 0 "#PWR0121" H 7100 3400 30  0001 C CNN
 F 1 "GND" H 7100 3330 30  0001 C CNN
 	1    7100 3400
@@
 $EndComp
 $Comp
-L GND #PWR24
+L GND #PWR0122
 U 1 1 4E232F44
 P 6450 2850
-F 0 "#PWR24" H 6450 2850 30  0001 C CNN
+F 0 "#PWR0122" H 6450 2850 30  0001 C CNN
 F 1 "GND" H 6450 2780 30  0001 C CNN
 	1    6450 2850
@@
 P 7100 2800
 F 0 "IC5" H 6900 2600 60  0000 C CNN
-F 1 "FDG6342L" H 7100 3100 60  0000 C CNN
+F 1 "FDG" H 6975 3100 60  0000 C CNN
 	1    7100 2800
 	1    0    0    -1

Commit message: Updated MicropendousX-LPC182x-GPS design. PCB routing is complete.
Connections:
- net labels added: P1_14-GPIO1_7, P2_7-GPIO0_7-ISP, P2_8-GPIO5_7-BOOT, P6_2-GPIO3_1
- net labels removed: P2_2-GPIO5_2, P2_7-ISP, P2_8, P6_4-GPIO3_3
- wire segments 25 -> 24
Other:
- note added: "Co = 4.81uF"
- note added: "Used in LCD Sheet"
- note added: "Used in System and Position Sensors Sheets"
- note removed: "Co = 10.11uF"
- moved on the sheet: TP3
Changed lines of the file:
@@
-EESchema Schematic File Version 2  date 6/8/2012 3:21:19 PM
+EESchema Schematic File Version 2  date 6/27/2012 5:02:37 AM
 LIBS:power
 LIBS:device
@@
 Sheet 6 10
 Title "MicropendousX-LPC182x-GPS"
-Date "8 jun 2012"
+Date "27 jun 2012"
 Rev "1.0"
 Comp "Opendous Inc."
@@
 Comment4 "www.MicropendousX.org"
 $EndDescr
-Text Label 3850 2100 0    20   ~ 0
-P2_7-ISP
-Wire Wire Line
-	3850 2100 4050 2100
+Text GLabel 6400 2100 0    40   BiDi ~ 0
+P2_7-GPIO0_7-ISP
+Text Notes 4525 2125 0    40   ~ 0
+Used in Power Supply Sheet
+Text GLabel 3850 2100 2    40   BiDi ~ 0
+P2_7-GPIO0_7-ISP
+Text Notes 4400 3375 0    40   ~ 0
+Used in LCD Sheet
+Text GLabel 3850 3350 2    40   Input ~ 0
+P1_14-GPIO1_7
+Text Notes 4350 5375 0    40   ~ 0
+Used in LCD Sheet
+Text GLabel 3850 5350 2    40   Input ~ 0
+P6_2-GPIO3_1
 Wire Wire Line
 	9800 3500 9200 3500
 Connection ~ 7750 2650
 Wire Wire Line
-	7750 2650 7750 2700
+	7750 2700 7750 2650
 Wire Wire Line
 	7550 2900 7750 2900
@@
 Connection ~ 8800 3650
 Wire Wire Line
-	8800 3650 8800 3700
+	8800 3700 8800 3650
 Wire Wire Line
 	8600 3650 9200 3650
@@
 Text Notes 7065 2539 0    60   ~ 0
 6342L
-Text GLabel 3850 2300 2    40   Input ~ 0
-P2_2-GPIO5_2
-Text Notes 4350 2325 0    40   ~ 0
-Used in Position Sensors Sheet
 Text GLabel 3850 1400 2    40   Input ~ 0
 P2_11-GPIO1_11
@@
 Text Notes 4350 4025 0    40   ~ 0
 Used in Power Supply Sheet
-Text Notes 4350 3925 0    40   ~ 0
-Used in Power Supply Sheet
 Text GLabel 3850 4000 2    40   Input ~ 0
 P6_5-GPIO3_4
-Text GLabel 3850 3900 2    40   Input ~ 0
-P6_4-GPIO3_3
 Text Notes 4350 4975 0    40   ~ 0
 Used in Position Sensors Sheet
@@
 Text GLabel 6600 3050 0    40   Output ~ 0
 P1_8-MMC_ENABLE
-Text Notes 4075 2025 0    40   ~ 0
-Used in System Sheet
+Text Notes 4575 2025 0    40   ~ 0
+Used in System and Position Sensors Sheets
 Text Notes 4075 1225 0    40   ~ 0
 Used in System Sheet
@@
 P2_12-GPIO1_12
 Text Notes 8625 3425 0    40   ~ 0
-Co = 10.11uF
-$Comp
-L VDD_MMC #PWR0116
+Co = 4.81uF
+$Comp
+L VDD_MMC #PWR0128
 U 1 1 4FC6B70B
 P 8600 2600
-F 0 "#PWR0116" H 8600 2700 30  0001 C CNN
+F 0 "#PWR0128" H 8600 2700 30  0001 C CNN
 F 1 "VDD_MMC" H 8600 2700 30  0000 C CNN
 	1    8600 2600
@@
 $EndComp
 $Comp
-L VDDIO_3V3 #PWR0117
+L VDDIO_3V3 #PWR0129
 U 1 1 4FC6B4E7
 P 8050 2950
-F 0 "#PWR0117" H 8050 3050 30  0001 C CNN
+F 0 "#PWR0129" H 8050 3050 30  0001 C CNN
 F 1 "VDDIO_3V3" H 8050 3050 30  0000 C CNN
 	1    8050 2950
@@
 $EndComp
 $Comp
-L VDDIO_3V3 #PWR0118
+L VDDIO_3V3 #PWR0130
 U 1 1 4FC698FB
 P 6450 2550
-F 0 "#PWR0118" H 6450 2650 30  0001 C CNN
+F 0 "#PWR0130" H 6450 2650 30  0001 C CNN
 F 1 "VDDIO_3V3" H 6450 2650 30  0000 C CNN
 	1    6450 2550
@@
 P2_9
 Text GLabel 3850 2000 2    40   BiDi ~ 0
-P2_8
-Text Notes 4425 2125 0    40   ~ 0
+P2_8-GPIO5_7-BOOT
+Text Notes 6775 2125 0    40   ~ 0
 P2_7 has weak internal pull-up to disable ISP
 Text GLabel 3850 2500 2    40   Output ~ 0
@@
 L CONN_1 TP3
 U 1 1 4FBDF820
-P 4200 2100
-F 0 "TP3" H 4250 2100 40  0000 L CNN
-F 1 "ISP" H 4200 2155 30  0001 C CNN
-	1    4200 2100
+P 6550 2100
+F 0 "TP3" H 6600 2100 40  0000 L CNN
+F 1 "ISP" H 6550 2155 30  0001 C CNN
+	1    6550 2100
 	1    0    0    -1
 $EndComp
@@
 Hirose DM3D-SF
 $Comp
-L GND #PWR0119
+L GND #PWR0131
 U 1 1 4FBDE98A
 P 10500 3800
-F 0 "#PWR0119" H 10500 3800 30  0001 C CNN
+F 0 "#PWR0131" H 10500 3800 30  0001 C CNN
 F 1 "GND" H 10500 3730 30  0001 C CNN
 	1    10500 3800
@@
 Notes:\n-
 $Comp
-L GND #PWR0120
+L GND #PWR0132
 U 1 1 4E23313A
 P 8800 3700
-F 0 "#PWR0120" H 8800 3700 30  0001 C CNN
+F 0 "#PWR0132" H 8800 3700 30  0001 C CNN
 F 1 "GND" H 8800 3630 30  0001 C CNN
 	1    8800 3700
@@
 $EndComp
 $Comp
-L GND #PWR0121
+L GND #PWR0133
 U 1 1 4E232F75
 P 7100 3400
-F 0 "#PWR0121" H 7100 3400 30  0001 C CNN
+F 0 "#PWR0133" H 7100 3400 30  0001 C CNN
 F 1 "GND" H 7100 3330 30  0001 C CNN
 	1    7100 3400
@@
 $EndComp
 $Comp
-L GND #PWR0122
+L GND #PWR0134
 U 1 1 4E232F44
 P 6450 2850
-F 0 "#PWR0122" H 6450 2850 30  0001 C CNN
+F 0 "#PWR0134" H 6450 2850 30  0001 C CNN
 F 1 "GND" H 6450 2780 30  0001 C CNN
 	1    6450 2850
