File: MicropendousX/Hardware/MicropendousX-GPS/MicropendousX-LPC182x-GPS-LCD.sch (KiCad schematic (older format))
At the start: 9 parts, among them IC1 LPC182x

Commit message: Updated MicropendousX-LPC182x-GPS design.  PCB routing almost complete.
Parts:
- added C71, C72, C76: 0u1, symbol C_MINI
- gave numbers to parts that had none: 8
Connections:
- net labels added: LCD_DATA, LCD_X+, LCD_X-, LCD_Y+, LCD_Y-
- net labels removed: X+, X-, Y+, Y-
- wire segments 67 -> 73
Other:
- note added: "I2C1 pins also used in\nPower Supply and\nSystem Sheets"
- note added: "Notes\n - Enable the Touchscreen controller to wake up the processor\n - Run STMPE610 on always-on VDD to enable Touchscreen wakeup\n - Run LCD on VDDIO since it does not need to always be on and has leakage currents\n - P1_7-GPIO0_12 is a High Drive Strength Pin that can source 32mA to the LCD Backlight LED"
- note removed: "I2C1 pins also used in\nPower Supply Sheet"
- note removed: "Notes\n - Enable the Touchscreen controller to wake up the processor\n - Run STMPE610 on always-on VDD to enable Touchscreen wakeup\n - Run LCD on VDDIO since it does not need to always be on\n - GPIO0_12 is a High Drive Strength Pin that can source 32mA to the LCD Backlight LED"
- moved on the sheet: IC4, R28, R29, R30, R31, U3

Commit message: Updated MicropendousX-LPC182x-GPS design. PCB routing is complete.
Connections:
- net labels added: LCD_LEDA, P1_14-GPIO1_7, P6_2-GPIO3_1
- no-connect marks 4 -> 6
Other:
- note added: "From EMI Sheet"
- note added: "Used in Position Sensors Sheet"
- moved on the sheet: R26, R27
