File: MicropendousX/Hardware/MicropendousX-GPS/MicropendousX-LPC182x-GPS-Power.sch (KiCad schematic (older format))
At the start: 57 parts, among them IC1 LPC182x, IC2 STC3100, IC6 LTC3559

Commit message: Updated MicropendousX-LPC182x-GPS design.  PCB routing almost complete.
Parts:
- removed C19: 0u1, symbol C_MINI
- removed L2: DNI, symbol L_MINI
- removed TP5: VBAT, symbol CONN_1
- removed TP6: STC_IO0, symbol CONN_1
- added C65: 4u7, symbol C_MINI
- added C73, C75: 0u1, symbol C_MINI
- added C74: u01, symbol C_MINI
- added R40: 10k, symbol R_MINI
- added U5: BUF, symbol BUFFER_GATE
- C17: value 4u7 -> 1u0
- C21, C36, C50: value 33n -> 0u1
- C24: value 10u -> 0u1
- C27, C29: value 10u -> 4u7
- C34: value 10u -> 1u0
- C37: value 1n0 -> 0u1
- gave numbers to parts that had none: 2
- renumbered R13 to R14, R14 to R15, R15 to R49
Connections:
- net labels added: LTC3559_EN1, LTC3559_EN2, P2_11-GPIO1_11
- net labels removed: IO0, P1_3-GPIO0_10
- wire segments 123 -> 129
- no-connect marks 0 -> 1
Other:
- note added: "74LVC1G125"
- note added: "EN1 and EN2 are high impedance inputs that are active-high"
- note added: "Notes:\n - Boot pins have weak internal pull-ups of about 50k Ohm to VDDIO\n so VDDIO_3V3 must be enabled at the same time as VDD_3V3 at startup\n - MODE HIGH enables Burst Mode which is more efficient at lower power\n - HPWR and SUSP have 2M Ohm weak pull-downs\n - regulator outputs 3.3V nominal but lowering the\n voltage to 3.0V will reduce power consumption and\n be within all components' supp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"
- note added: "This buffer is powered by EN1 to\nensure that VDD and VDDIO ramp\nup at the same time after reset.\nMCU can later tri-state this buffer\nto disable VDDIO."
- note removed: "For Testing"
- note removed: "In deep sleep mode\nVDDIO can be\ndisabled."
- note removed: "MODE HIGH\nenables\nlower power\nBurst Mode"
- note removed: "Notes:\n - Boot pins have weak internal pull-ups of about 50k Ohm to VDDIO\n so VDDIO_3V3 must be enabled at startup\n - HPWR and SUSP have 2M Ohm weak pull-downs\n - both regulators output 3.3V nominal but lowering the\n voltage to 3.0V will reduce power and be within\n all components' supply margins\n - use low ESL reverse geometry X?R caps closest to device\n - BAT54C reverse leakage is maximu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"
- moved on the sheet: BAT1, C10, C11, C13, C14, C17, C21, C24, C26, C27, C29, C30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

Commit message: Updated MicropendousX-LPC182x-GPS design. PCB routing is complete.
Parts:
- removed U5: BUF, symbol BUFFER_GATE
- added unit 12 of IC1
- added R56: 0, symbol R_MINI
- added U5: BUF, symbol BUFFER_GATE_NONINV
- R40: value 10k -> 47k
Connections:
- net labels added: P2_7-GPIO0_7-ISP, P6_11-GPIO3_7
- net labels removed: P6_4-GPIO3_3, P6_5-GPIO3_4
- wire segments 129 -> 128
- no-connect marks 1 -> 2
Other:
- note added: "74LVC1G126"
- note added: "P2_7-GPIO0_7-ISP has a weak internal pull-up to disable ISP"
- note added: "SUSP internal pull-down is too weak\nto overcome LPC182x 45k+ pull-up\nand thus requires external pull-down\n3.3(5.1/(5.1+45))=0.34V < Vil=0.4V"
- note removed: "74LVC1G125"
- note removed: "SUSP internal pull-down is too weak\nto overcome LPC182x 45k+ pull-up\nand requires external pull-down\n3.3(5.1/(5.1+45))=0.34V < Vil=0.4V"
- moved on the sheet: BAT1, C10, C11, C13, C14, C26, C30, C32, C54, C55, C73, C74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
