File: MicropendousX/Hardware/MicropendousX-GPS/MicropendousX-LPC182x-GPS-RF.sch (KiCad schematic (older format))
At the start: 44 parts, among them IC9 CC112X, X3 40MHz

Commit message: Updated MicropendousX-LPC182x-GPS design.  PCB routing almost complete.
Parts:
- added C19: 1u0, symbol C_MINI
- gave numbers to parts that had none: 37
Connections:
- net labels added: ANTenna, RF_DCPL, RF_DCPL_PFD_CHP, RF_DCPL_VCO, RF_DCPL_XOSC, RF_EXT_OSC, RF_LNA_N, RF_LNA_P, RF_LPF0, RF_LPF1, RF_PA, RF_RBIAS, RF_TRX_SW, RF_XOSC_Q1, RF_XOSC_Q2
- wire segments 71 -> 72
Other:
- note added: "WARNING: Current RF filter inductor\nand capacitor values are for 420MHz"
- note removed: "CAUTION: Current RF filter inductor\nand capacitor values are for 420MHz"
- moved on the sheet: C20, C23, C25, C33, C35, C38, C39, C40, C41, C42, R25
