File: MicropendousX/Hardware/MicropendousX-GPS/MicropendousX-LPC182x-GPS-System.sch (KiCad schematic (older format))
At the start: 26 parts, among them IC1 LPC182x, IC7 25Q, U4 JTAG, X1 12MHz, X2 32.768kHz

Commit message: Updated MicropendousX-LPC182x-GPS design.  PCB routing almost complete.
Parts:
- removed TP?: RESET, symbol CONN_1
- added C63: 0u1, symbol C_MINI
- added IC10: E48, symbol 24AA02E48
- gave numbers to parts that had none: 2
Connections:
- net labels added: P2_3-I2C1_SDA, P2_4-I2C1_SCL
- net labels removed: VBUS
- wire segments 61 -> 68
- no-connect marks 1 -> 2
Other:
- note added: "(SPF)"
- note added: "(USB)"
- note added: "24AA02"
- note added: "All WAKEUP signal sources\nhave programmable polarity"
- note added: "EUI-64 Node Identity"
- note added: "From LCD Sheet"
- note added: "Notes:\n - Run core system on always-on VDD_3V3\n - Internal Rpu is minimum 45k Ohm, so for boot selection pull-down resistor,\n 19k is max. usable as 3.3(19/(19+45))=0.98V < Vil=(3.3*.3)=1V\n - E48 EEPROM is used to give every node its own unique EUI-64 address"
- note added: "nTRST, TMS, and TDI have weak internal pull-up resistors"
- note removed: "DFN 6x5mm"
- note removed: "Has internal weak pull-up"
- note removed: "Notes:\n - Run core system on always-on VDD_3V3\n - Rpu is min. 45k Ohm, so for boot selection pull-down resistor,\n 19k is max. usable as 3.3(19/(19+45))=0.98V < Vil=(3.3*.3)=1V\n - LTC3559 soft-start takes 500us but Vih(EN2)=1.2V means\n that VDD ramp will begin VDDIO ramp after about 200us.\n VDDIO should be >2.0V=Vih(GPIO) about 300us after\n VDD>1.2V or 500us after VDD ramp begins.\n Vih(RES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"
- note removed: "TODO - are all the wakeup signals Active-LOW"
- note removed: "USB0_VBUS includes 64k Ohm pull-down"
- moved on the sheet: R37, R42, R43, R44

Commit message: Updated MicropendousX-LPC182x-GPS design. PCB routing is complete.
Connections:
- net labels added: P2_8-GPIO5_7-BOOT
- net labels removed: P2_8
Other:
- moved on the sheet: R37, R42, R43
Changed lines of the file:
@@
-EESchema Schematic File Version 2  date 6/8/2012 3:21:19 PM
+EESchema Schematic File Version 2  date 6/27/2012 5:02:37 AM
 LIBS:power
 LIBS:device
@@
 Sheet 8 10
 Title "MicropendousX-LPC182x-GPS"
-Date "8 jun 2012"
+Date "27 jun 2012"
 Rev "1.0"
 Comp "Opendous Inc."
@@
 RTC_ALARM
 $Comp
-L VDD_3V3 #PWR0132
+L VDD_3V3 #PWR0142
 U 1 1 4FCC4AF3
-P 9400 3700
-F 0 "#PWR0132" H 9400 3800 30  0001 C CNN
-F 1 "VDD_3V3" H 9400 3800 30  0000 C CNN
-	1    9400 3700
+P 9500 3700
+F 0 "#PWR0142" H 9500 3800 30  0001 C CNN
+F 1 "VDD_3V3" H 9500 3800 30  0000 C CNN
+	1    9500 3700
 	1    0    0    -1
 $EndComp
@@
 	7400 1450 7300 1450
 Wire Wire Line
-	8600 4100 8600 4150
-Wire Wire Line
-	8600 3900 8600 3800
-Wire Wire Line
-	8600 3800 8550 3800
+	8350 4100 8350 4150
+Wire Wire Line
+	8350 3900 8350 3800
+Wire Wire Line
+	8350 3800 8300 3800
 Wire Wire Line
 	10600 3800 10650 3800
@@
 	5600 5850 5600 5900
 Wire Wire Line
-	9200 3900 9200 3800
-Wire Wire Line
-	9200 3800 9100 3800
-Wire Wire Line
-	9300 3950 9400 3950
-Wire Wire Line
-	9000 4150 9000 4200
-Wire Wire Line
-	9400 3750 9400 3700
-Wire Wire Line
-	9100 3950 9000 3950
+	9300 3900 9300 3800
+Wire Wire Line
+	9300 3800 9200 3800
+Wire Wire Line
+	9400 3950 9500 3950
+Wire Wire Line
+	9100 4150 9100 4200
+Wire Wire Line
+	9500 3750 9500 3700
+Wire Wire Line
+	9200 3950 9100 3950
 Wire Wire Line
 	10650 4100 10650 4150
@@
 $EndComp
 $Comp
-L GND #PWR0133
+L GND #PWR0143
 U 1 1 4FC89B57
 P 7500 1650
-F 0 "#PWR0133" H 7500 1650 30  0001 C CNN
+F 0 "#PWR0143" H 7500 1650 30  0001 C CNN
 F 1 "GND" H 7500 1580 30  0001 C CNN
 	1    7500 1650
@@
 $EndComp
 $Comp
-L VDDIO_3V3 #PWR0134
+L VDDIO_3V3 #PWR0144
 U 1 1 4FC89B54
 P 7500 1350
-F 0 "#PWR0134" H 7500 1450 30  0001 C CNN
+F 0 "#PWR0144" H 7500 1450 30  0001 C CNN
 F 1 "VDDIO_3V3" H 7500 1450 30  0000 C CNN
 	1    7500 1350
@@
 $EndComp
 $Comp
-L GND #PWR0135
+L GND #PWR0145
 U 1 1 4FC7294E
-P 8600 4150
-F 0 "#PWR0135" H 8600 4150 30  0001 C CNN
-F 1 "GND" H 8600 4080 30  0001 C CNN
-	1    8600 4150
+P 8350 4150
+F 0 "#PWR0145" H 8350 4150 30  0001 C CNN
+F 1 "GND" H 8350 4080 30  0001 C CNN
+	1    8350 4150
 	1    0    0    -1
 $EndComp
@@
 L R_MINI R37
 U 1 1 4FC7294D
-P 8600 4000
-F 0 "R37" V 8575 4050 25  0000 C CNN
-F 1 "10k" V 8625 4050 20  0000 C CNN
-	1    8600 4000
+P 8350 4000
+F 0 "R37" V 8325 4050 25  0000 C CNN
+F 1 "10k" V 8375 4050 20  0000 C CNN
+	1    8350 4000
 	0    1    1    0
 $EndComp
@@
 WAKEUP_Touchscreen
 $Comp
-L VDD_3V3 #PWR0136
+L VDD_3V3 #PWR0146
 U 1 1 4FC6BB03
 P 4500 4600
-F 0 "#PWR0136" H 4500 4700 30  0001 C CNN
+F 0 "#PWR0146" H 4500 4700 30  0001 C CNN
 F 1 "VDD_3V3" H 4500 4700 30  0000 C CNN
 	1    4500 4600
@@
 $EndComp
 $Comp
-L GND #PWR0137
+L GND #PWR0147
 U 1 1 4FC6BAF9
 P 4500 5100
-F 0 "#PWR0137" H 4500 5100 30  0001 C CNN
+F 0 "#PWR0147" H 4500 5100 30  0001 C CNN
 F 1 "GND" H 4500 5030 30  0001 C CNN
 	1    4500 5100
@@
 $EndComp
 $Comp
-L VDD_3V3 #PWR0138
+L VDD_3V3 #PWR0148
 U 1 1 4FC696D4
 P 4300 4100
-F 0 "#PWR0138" H 4300 4200 30  0001 C CNN
+F 0 "#PWR0148" H 4300 4200 30  0001 C CNN
 F 1 "VDD_3V3" H 4300 4200 30  0000 C CNN
 	1    4300 4100
@@
 $EndComp
 $Comp
-L VDD_3V3 #PWR0139
+L VDD_3V3 #PWR0149
 U 1 1 4FC696CB
 P 6250 6100
-F 0 "#PWR0139" H 6250 6200 30  0001 C CNN
+F 0 "#PWR0149" H 6250 6200 30  0001 C CNN
 F 1 "VDD_3V3" H 6250 6200 30  0000 C CNN
 	1    6250 6100
@@
 $EndComp
 $Comp
-L VDD_3V3 #PWR0140
+L VDD_3V3 #PWR0150
 U 1 1 4FC696BC
 P 5650 2450
-F 0 "#PWR0140" H 5650 2550 30  0001 C CNN
+F 0 "#PWR0150" H 5650 2550 30  0001 C CNN
 F 1 "VDD_3V3" H 5650 2550 30  0000 C CNN
 	1    5650 2450
@@
 $EndComp
 $Comp
-L VDD_3V3 #PWR0141
+L VDD_3V3 #PWR0151
 U 1 1 4FC696B9
 P 5600 5600
-F 0 "#PWR0141" H 5600 5700 30  0001 C CNN
+F 0 "#PWR0151" H 5600 5700 30  0001 C CNN
 F 1 "VDD_3V3" H 5600 5700 30  0000 C CNN
 	1    5600 5600
@@
 $EndComp
 $Comp
-L VDD_3V3 #PWR0142
+L VDD_3V3 #PWR0152
 U 1 1 4FC696B4
 P 8450 1100
-F 0 "#PWR0142" H 8450 1200 30  0001 C CNN
+F 0 "#PWR0152" H 8450 1200 30  0001 C CNN
 F 1 "VDD_3V3" H 8450 1200 30  0000 C CNN
 	1    8450 1100
@@
 $EndComp
 $Comp
-L GND #PWR0143
+L GND #PWR0153
 U 1 1 4FBDF970
 P 10100 1400
-F 0 "#PWR0143" H 10100 1400 30  0001 C CNN
+F 0 "#PWR0153" H 10100 1400 30  0001 C CNN
 F 1 "GND" H 10100 1330 30  0001 C CNN
 	1    10100 1400
@@
 $EndComp
 $Comp
-L GND #PWR0144
+L GND #PWR0154
 U 1 1 4E22F2F2
 P 10650 4150
-F 0 "#PWR0144" H 10650 4150 30  0001 C CNN
+F 0 "#PWR0154" H 10650 4150 30  0001 C CNN
 F 1 "GND" H 10650 4080 30  0001 C CNN
 	1    10650 4150
@@
 L JUMPER-3 JP8
 U 1 1 4E22F2E5
-P 9200 3950
-F 0 "JP8" H 9200 3890 30  0000 C CNN
-F 1 "JUMPER-3" H 9200 3950 30  0001 C CNN
-	1    9200 3950
+P 9300 3950
+F 0 "JP8" H 9300 3890 30  0000 C CNN
+F 1 "JUMPER-3" H 9300 3950 30  0001 C CNN
+	1    9300 3950
 	1    0    0    -1
 $EndComp
@@
 L R_MINI R42
 U 1 1 4E22F2E4
-P 9000 4050
-F 0 "R42" V 8975 4100 25  0000 C CNN
-F 1 "10k" V 9025 4100 20  0000 C CNN
-	1    9000 4050
+P 9100 4050
+F 0 "R42" V 9075 4100 25  0000 C CNN
+F 1 "10k" V 9125 4100 20  0000 C CNN
+	1    9100 4050
 	0    1    1    0
 $EndComp
@@
 L R_MINI R43
 U 1 1 4E22F2E3
-P 9400 3850
-F 0 "R43" V 9375 3900 25  0000 C CNN
-F 1 "10k" V 9425 3900 20  0000 C CNN
-	1    9400 3850
-	0    1    1    0
-$EndComp
-$Comp
-L GND #PWR0145
+P 9500 3850
+F 0 "R43" V 9475 3900 25  0000 C CNN
+F 1 "10k" V 9525 3900 20  0000 C CNN
+	1    9500 3850
+	0    1    1    0
+$EndComp
+$Comp
+L GND #PWR0155
 U 1 1 4E22F2E1
-P 9000 4200
-F 0 "#PWR0145" H 9000 4200 30  0001 C CNN
-F 1 "GND" H 9000 4130 30  0001 C CNN
-	1    9000 4200
-	1    0    0    -1
-$EndComp
-Text GLabel 8550 3800 0    40   BiDi ~ 0
+P 9100 4200
+F 0 "#PWR0155" H 9100 4200 30  0001 C CNN
+F 1 "GND" H 9100 4130 30  0001 C CNN
+	1    9100 4200
+	1    0    0    -1
+$EndComp
+Text GLabel 8300 3800 0    40   BiDi ~ 0
 P2_9
-Text GLabel 9100 3800 0    40   BiDi ~ 0
-P2_8
-Text GLabel 10100 4150 0    40   BiDi ~ 0
+Text GLabel 9200 3800 0    40   BiDi ~ 0
+P2_8-GPIO5_7-BOOT
+Text GLabel 10200 4150 0    40   BiDi ~ 0
 P1_1-SSP0_MISO
 Text GLabel 10600 3800 0    40   BiDi ~ 0
 P1_2-SSP0_MOSI
 $Comp
-L GND #PWR0146
+L GND #PWR0156
 U 1 1 4E22A159
 P 4950 6600
-F 0 "#PWR0146" H 4950 6600 30  0001 C CNN
+F 0 "#PWR0156" H 4950 6600 30  0001 C CNN
 F 1 "GND" H 4950 6530 30  0001 C CNN
 	1    4950 6600
@@
 $EndComp
 $Comp
-L GND #PWR0147
+L GND #PWR0157
 U 1 1 4E22A148
 P 5600 5900
-F 0 "#PWR0147" H 5600 5900 30  0001 C CNN
+F 0 "#PWR0157" H 5600 5900 30  0001 C CNN
 F 1 "GND" H 5600 5830 30  0001 C CNN
 	1    5600 5900
@@
 Power-up Reset is not reliable with\nfast VDD ramps so a Reset delay is\nrequired (Errata 20110701 POR.1)
 $Comp
-L GND #PWR0148
+L GND #PWR0158
 U 1 1 4E2299FE
 P 5200 2950
-F 0 "#PWR0148" H 5200 2950 30  0001 C CNN
+F 0 "#PWR0158" H 5200 2950 30  0001 C CNN
 F 1 "GND" H 5200 2880 30  0001 C CNN
 	1    5200 2950
@@
 $EndComp
 $Comp
-L GND #PWR0149
+L GND #PWR0159
 U 1 1 4E229902
 P 4650 3800
-F 0 "#PWR0149" H 4650 3800 30  0001 C CNN
+F 0 "#PWR0159" H 4650 3800 30  0001 C CNN
 F 1 "GND" H 4650 3730 30  0001 C CNN
 	1    4650 3800
@@
 XTAL1
 $Comp
-L GND #PWR0150
+L GND #PWR0160
 U 1 1 4E2298C3
 P 4650 3300
-F 0 "#PWR0150" H 4650 3300 30  0001 C CNN
+F 0 "#PWR0160" H 4650 3300 30  0001 C CNN
 F 1 "GND" H 4650 3230 30  0001 C CNN
 	1    4650 3300
@@
 nRESET
 $Comp
-L GND #PWR0151
+L GND #PWR0161
 U 1 1 4DE9F22E
 P 8450 1600
-F 0 "#PWR0151" H 8450 1600 30  0001 C CNN
+F 0 "#PWR0161" H 8450 1600 30  0001 C CNN
 F 1 "GND" H 8450 1530 30  0001 C CNN
 	1    8450 1600
