File: MicropendousX/Hardware/MicropendousX-GPS/MicropendousX-LPC182x-GPS-Vias.sch (KiCad schematic (older format))
At the start: 393 parts

Commit message: Updated MicropendousX-LPC182x-GPS design.  PCB routing almost complete.
Parts:
- removed Mask1, Mask2, Mask3, Mask4: Mask, symbol VIA
Connections:
- net labels added: ADC0_0, ADC0_3, ADCTRIG1, LCD_DATA, LCD_X+, LCD_X-, LCD_Y+, LCD_Y-, LTC3559_EN1, LTC3559_EN2, P1_0-SSP0_SSEL, P1_1-SSP0_MISO, P1_2-SSP0_MOSI, P2_10-GPIO0_14, P2_11-GPIO1_11, P2_12-GPIO1_12, P2_13-GPIO1_13, P2_3-I2C1_SDA, P2_4-I2C1_SCL, P2_8, P3_0-SSP0_SCK, P3_3-SPIFI_SCK, P3_4-SPIFI_SIO3, P3_5-SPIFI_SIO2, P3_6-SPIFI_MISO, P3_7-SPIFI_MOSI, P3_8-SPIFI_CS, P6_4-GPIO3_3, P6_5-GPIO3_4, RTC_ALARM, TDI, VDD_3V3, VDD_MOT, VDD_RF, WAKEUP0, WAKEUP_Movement, WAKEUP_Touchscreen
- wire segments 54 -> 90
- no-connect marks 4 -> 0
Other:
- moved on the sheet: V1, V10, V100, V101, V102, V103, V104, V105, V106, V107, V108, V109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

Commit message: Updated MicropendousX-LPC182x-GPS design. PCB routing is complete.
Parts:
- removed V192, V213, V231, V272, V273, V274, V275, V276, V277, V278, V279, V280, V281, V282, V283, V284, V285, V286, V287, V288, V289, V290, V291, V292, V293, V294, V295, V296, V297, V298, V299, V342, V343, V347, V348, V349, V350, V351, V352, V353, V354, V355, V356, V357, V358, V359, V360, V361, V362, V363, V364, V365, V366, V367, V368, V369, V370, V371, V372, V373, V374, V375, V376, V377, V379, V380, V381, V382, V383, V384, V385, V386, V387, V388, V389: VIA, symbol VIA
Connections:
- net labels added: CLK2-MMC_CLK, GPS_FIX, LCD_LEDA, P1_10-MMC_DAT1, P1_11-MMC_DAT2, P1_12-MMC_DAT3, P1_13-MMC_CD, P1_14-GPIO1_7, P1_15-GPIO0_2, P1_19-SSP1_SCK, P1_20-SSP1_SSEL, P1_6-MMC_CMD, P1_8-MMC_ENABLE, P1_9-MMC_DAT0, P2_0-U0_TXD, P2_1-U0_RXD, P2_7-GPIO0_7-ISP, P2_8-GPIO5_7-BOOT, P6_11-GPIO3_7, P6_2-GPIO3_1
- net labels removed: 3V3, 5V0, ADC0_0-DAC, ADC1_1, CLKOUT-I2S1_RX_SCK, EMC_A00, EMC_A02, EMC_A03, EMC_A04, EMC_A05, EMC_A06, EMC_A07, EMC_A08, EMC_D00, EMC_D01, EMC_D02-MMC_DAT0, EMC_D03-MMC_DAT1, EMC_D04-MMC_DAT2, EMC_D05-MMC_DAT3, EMC_D06-MMC_CD, EMC_D07, GPIO0_11, GPIO0_12, GPIO0_13, GPIO3_5, GPIO3_7, GPIO5_0-EMC_A13, GPIO5_2, I2C1_SCL-U3_RXD, I2C1_SDA-U3_TXD, I2S0_TX_SCK, LTC3559_VCC, LTC3559_~CHRG~, MMC_CLK, MMC_VDD, P2_8, P6_4-GPIO3_3, P6_5-GPIO3_4, SPIFI_SCK-CGU_OUT1, SPIFI_SIO2-I2S1_RX_WS, SPIFI_SIO3-I2S1_RX_SDA, SSP1_MISO, SSP1_MOSI, SSP1_SCK, SSP1_SSEL, TDO, TX0, TX1, U2_RXD-GPIO0_3, U2_TXD-GPIO0_2, USB0_DM, USB0_DP, USB0_ID, VDD3V3, ~EMC_CS0~, ~EMC_OE~, ~EMC_WE~-MMC_CMD, ~RESET~
- wire segments 90 -> 89
Other:
- moved on the sheet: V1, V10, V100, V101, V102, V103, V104, V105, V106, V107, V108, V109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
